File: mower/PCB/TRANSMITTER_DIP/TRANSMITTER.kicad_sch (KiCad schematic)
At the start: 16 parts, among them J1 BOT POWER, J2 POWER IN, J3 SHUNT, J4 COIL OUT, J5 COIL POWER IN, Q1 IRF3205, U1 LM358, U4 LM555xN

Commit message: .
Connections:
- net GND: now also U1.4 (V-)
- net VCC: now also U1.8 (V+)
Changed lines of the file:
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@@
 	(wire
 		(pts
-			(xy 81.28 119.38) (xy 81.28 125.73)
+			(xy 78.74 119.38) (xy 78.74 127)
 		)
 		(stroke
@@
 	(wire
 		(pts
-			(xy 81.28 140.97) (xy 81.28 149.86)
+			(xy 78.74 142.24) (xy 78.74 153.67)
 		)
 		(stroke
@@
 	(symbol
 		(lib_id "power:VCC")
-		(at 81.28 119.38 0)
+		(at 78.74 119.38 0)
 		(unit 1)
 		(exclude_from_sim no)
@@
 		(fields_autoplaced yes)
 		(property "Reference" "#PWR06"
-			(at 81.28 123.19 0)
+			(at 78.74 123.19 0)
 			(effects
 				(font
@@
 		)
 		(property "Value" "VCC"
-			(at 81.28 114.3 0)
+			(at 78.74 114.3 0)
 			(effects
 				(font
@@
 		)
 		(property "Footprint" ""
-			(at 81.28 119.38 0)
+			(at 78.74 119.38 0)
 			(effects
 				(font
@@
 		)
 		(property "Datasheet" ""
-			(at 81.28 119.38 0)
+			(at 78.74 119.38 0)
 			(effects
 				(font
@@
 		)
 		(property "Description" "Power symbol creates a global label with name \"VCC\""
-			(at 81.28 119.38 0)
+			(at 78.74 119.38 0)
 			(effects
 				(font
@@
 	(symbol
 		(lib_id "power:GND")
-		(at 81.28 149.86 0)
+		(at 78.74 153.67 0)
 		(unit 1)
 		(exclude_from_sim no)
@@
 		(fields_autoplaced yes)
 		(property "Reference" "#PWR07"
-			(at 81.28 156.21 0)
+			(at 78.74 160.02 0)
 			(effects
 				(font
@@
 		)
 		(property "Value" "GND"
-			(at 81.28 154.94 0)
+			(at 78.74 158.75 0)
 			(effects
 				(font
@@
 		)
 		(property "Footprint" ""
-			(at 81.28 149.86 0)
+			(at 78.74 153.67 0)
 			(effects
 				(font
@@
 		)
 		(property "Datasheet" ""
-			(at 81.28 149.86 0)
+			(at 78.74 153.67 0)
 			(effects
 				(font
@@
 		)
 		(property "Description" "Power symbol creates a global label with name \"GND\" , ground"
-			(at 81.28 149.86 0)
-			(effects
-				(font
+			(at 78.74 153.67 0)
+			(effects
+				(font
