File: mower/PCB/TRANSMITTER_DIP/TRANSMITTER_PANEL.kicad_pcb (KiCad board)
At the start: 2 copper layers, 335 x 169.4 mm, 336 parts, among them J1 BOT POWER, J2 POWER IN, J3 SHUNT, J4 COIL OUT, J5 COIL POWER IN, Q1 IRF3205, U1 LM358, U4 LM555xN

Commit message: .
Parts:
- removed the C1 at (121.3, 179.5)
- removed the C1 at (9.28, 94.3)
- removed the C1 at (177.3, 94.3)
- removed the C1 at (177.3, 179.5)
- removed the C1 at (289.3, 179.5)
- removed the C1 at (177.3, 51.7)
- removed the C1 at (289.3, 94.3)
- removed the C1 at (121.3, 94.3)
- removed the C1 at (121.3, 136.9)
- removed the C1 at (65.3, 179.5)
- removed the C1 at (289.3, 51.7)
- removed the C1 at (233.3, 136.9)
- removed the C1 at (9.28, 51.7)
- removed the C1 at (233.3, 94.3)
- removed the C1 at (289.3, 136.9)
- removed the C1 at (9.28, 179.5)
- removed the C1 at (65.3, 51.7)
- removed the C1 at (9.28, 136.9)
- removed the C1 at (121.3, 51.7)
- removed the C1 at (65.3, 94.3)
- removed the C1 at (233.3, 51.7)
- removed the C1 at (65.3, 136.9)
- removed the C1 at (233.3, 179.5)
- removed the C1 at (177.3, 136.9)
- removed the D1 at (100.6, 123.0)
- removed the D1 at (212.6, 80.4)
- removed the D1 at (268.6, 123.0)
- removed the D1 at (100.6, 80.4)
- removed the D1 at (-11.4, 80.4)
- removed the D1 at (268.6, 165.6)
- removed the D1 at (100.6, 37.8)
- removed the D1 at (156.6, 37.8)
- removed the D1 at (44.6, 123.0)
- removed the D1 at (44.6, 165.6)
- removed the D1 at (-11.4, 123.0)
- removed the D1 at (44.6, 37.8)
- removed the D1 at (156.6, 123.0)
- removed the D1 at (268.6, 37.8)
- removed the D1 at (212.6, 165.6)
- removed the D1 at (156.6, 80.4)
- removed the D1 at (-11.4, 37.8)
- removed the D1 at (156.6, 165.6)
- removed the D1 at (212.6, 37.8)
- removed the D1 at (212.6, 123.0)
- removed the D1 at (-11.4, 165.6)
- removed the D1 at (44.6, 80.4)
- removed the D1 at (100.6, 165.6)
- removed the D1 at (268.6, 80.4)
- removed the J1 at (175.5, 30.2)
- removed the J1 at (287.5, 115.4)
- removed the J1 at (175.5, 115.4)
- removed the J1 at (119.5, 158.0)
- removed the J1 at (63.5, 158.0)
- removed the J1 at (63.5, 115.4)
- removed the J1 at (231.5, 115.4)
- removed the J1 at (63.5, 72.8)
- removed the J1 at (231.5, 72.8)
- removed the J1 at (175.5, 72.8)
- removed the J1 at (7.50, 115.4)
- removed the J1 at (231.5, 30.2)
- removed the J1 at (287.5, 158.0)
- removed the J1 at (119.5, 72.8)
- removed the J1 at (7.50, 72.8)
- removed the J1 at (7.50, 30.2)
- removed the J1 at (287.5, 30.2)
- removed the J1 at (7.50, 158.0)
- removed the J1 at (63.5, 30.2)
- removed the J1 at (287.5, 72.8)
- removed the J1 at (119.5, 30.2)
- removed the J1 at (175.5, 158.0)
- removed the J1 at (231.5, 158.0)
- removed the J1 at (119.5, 115.4)
- removed the J2 at (86.5, 72.8)
- removed the J2 at (30.5, 158.0)
- removed the J2 at (142.5, 30.2)
- removed the J2 at (86.5, 158.0)
- removed the J2 at (30.5, 72.8)
- removed the J2 at (254.5, 158.0)
- removed the J2 at (198.5, 158.0)
- removed the J2 at (198.5, 30.2)
- removed the J2 at (310.5, 30.2)
- removed the J2 at (86.5, 30.2)
- removed the J2 at (254.5, 30.2)
- removed the J2 at (86.5, 115.4)
- removed the J2 at (142.5, 115.4)
- removed the J2 at (254.5, 115.4)
- removed the J2 at (310.5, 158.0)
- removed the J2 at (142.5, 158.0)
- removed the J2 at (254.5, 72.8)
- removed the J2 at (30.5, 30.2)
- removed the J2 at (310.5, 115.4)
- removed the J2 at (198.5, 115.4)
- removed the J2 at (310.5, 72.8)
- removed the J2 at (30.5, 115.4)
- removed the J2 at (198.5, 72.8)
- removed the J2 at (142.5, 72.8)
- removed the J3 at (186.9, 115.4)
- removed the J3 at (74.9, 72.8)
- removed the J3 at (298.9, 72.8)
- removed the J3 at (18.9, 115.4)
- removed the J3 at (298.9, 158.0)
- removed the J3 at (74.9, 115.4)
- removed the J3 at (74.9, 30.2)
- removed the J3 at (298.9, 115.4)
- removed the J3 at (130.9, 158.0)
- removed the J3 at (242.9, 115.4)
- removed the J3 at (130.9, 115.4)
- removed the J3 at (242.9, 158.0)
- removed the J3 at (18.9, 158.0)
- removed the J3 at (18.9, 30.2)
- removed the J3 at (130.9, 72.8)
- removed the J3 at (242.9, 72.8)
- removed the J3 at (130.9, 30.2)
- removed the J3 at (298.9, 30.2)
- removed the J3 at (186.9, 30.2)
- removed the J3 at (186.9, 72.8)
- removed the J3 at (74.9, 158.0)
- removed the J3 at (18.9, 72.8)
- removed the J3 at (186.9, 158.0)
- removed the J3 at (242.9, 30.2)
- removed the J4 at (107.9, 72.8)
- removed the J4 at (-4.06, 115.4)
- removed the J4 at (163.9, 30.2)
- removed the J4 at (-4.06, 72.8)
- removed the J4 at (107.9, 30.2)
- removed the J4 at (219.9, 158.0)
- removed the J4 at (275.9, 158.0)
- removed the J4 at (51.9, 72.8)
- removed the J4 at (-4.06, 30.2)
- removed the J4 at (219.9, 72.8)
- removed the J4 at (219.9, 115.4)
- removed the J4 at (275.9, 115.4)
- removed the J4 at (107.9, 158.0)
- removed the J4 at (163.9, 115.4)
- removed the J4 at (51.9, 158.0)
- removed the J4 at (163.9, 158.0)
- removed the J4 at (51.9, 30.2)
- removed the J4 at (275.9, 30.2)
- removed the J4 at (275.9, 72.8)
- removed the J4 at (107.9, 115.4)
- removed the J4 at (51.9, 115.4)
- removed the J4 at (219.9, 30.2)
- removed the J4 at (-4.06, 158.0)
- removed the J4 at (163.9, 72.8)
- removed the J5 at (210.3, 42.5)
- removed the J5 at (154.3, 170.3)
- removed the J5 at (210.3, 85.1)
- removed the J5 at (154.3, 127.7)
- removed the J5 at (98.3, 42.5)
- removed the J5 at (266.3, 170.3)
- removed the J5 at (154.3, 42.5)
- removed the J5 at (266.3, 85.1)
- removed the J5 at (42.3, 127.7)
- removed the J5 at (266.3, 42.5)
- removed the J5 at (98.3, 170.3)
- removed the J5 at (154.3, 85.1)
- removed the J5 at (266.3, 127.7)
- removed the J5 at (210.3, 127.7)
- removed the J5 at (-13.7, 170.3)
- removed the J5 at (42.3, 170.3)
- removed the J5 at (42.3, 42.5)
- removed the J5 at (-13.7, 42.5)
- removed the J5 at (210.3, 170.3)
- removed the J5 at (-13.7, 127.7)
- removed the J5 at (-13.7, 85.1)
- removed the J5 at (42.3, 85.1)
- removed the J5 at (98.3, 85.1)
- removed the J5 at (98.3, 127.7)
- removed the Q1 at (2.90, 40.8)
- removed the Q1 at (114.9, 40.8)
- removed the Q1 at (170.9, 168.6)
- removed the Q1 at (2.90, 168.6)
- removed the Q1 at (58.9, 40.8)
- removed the Q1 at (226.9, 168.6)
- removed the Q1 at (226.9, 40.8)
- removed the Q1 at (226.9, 126.0)
- removed the Q1 at (114.9, 83.4)
- removed the Q1 at (170.9, 40.8)
- removed the Q1 at (170.9, 126.0)
- removed the Q1 at (282.9, 168.6)
- removed the Q1 at (282.9, 40.8)
- removed the Q1 at (58.9, 126.0)
- removed the Q1 at (58.9, 83.4)
- removed the Q1 at (226.9, 83.4)
- removed the Q1 at (58.9, 168.6)
- removed the Q1 at (282.9, 126.0)
- removed the Q1 at (2.90, 83.4)
- removed the Q1 at (114.9, 168.6)
- removed the Q1 at (282.9, 83.4)
- removed the Q1 at (2.90, 126.0)
- removed the Q1 at (114.9, 126.0)
- removed the Q1 at (170.9, 83.4)
- removed the R1 at (127.4, 168.2)
- removed the R1 at (183.4, 40.4)
- removed the R1 at (71.4, 125.6)
- removed the R1 at (295.4, 125.6)
- removed the R1 at (15.4, 168.2)
- removed the R1 at (71.4, 40.4)
- removed the R1 at (295.4, 83.0)
- removed the R1 at (71.4, 83.0)
- removed the R1 at (295.4, 40.4)
- removed the R1 at (127.4, 125.6)
- removed the R1 at (183.4, 83.0)
- removed the R1 at (239.4, 168.2)
- removed the R1 at (127.4, 83.0)
- removed the R1 at (239.4, 83.0)
- removed the R1 at (71.4, 168.2)
- removed the R1 at (183.4, 168.2)
- removed the R1 at (15.4, 40.4)
- removed the R1 at (15.4, 125.6)
- removed the R1 at (239.4, 125.6)
- removed the R1 at (127.4, 40.4)
- removed the R1 at (239.4, 40.4)
- removed the R1 at (295.4, 168.2)
- removed the R1 at (15.4, 83.0)
- removed the R1 at (183.4, 125.6)
- removed the R2 at (16.1, 174.4)
- removed the R2 at (72.1, 131.8)
- removed the R2 at (16.1, 131.8)
- removed the R2 at (16.1, 89.2)
- removed the R2 at (72.1, 174.4)
- removed the R2 at (240.1, 174.4)
- removed the R2 at (296.1, 174.4)
- removed the R2 at (240.1, 131.8)
- removed the R2 at (240.1, 89.2)
- removed the R2 at (296.1, 46.6)
- removed the R2 at (296.1, 89.2)
- removed the R2 at (128.1, 131.8)
- removed the R2 at (184.1, 131.8)
- removed the R2 at (72.1, 46.6)
- removed the R2 at (128.1, 89.2)
- removed the R2 at (296.1, 131.8)
- removed the R2 at (240.1, 46.6)
- removed the R2 at (184.1, 89.2)
- removed the R2 at (184.1, 46.6)
- removed the R2 at (128.1, 174.4)
- removed the R2 at (128.1, 46.6)
- removed the R2 at (16.1, 46.6)
- removed the R2 at (72.1, 89.2)
- removed the R2 at (184.1, 174.4)
- removed the R3 at (-5.92, 140.3)
- removed the R3 at (-5.92, 55.1)
- removed the R3 at (50.1, 97.7)
- removed the R3 at (274.1, 140.3)
- removed the R3 at (162.1, 97.7)
- removed the R3 at (218.1, 182.9)
- removed the R3 at (-5.92, 182.9)
- removed the R3 at (274.1, 97.7)
- removed the R3 at (218.1, 140.3)
- removed the R3 at (50.1, 182.9)
- removed the R3 at (-5.92, 97.7)
- removed the R3 at (106.1, 55.1)
- removed the R3 at (162.1, 55.1)
- removed the R3 at (106.1, 97.7)
- removed the R3 at (162.1, 140.3)
- removed the R3 at (50.1, 140.3)
- removed the R3 at (106.1, 140.3)
- removed the R3 at (274.1, 182.9)
- removed the R3 at (50.1, 55.1)
- removed the R3 at (162.1, 182.9)
- removed the R3 at (106.1, 182.9)
- removed the R3 at (218.1, 55.1)
- removed the R3 at (274.1, 55.1)
- removed the R3 at (218.1, 97.7)
- removed the R4 at (162.0, 185.4)
- removed the R4 at (274.0, 57.6)
- removed the R4 at (218.0, 185.4)
- removed the R4 at (162.0, 100.2)
- removed the R4 at (162.0, 57.6)
- removed the R4 at (106.0, 57.6)
- removed the R4 at (106.0, 185.4)
- removed the R4 at (50.0, 100.2)
- removed the R4 at (106.0, 100.2)
- removed the R4 at (106.0, 142.8)
- removed the R4 at (-6.00, 185.4)
- removed the R4 at (-6.00, 100.2)
- removed the R4 at (218.0, 57.6)
- removed the R4 at (-6.00, 57.6)
- removed the R4 at (274.0, 185.4)
- removed the R4 at (218.0, 142.8)
- removed the R4 at (218.0, 100.2)
- removed the R4 at (162.0, 142.8)
- removed the R4 at (50.0, 57.6)
- removed the R4 at (274.0, 142.8)
- removed the R4 at (-6.00, 142.8)
- removed the R4 at (50.0, 185.4)
- removed the R4 at (274.0, 100.2)
- removed the R4 at (50.0, 142.8)
- removed the U1 at (248.2, 45.7)
- removed the U1 at (24.2, 45.7)
- removed the U1 at (80.2, 88.3)
- removed the U1 at (24.2, 173.5)
- removed the U1 at (80.2, 130.9)
- removed the U1 at (192.2, 173.5)
- removed the U1 at (192.2, 88.3)
- removed the U1 at (248.2, 130.9)
- removed the U1 at (136.2, 173.5)
- removed the U1 at (248.2, 88.3)
- removed the U1 at (24.2, 130.9)
- removed the U1 at (304.2, 173.5)
- removed the U1 at (304.2, 130.9)
- removed the U1 at (304.2, 88.3)
- removed the U1 at (192.2, 45.7)
- removed the U1 at (136.2, 88.3)
- removed the U1 at (24.2, 88.3)
- removed the U1 at (80.2, 45.7)
- removed the U1 at (248.2, 173.5)
- removed the U1 at (80.2, 173.5)
- removed the U1 at (192.2, 130.9)
- removed the U1 at (304.2, 45.7)
- removed the U1 at (136.2, 130.9)
- removed the U1 at (136.2, 45.7)
- removed the U4 at (-2.51, 46.8)
- removed the U4 at (109.5, 132.0)
- removed the U4 at (109.5, 46.8)
- removed the U4 at (277.5, 132.0)
- removed the U4 at (109.5, 174.6)
- removed the U4 at (109.5, 89.4)
- removed the U4 at (53.5, 132.0)
- removed the U4 at (221.5, 89.4)
- removed the U4 at (221.5, 132.0)
- removed the U4 at (-2.51, 174.6)
- removed the U4 at (165.5, 46.8)
- removed the U4 at (53.5, 174.6)
- removed the U4 at (165.5, 174.6)
- removed the U4 at (277.5, 174.6)
- removed the U4 at (165.5, 132.0)
- removed the U4 at (277.5, 46.8)
- removed the U4 at (165.5, 89.4)
- removed the U4 at (221.5, 46.8)
- removed the U4 at (277.5, 89.4)
- removed the U4 at (221.5, 174.6)
- removed the U4 at (-2.51, 132.0)
- removed the U4 at (53.5, 89.4)
- removed the U4 at (-2.51, 89.4)
- removed the U4 at (53.5, 46.8)
- added C1: 10nF, IMRANS_LIBRARY:C_Disc_D3.0mm_W1.6mm_P2.50mm, F.Cu at (56.6, 44.4)
- added C1: 10nF, IMRANS_LIBRARY:C_Disc_D3.0mm_W1.6mm_P2.50mm, F.Cu at (248.6, 44.4)
- added C1: 10nF, IMRANS_LIBRARY:C_Disc_D3.0mm_W1.6mm_P2.50mm, F.Cu at (184.6, 144.3)
- added C1: 10nF, IMRANS_LIBRARY:C_Disc_D3.0mm_W1.6mm_P2.50mm, F.Cu at (56.6, 111.0)
- added C1: 10nF, IMRANS_LIBRARY:C_Disc_D3.0mm_W1.6mm_P2.50mm, F.Cu at (120.6, 44.4)
- added C1: 10nF, IMRANS_LIBRARY:C_Disc_D3.0mm_W1.6mm_P2.50mm, F.Cu at (248.6, 144.3)
- added C1: 10nF, IMRANS_LIBRARY:C_Disc_D3.0mm_W1.6mm_P2.50mm, F.Cu at (120.6, 77.7)
- added C1: 10nF, IMRANS_LIBRARY:C_Disc_D3.0mm_W1.6mm_P2.50mm, F.Cu at (184.6, 111.0)
- added C1: 10nF, IMRANS_LIBRARY:C_Disc_D3.0mm_W1.6mm_P2.50mm, F.Cu at (120.6, 144.3)
- added C1: 10nF, IMRANS_LIBRARY:C_Disc_D3.0mm_W1.6mm_P2.50mm, F.Cu at (120.6, 111.0)
- added C1: 10nF, IMRANS_LIBRARY:C_Disc_D3.0mm_W1.6mm_P2.50mm, F.Cu at (56.6, 144.3)
- added C1: 10nF, IMRANS_LIBRARY:C_Disc_D3.0mm_W1.6mm_P2.50mm, F.Cu at (248.6, 111.0)
- added C1: 10nF, IMRANS_LIBRARY:C_Disc_D3.0mm_W1.6mm_P2.50mm, F.Cu at (248.6, 77.7)
- added C1: 10nF, IMRANS_LIBRARY:C_Disc_D3.0mm_W1.6mm_P2.50mm, F.Cu at (184.6, 77.7)
- added C1: 10nF, IMRANS_LIBRARY:C_Disc_D3.0mm_W1.6mm_P2.50mm, F.Cu at (56.6, 77.7)
- added C1: 10nF, IMRANS_LIBRARY:C_Disc_D3.0mm_W1.6mm_P2.50mm, F.Cu at (184.6, 44.4)
- added C2: 100nF, IMRANS_LIBRARY:C_Disc_D3.0mm_W1.6mm_P2.50mm, F.Cu at (30.2, 149.3)
- added C2: 100nF, IMRANS_LIBRARY:C_Disc_D3.0mm_W1.6mm_P2.50mm, F.Cu at (158.2, 82.7)
- added C2: 100nF, IMRANS_LIBRARY:C_Disc_D3.0mm_W1.6mm_P2.50mm, F.Cu at (158.2, 149.3)
- added C2: 100nF, IMRANS_LIBRARY:C_Disc_D3.0mm_W1.6mm_P2.50mm, F.Cu at (158.2, 116.0)
- added C2: 100nF, IMRANS_LIBRARY:C_Disc_D3.0mm_W1.6mm_P2.50mm, F.Cu at (30.2, 116.0)
- added C2: 100nF, IMRANS_LIBRARY:C_Disc_D3.0mm_W1.6mm_P2.50mm, F.Cu at (30.2, 49.4)
- added C2: 100nF, IMRANS_LIBRARY:C_Disc_D3.0mm_W1.6mm_P2.50mm, F.Cu at (222.2, 116.0)
- added C2: 100nF, IMRANS_LIBRARY:C_Disc_D3.0mm_W1.6mm_P2.50mm, F.Cu at (222.2, 149.3)
- added C2: 100nF, IMRANS_LIBRARY:C_Disc_D3.0mm_W1.6mm_P2.50mm, F.Cu at (94.2, 82.7)
- added C2: 100nF, IMRANS_LIBRARY:C_Disc_D3.0mm_W1.6mm_P2.50mm, F.Cu at (94.2, 116.0)
- added C2: 100nF, IMRANS_LIBRARY:C_Disc_D3.0mm_W1.6mm_P2.50mm, F.Cu at (30.2, 82.7)
- added C2: 100nF, IMRANS_LIBRARY:C_Disc_D3.0mm_W1.6mm_P2.50mm, F.Cu at (222.2, 49.4)
- added C2: 100nF, IMRANS_LIBRARY:C_Disc_D3.0mm_W1.6mm_P2.50mm, F.Cu at (94.2, 49.4)
- added C2: 100nF, IMRANS_LIBRARY:C_Disc_D3.0mm_W1.6mm_P2.50mm, F.Cu at (158.2, 49.4)
- added C2: 100nF, IMRANS_LIBRARY:C_Disc_D3.0mm_W1.6mm_P2.50mm, F.Cu at (94.2, 149.3)
- added C2: 100nF, IMRANS_LIBRARY:C_Disc_D3.0mm_W1.6mm_P2.50mm, F.Cu at (222.2, 82.7)
- added D1: 1N4007, IMRANS_LIBRARY:R_Axial_DIN0207_L6.3mm_D2.5mm_P10.16mm_Horizontal_2, F.Cu at (152.7, 67.9)
- added D1: 1N4007, IMRANS_LIBRARY:R_Axial_DIN0207_L6.3mm_D2.5mm_P10.16mm_Horizontal_2, F.Cu at (24.7, 101.2)
- added D1: 1N4007, IMRANS_LIBRARY:R_Axial_DIN0207_L6.3mm_D2.5mm_P10.16mm_Horizontal_2, F.Cu at (24.7, 34.6)
- added D1: 1N4007, IMRANS_LIBRARY:R_Axial_DIN0207_L6.3mm_D2.5mm_P10.16mm_Horizontal_2, F.Cu at (216.7, 134.5)
- added D1: 1N4007, IMRANS_LIBRARY:R_Axial_DIN0207_L6.3mm_D2.5mm_P10.16mm_Horizontal_2, F.Cu at (24.7, 67.9)
- added D1: 1N4007, IMRANS_LIBRARY:R_Axial_DIN0207_L6.3mm_D2.5mm_P10.16mm_Horizontal_2, F.Cu at (152.7, 34.6)
- added D1: 1N4007, IMRANS_LIBRARY:R_Axial_DIN0207_L6.3mm_D2.5mm_P10.16mm_Horizontal_2, F.Cu at (216.7, 67.9)
- added D1: 1N4007, IMRANS_LIBRARY:R_Axial_DIN0207_L6.3mm_D2.5mm_P10.16mm_Horizontal_2, F.Cu at (24.7, 134.5)
- added D1: 1N4007, IMRANS_LIBRARY:R_Axial_DIN0207_L6.3mm_D2.5mm_P10.16mm_Horizontal_2, F.Cu at (88.7, 134.5)
- added D1: 1N4007, IMRANS_LIBRARY:R_Axial_DIN0207_L6.3mm_D2.5mm_P10.16mm_Horizontal_2, F.Cu at (152.7, 101.2)
- added D1: 1N4007, IMRANS_LIBRARY:R_Axial_DIN0207_L6.3mm_D2.5mm_P10.16mm_Horizontal_2, F.Cu at (88.7, 34.6)
- added D1: 1N4007, IMRANS_LIBRARY:R_Axial_DIN0207_L6.3mm_D2.5mm_P10.16mm_Horizontal_2, F.Cu at (152.7, 134.5)
- added D1: 1N4007, IMRANS_LIBRARY:R_Axial_DIN0207_L6.3mm_D2.5mm_P10.16mm_Horizontal_2, F.Cu at (88.7, 67.9)
- added D1: 1N4007, IMRANS_LIBRARY:R_Axial_DIN0207_L6.3mm_D2.5mm_P10.16mm_Horizontal_2, F.Cu at (88.7, 101.2)
- added D1: 1N4007, IMRANS_LIBRARY:R_Axial_DIN0207_L6.3mm_D2.5mm_P10.16mm_Horizontal_2, F.Cu at (216.7, 34.6)
- added D1: 1N4007, IMRANS_LIBRARY:R_Axial_DIN0207_L6.3mm_D2.5mm_P10.16mm_Horizontal_2, F.Cu at (216.7, 101.2)
- added J1: BOT POWER, TerminalBlock_Phoenix:TerminalBlock_Phoenix_MKDS-1,5-2-5.08_1x02_P5.08mm_Horizontal, F.Cu at (55.1, 27.1)
- added J1: BOT POWER, TerminalBlock_Phoenix:TerminalBlock_Phoenix_MKDS-1,5-2-5.08_1x02_P5.08mm_Horizontal, F.Cu at (183.1, 93.7)
- added J1: BOT POWER, TerminalBlock_Phoenix:TerminalBlock_Phoenix_MKDS-1,5-2-5.08_1x02_P5.08mm_Horizontal, F.Cu at (119.1, 27.1)
- added J1: BOT POWER, TerminalBlock_Phoenix:TerminalBlock_Phoenix_MKDS-1,5-2-5.08_1x02_P5.08mm_Horizontal, F.Cu at (55.1, 127.0)
- added J1: BOT POWER, TerminalBlock_Phoenix:TerminalBlock_Phoenix_MKDS-1,5-2-5.08_1x02_P5.08mm_Horizontal, F.Cu at (247.1, 27.1)
- added J1: BOT POWER, TerminalBlock_Phoenix:TerminalBlock_Phoenix_MKDS-1,5-2-5.08_1x02_P5.08mm_Horizontal, F.Cu at (119.1, 93.7)
- added J1: BOT POWER, TerminalBlock_Phoenix:TerminalBlock_Phoenix_MKDS-1,5-2-5.08_1x02_P5.08mm_Horizontal, F.Cu at (183.1, 27.1)
- added J1: BOT POWER, TerminalBlock_Phoenix:TerminalBlock_Phoenix_MKDS-1,5-2-5.08_1x02_P5.08mm_Horizontal, F.Cu at (119.1, 127.0)
- added J1: BOT POWER, TerminalBlock_Phoenix:TerminalBlock_Phoenix_MKDS-1,5-2-5.08_1x02_P5.08mm_Horizontal, F.Cu at (183.1, 127.0)
- added J1: BOT POWER, TerminalBlock_Phoenix:TerminalBlock_Phoenix_MKDS-1,5-2-5.08_1x02_P5.08mm_Horizontal, F.Cu at (119.1, 60.4)
- added J1: BOT POWER, TerminalBlock_Phoenix:TerminalBlock_Phoenix_MKDS-1,5-2-5.08_1x02_P5.08mm_Horizontal, F.Cu at (55.1, 93.7)
- added J1: BOT POWER, TerminalBlock_Phoenix:TerminalBlock_Phoenix_MKDS-1,5-2-5.08_1x02_P5.08mm_Horizontal, F.Cu at (183.1, 60.4)
- added J1: BOT POWER, TerminalBlock_Phoenix:TerminalBlock_Phoenix_MKDS-1,5-2-5.08_1x02_P5.08mm_Horizontal, F.Cu at (247.1, 93.7)
- added J1: BOT POWER, TerminalBlock_Phoenix:TerminalBlock_Phoenix_MKDS-1,5-2-5.08_1x02_P5.08mm_Horizontal, F.Cu at (247.1, 127.0)
- added J1: BOT POWER, TerminalBlock_Phoenix:TerminalBlock_Phoenix_MKDS-1,5-2-5.08_1x02_P5.08mm_Horizontal, F.Cu at (55.1, 60.4)
- added J1: BOT POWER, TerminalBlock_Phoenix:TerminalBlock_Phoenix_MKDS-1,5-2-5.08_1x02_P5.08mm_Horizontal, F.Cu at (247.1, 60.4)
- added J2: POWER IN, TerminalBlock_Phoenix:TerminalBlock_Phoenix_MKDS-1,5-2-5.08_1x02_P5.08mm_Horizontal, F.Cu at (78.1, 60.5)
- added J2: POWER IN, TerminalBlock_Phoenix:TerminalBlock_Phoenix_MKDS-1,5-2-5.08_1x02_P5.08mm_Horizontal, F.Cu at (78.1, 127.1)
- added J2: POWER IN, TerminalBlock_Phoenix:TerminalBlock_Phoenix_MKDS-1,5-2-5.08_1x02_P5.08mm_Horizontal, F.Cu at (270.1, 93.8)
- added J2: POWER IN, TerminalBlock_Phoenix:TerminalBlock_Phoenix_MKDS-1,5-2-5.08_1x02_P5.08mm_Horizontal, F.Cu at (142.1, 127.1)
- added J2: POWER IN, TerminalBlock_Phoenix:TerminalBlock_Phoenix_MKDS-1,5-2-5.08_1x02_P5.08mm_Horizontal, F.Cu at (142.1, 27.2)
- added J2: POWER IN, TerminalBlock_Phoenix:TerminalBlock_Phoenix_MKDS-1,5-2-5.08_1x02_P5.08mm_Horizontal, F.Cu at (270.1, 60.5)
- added J2: POWER IN, TerminalBlock_Phoenix:TerminalBlock_Phoenix_MKDS-1,5-2-5.08_1x02_P5.08mm_Horizontal, F.Cu at (78.1, 27.2)
- added J2: POWER IN, TerminalBlock_Phoenix:TerminalBlock_Phoenix_MKDS-1,5-2-5.08_1x02_P5.08mm_Horizontal, F.Cu at (206.1, 127.1)
- added J2: POWER IN, TerminalBlock_Phoenix:TerminalBlock_Phoenix_MKDS-1,5-2-5.08_1x02_P5.08mm_Horizontal, F.Cu at (206.1, 93.8)
- added J2: POWER IN, TerminalBlock_Phoenix:TerminalBlock_Phoenix_MKDS-1,5-2-5.08_1x02_P5.08mm_Horizontal, F.Cu at (270.1, 127.1)
- added J2: POWER IN, TerminalBlock_Phoenix:TerminalBlock_Phoenix_MKDS-1,5-2-5.08_1x02_P5.08mm_Horizontal, F.Cu at (142.1, 60.5)
- added J2: POWER IN, TerminalBlock_Phoenix:TerminalBlock_Phoenix_MKDS-1,5-2-5.08_1x02_P5.08mm_Horizontal, F.Cu at (206.1, 27.2)
- added J2: POWER IN, TerminalBlock_Phoenix:TerminalBlock_Phoenix_MKDS-1,5-2-5.08_1x02_P5.08mm_Horizontal, F.Cu at (78.1, 93.8)
- added J2: POWER IN, TerminalBlock_Phoenix:TerminalBlock_Phoenix_MKDS-1,5-2-5.08_1x02_P5.08mm_Horizontal, F.Cu at (270.1, 27.2)
- added J2: POWER IN, TerminalBlock_Phoenix:TerminalBlock_Phoenix_MKDS-1,5-2-5.08_1x02_P5.08mm_Horizontal, F.Cu at (142.1, 93.8)
- added J2: POWER IN, TerminalBlock_Phoenix:TerminalBlock_Phoenix_MKDS-1,5-2-5.08_1x02_P5.08mm_Horizontal, F.Cu at (206.1, 60.5)
- added J3: SHUNT, TerminalBlock_Phoenix:TerminalBlock_Phoenix_MKDS-1,5-2-5.08_1x02_P5.08mm_Horizontal, F.Cu at (66.5, 60.4)
- added J3: SHUNT, TerminalBlock_Phoenix:TerminalBlock_Phoenix_MKDS-1,5-2-5.08_1x02_P5.08mm_Horizontal, F.Cu at (258.5, 127.0)
- added J3: SHUNT, TerminalBlock_Phoenix:TerminalBlock_Phoenix_MKDS-1,5-2-5.08_1x02_P5.08mm_Horizontal, F.Cu at (194.5, 93.7)
- added J3: SHUNT, TerminalBlock_Phoenix:TerminalBlock_Phoenix_MKDS-1,5-2-5.08_1x02_P5.08mm_Horizontal, F.Cu at (66.5, 93.7)
- added J3: SHUNT, TerminalBlock_Phoenix:TerminalBlock_Phoenix_MKDS-1,5-2-5.08_1x02_P5.08mm_Horizontal, F.Cu at (130.5, 60.4)
- added J3: SHUNT, TerminalBlock_Phoenix:TerminalBlock_Phoenix_MKDS-1,5-2-5.08_1x02_P5.08mm_Horizontal, F.Cu at (258.5, 27.1)
- added J3: SHUNT, TerminalBlock_Phoenix:TerminalBlock_Phoenix_MKDS-1,5-2-5.08_1x02_P5.08mm_Horizontal, F.Cu at (194.5, 27.1)
- added J3: SHUNT, TerminalBlock_Phoenix:TerminalBlock_Phoenix_MKDS-1,5-2-5.08_1x02_P5.08mm_Horizontal, F.Cu at (66.5, 27.1)
- added J3: SHUNT, TerminalBlock_Phoenix:TerminalBlock_Phoenix_MKDS-1,5-2-5.08_1x02_P5.08mm_Horizontal, F.Cu at (258.5, 60.4)
- added J3: SHUNT, TerminalBlock_Phoenix:TerminalBlock_Phoenix_MKDS-1,5-2-5.08_1x02_P5.08mm_Horizontal, F.Cu at (66.5, 127.0)
- added J3: SHUNT, TerminalBlock_Phoenix:TerminalBlock_Phoenix_MKDS-1,5-2-5.08_1x02_P5.08mm_Horizontal, F.Cu at (194.5, 60.4)
- added J3: SHUNT, TerminalBlock_Phoenix:TerminalBlock_Phoenix_MKDS-1,5-2-5.08_1x02_P5.08mm_Horizontal, F.Cu at (130.5, 27.1)
- added J3: SHUNT, TerminalBlock_Phoenix:TerminalBlock_Phoenix_MKDS-1,5-2-5.08_1x02_P5.08mm_Horizontal, F.Cu at (130.5, 127.0)
- added J3: SHUNT, TerminalBlock_Phoenix:TerminalBlock_Phoenix_MKDS-1,5-2-5.08_1x02_P5.08mm_Horizontal, F.Cu at (130.5, 93.7)
- added J3: SHUNT, TerminalBlock_Phoenix:TerminalBlock_Phoenix_MKDS-1,5-2-5.08_1x02_P5.08mm_Horizontal, F.Cu at (194.5, 127.0)
- added J3: SHUNT, TerminalBlock_Phoenix:TerminalBlock_Phoenix_MKDS-1,5-2-5.08_1x02_P5.08mm_Horizontal, F.Cu at (258.5, 93.7)
- added J4: COIL OUT, TerminalBlock_Phoenix:TerminalBlock_Phoenix_MKDS-1,5-2-5.08_1x02_P5.08mm_Horizontal, F.Cu at (160.4, 27.1)
- added J4: COIL OUT, TerminalBlock_Phoenix:TerminalBlock_Phoenix_MKDS-1,5-2-5.08_1x02_P5.08mm_Horizontal, F.Cu at (32.4, 60.4)
- added J4: COIL OUT, TerminalBlock_Phoenix:TerminalBlock_Phoenix_MKDS-1,5-2-5.08_1x02_P5.08mm_Horizontal, F.Cu at (96.4, 127.0)
- added J4: COIL OUT, TerminalBlock_Phoenix:TerminalBlock_Phoenix_MKDS-1,5-2-5.08_1x02_P5.08mm_Horizontal, F.Cu at (32.4, 127.0)
- added J4: COIL OUT, TerminalBlock_Phoenix:TerminalBlock_Phoenix_MKDS-1,5-2-5.08_1x02_P5.08mm_Horizontal, F.Cu at (160.4, 60.4)
- added J4: COIL OUT, TerminalBlock_Phoenix:TerminalBlock_Phoenix_MKDS-1,5-2-5.08_1x02_P5.08mm_Horizontal, F.Cu at (224.4, 93.7)
- added J4: COIL OUT, TerminalBlock_Phoenix:TerminalBlock_Phoenix_MKDS-1,5-2-5.08_1x02_P5.08mm_Horizontal, F.Cu at (160.4, 93.7)
- added J4: COIL OUT, TerminalBlock_Phoenix:TerminalBlock_Phoenix_MKDS-1,5-2-5.08_1x02_P5.08mm_Horizontal, F.Cu at (96.4, 93.7)
- added J4: COIL OUT, TerminalBlock_Phoenix:TerminalBlock_Phoenix_MKDS-1,5-2-5.08_1x02_P5.08mm_Horizontal, F.Cu at (224.4, 60.4)
- added J4: COIL OUT, TerminalBlock_Phoenix:TerminalBlock_Phoenix_MKDS-1,5-2-5.08_1x02_P5.08mm_Horizontal, F.Cu at (96.4, 27.1)
- added J4: COIL OUT, TerminalBlock_Phoenix:TerminalBlock_Phoenix_MKDS-1,5-2-5.08_1x02_P5.08mm_Horizontal, F.Cu at (32.4, 93.7)
- added J4: COIL OUT, TerminalBlock_Phoenix:TerminalBlock_Phoenix_MKDS-1,5-2-5.08_1x02_P5.08mm_Horizontal, F.Cu at (224.4, 27.1)
- added J4: COIL OUT, TerminalBlock_Phoenix:TerminalBlock_Phoenix_MKDS-1,5-2-5.08_1x02_P5.08mm_Horizontal, F.Cu at (96.4, 60.4)
- added J4: COIL OUT, TerminalBlock_Phoenix:TerminalBlock_Phoenix_MKDS-1,5-2-5.08_1x02_P5.08mm_Horizontal, F.Cu at (224.4, 127.0)
- added J4: COIL OUT, TerminalBlock_Phoenix:TerminalBlock_Phoenix_MKDS-1,5-2-5.08_1x02_P5.08mm_Horizontal, F.Cu at (32.4, 27.1)
- added J4: COIL OUT, TerminalBlock_Phoenix:TerminalBlock_Phoenix_MKDS-1,5-2-5.08_1x02_P5.08mm_Horizontal, F.Cu at (160.4, 127.0)
- added J5: COIL POWER IN, TerminalBlock_Phoenix:TerminalBlock_Phoenix_MKDS-1,5-2-5.08_1x02_P5.08mm_Horizontal, F.Cu at (235.7, 27.1)
- added J5: COIL POWER IN, TerminalBlock_Phoenix:TerminalBlock_Phoenix_MKDS-1,5-2-5.08_1x02_P5.08mm_Horizontal, F.Cu at (107.7, 27.1)
- added J5: COIL POWER IN, TerminalBlock_Phoenix:TerminalBlock_Phoenix_MKDS-1,5-2-5.08_1x02_P5.08mm_Horizontal, F.Cu at (43.7, 93.7)
- added J5: COIL POWER IN, TerminalBlock_Phoenix:TerminalBlock_Phoenix_MKDS-1,5-2-5.08_1x02_P5.08mm_Horizontal, F.Cu at (107.7, 60.4)
- added J5: COIL POWER IN, TerminalBlock_Phoenix:TerminalBlock_Phoenix_MKDS-1,5-2-5.08_1x02_P5.08mm_Horizontal, F.Cu at (235.7, 60.4)
- added J5: COIL POWER IN, TerminalBlock_Phoenix:TerminalBlock_Phoenix_MKDS-1,5-2-5.08_1x02_P5.08mm_Horizontal, F.Cu at (43.7, 127.0)
- added J5: COIL POWER IN, TerminalBlock_Phoenix:TerminalBlock_Phoenix_MKDS-1,5-2-5.08_1x02_P5.08mm_Horizontal, F.Cu at (171.7, 127.0)
- added J5: COIL POWER IN, TerminalBlock_Phoenix:TerminalBlock_Phoenix_MKDS-1,5-2-5.08_1x02_P5.08mm_Horizontal, F.Cu at (107.7, 93.7)
- added J5: COIL POWER IN, TerminalBlock_Phoenix:TerminalBlock_Phoenix_MKDS-1,5-2-5.08_1x02_P5.08mm_Horizontal, F.Cu at (171.7, 27.1)
- added J5: COIL POWER IN, TerminalBlock_Phoenix:TerminalBlock_Phoenix_MKDS-1,5-2-5.08_1x02_P5.08mm_Horizontal, F.Cu at (107.7, 127.0)
- added J5: COIL POWER IN, TerminalBlock_Phoenix:TerminalBlock_Phoenix_MKDS-1,5-2-5.08_1x02_P5.08mm_Horizontal, F.Cu at (43.7, 27.1)
- added J5: COIL POWER IN, TerminalBlock_Phoenix:TerminalBlock_Phoenix_MKDS-1,5-2-5.08_1x02_P5.08mm_Horizontal, F.Cu at (171.7, 60.4)
- added J5: COIL POWER IN, TerminalBlock_Phoenix:TerminalBlock_Phoenix_MKDS-1,5-2-5.08_1x02_P5.08mm_Horizontal, F.Cu at (43.7, 60.4)
- added J5: COIL POWER IN, TerminalBlock_Phoenix:TerminalBlock_Phoenix_MKDS-1,5-2-5.08_1x02_P5.08mm_Horizontal, F.Cu at (235.7, 127.0)
- added J5: COIL POWER IN, TerminalBlock_Phoenix:TerminalBlock_Phoenix_MKDS-1,5-2-5.08_1x02_P5.08mm_Horizontal, F.Cu at (235.7, 93.7)
- added J5: COIL POWER IN, TerminalBlock_Phoenix:TerminalBlock_Phoenix_MKDS-1,5-2-5.08_1x02_P5.08mm_Horizontal, F.Cu at (171.7, 93.7)
- added Q1: IRF3205, IMRANS_LIBRARY:TO-220-3_Vertical, F.Cu at (34.6, 111.2)
- added Q1: IRF3205, IMRANS_LIBRARY:TO-220-3_Vertical, F.Cu at (226.6, 111.2)
- added Q1: IRF3205, IMRANS_LIBRARY:TO-220-3_Vertical, F.Cu at (34.6, 144.5)
- added Q1: IRF3205, IMRANS_LIBRARY:TO-220-3_Vertical, F.Cu at (34.6, 77.9)
- added Q1: IRF3205, IMRANS_LIBRARY:TO-220-3_Vertical, F.Cu at (226.6, 77.9)
- added Q1: IRF3205, IMRANS_LIBRARY:TO-220-3_Vertical, F.Cu at (162.6, 111.2)
- added Q1: IRF3205, IMRANS_LIBRARY:TO-220-3_Vertical, F.Cu at (98.6, 111.2)
- added Q1: IRF3205, IMRANS_LIBRARY:TO-220-3_Vertical, F.Cu at (98.6, 44.6)
- added Q1: IRF3205, IMRANS_LIBRARY:TO-220-3_Vertical, F.Cu at (162.6, 44.6)
- added Q1: IRF3205, IMRANS_LIBRARY:TO-220-3_Vertical, F.Cu at (98.6, 77.9)
- added Q1: IRF3205, IMRANS_LIBRARY:TO-220-3_Vertical, F.Cu at (162.6, 77.9)
- added Q1: IRF3205, IMRANS_LIBRARY:TO-220-3_Vertical, F.Cu at (98.6, 144.5)
- added Q1: IRF3205, IMRANS_LIBRARY:TO-220-3_Vertical, F.Cu at (226.6, 44.6)
- added Q1: IRF3205, IMRANS_LIBRARY:TO-220-3_Vertical, F.Cu at (226.6, 144.5)
- added Q1: IRF3205, IMRANS_LIBRARY:TO-220-3_Vertical, F.Cu at (34.6, 44.6)
- added Q1: IRF3205, IMRANS_LIBRARY:TO-220-3_Vertical, F.Cu at (162.6, 144.5)
- added R1: 10K, IMRANS_LIBRARY:R_Axial_DIN0207_L6.3mm_D2.5mm_P10.16mm_Horizontal_2, F.Cu at (75.1, 135.7)
- added R1: 10K, IMRANS_LIBRARY:R_Axial_DIN0207_L6.3mm_D2.5mm_P10.16mm_Horizontal_2, F.Cu at (139.1, 135.7)
- added R1: 10K, IMRANS_LIBRARY:R_Axial_DIN0207_L6.3mm_D2.5mm_P10.16mm_Horizontal_2, F.Cu at (139.1, 69.1)
- added R1: 10K, IMRANS_LIBRARY:R_Axial_DIN0207_L6.3mm_D2.5mm_P10.16mm_Horizontal_2, F.Cu at (139.1, 35.8)
- added R1: 10K, IMRANS_LIBRARY:R_Axial_DIN0207_L6.3mm_D2.5mm_P10.16mm_Horizontal_2, F.Cu at (267.1, 69.1)
- added R1: 10K, IMRANS_LIBRARY:R_Axial_DIN0207_L6.3mm_D2.5mm_P10.16mm_Horizontal_2, F.Cu at (139.1, 102.4)
- added R1: 10K, IMRANS_LIBRARY:R_Axial_DIN0207_L6.3mm_D2.5mm_P10.16mm_Horizontal_2, F.Cu at (75.1, 102.4)
- added R1: 10K, IMRANS_LIBRARY:R_Axial_DIN0207_L6.3mm_D2.5mm_P10.16mm_Horizontal_2, F.Cu at (267.1, 135.7)
- added R1: 10K, IMRANS_LIBRARY:R_Axial_DIN0207_L6.3mm_D2.5mm_P10.16mm_Horizontal_2, F.Cu at (203.1, 35.8)
- added R1: 10K, IMRANS_LIBRARY:R_Axial_DIN0207_L6.3mm_D2.5mm_P10.16mm_Horizontal_2, F.Cu at (203.1, 135.7)
- added R1: 10K, IMRANS_LIBRARY:R_Axial_DIN0207_L6.3mm_D2.5mm_P10.16mm_Horizontal_2, F.Cu at (203.1, 69.1)
- added R1: 10K, IMRANS_LIBRARY:R_Axial_DIN0207_L6.3mm_D2.5mm_P10.16mm_Horizontal_2, F.Cu at (267.1, 102.4)
- added R1: 10K, IMRANS_LIBRARY:R_Axial_DIN0207_L6.3mm_D2.5mm_P10.16mm_Horizontal_2, F.Cu at (203.1, 102.4)
- added R1: 10K, IMRANS_LIBRARY:R_Axial_DIN0207_L6.3mm_D2.5mm_P10.16mm_Horizontal_2, F.Cu at (75.1, 35.8)
- added R1: 10K, IMRANS_LIBRARY:R_Axial_DIN0207_L6.3mm_D2.5mm_P10.16mm_Horizontal_2, F.Cu at (267.1, 35.8)
- added R1: 10K, IMRANS_LIBRARY:R_Axial_DIN0207_L6.3mm_D2.5mm_P10.16mm_Horizontal_2, F.Cu at (75.1, 69.1)
- added R2: 10K, IMRANS_LIBRARY:R_Axial_DIN0207_L6.3mm_D2.5mm_P10.16mm_Horizontal_2, F.Cu at (199.8, 147.8)
- added R2: 10K, IMRANS_LIBRARY:R_Axial_DIN0207_L6.3mm_D2.5mm_P10.16mm_Horizontal_2, F.Cu at (199.8, 114.5)
- added R2: 10K, IMRANS_LIBRARY:R_Axial_DIN0207_L6.3mm_D2.5mm_P10.16mm_Horizontal_2, F.Cu at (71.8, 47.9)
- added R2: 10K, IMRANS_LIBRARY:R_Axial_DIN0207_L6.3mm_D2.5mm_P10.16mm_Horizontal_2, F.Cu at (263.8, 47.9)
- added R2: 10K, IMRANS_LIBRARY:R_Axial_DIN0207_L6.3mm_D2.5mm_P10.16mm_Horizontal_2, F.Cu at (199.8, 81.2)
- added R2: 10K, IMRANS_LIBRARY:R_Axial_DIN0207_L6.3mm_D2.5mm_P10.16mm_Horizontal_2, F.Cu at (263.8, 81.2)
- added R2: 10K, IMRANS_LIBRARY:R_Axial_DIN0207_L6.3mm_D2.5mm_P10.16mm_Horizontal_2, F.Cu at (71.8, 147.8)
- added R2: 10K, IMRANS_LIBRARY:R_Axial_DIN0207_L6.3mm_D2.5mm_P10.16mm_Horizontal_2, F.Cu at (135.8, 81.2)
- added R2: 10K, IMRANS_LIBRARY:R_Axial_DIN0207_L6.3mm_D2.5mm_P10.16mm_Horizontal_2, F.Cu at (135.8, 147.8)
- added R2: 10K, IMRANS_LIBRARY:R_Axial_DIN0207_L6.3mm_D2.5mm_P10.16mm_Horizontal_2, F.Cu at (199.8, 47.9)
- added R2: 10K, IMRANS_LIBRARY:R_Axial_DIN0207_L6.3mm_D2.5mm_P10.16mm_Horizontal_2, F.Cu at (263.8, 147.8)
- added R2: 10K, IMRANS_LIBRARY:R_Axial_DIN0207_L6.3mm_D2.5mm_P10.16mm_Horizontal_2, F.Cu at (71.8, 114.5)
- added R2: 10K, IMRANS_LIBRARY:R_Axial_DIN0207_L6.3mm_D2.5mm_P10.16mm_Horizontal_2, F.Cu at (135.8, 114.5)
- added R2: 10K, IMRANS_LIBRARY:R_Axial_DIN0207_L6.3mm_D2.5mm_P10.16mm_Horizontal_2, F.Cu at (263.8, 114.5)
- added R2: 10K, IMRANS_LIBRARY:R_Axial_DIN0207_L6.3mm_D2.5mm_P10.16mm_Horizontal_2, F.Cu at (71.8, 81.2)
- added R2: 10K, IMRANS_LIBRARY:R_Axial_DIN0207_L6.3mm_D2.5mm_P10.16mm_Horizontal_2, F.Cu at (135.8, 47.9)
- added R3: 6.8K, IMRANS_LIBRARY:R_Axial_DIN0207_L6.3mm_D2.5mm_P10.16mm_Horizontal_2, F.Cu at (105.7, 114.0)
- added R3: 6.8K, IMRANS_LIBRARY:R_Axial_DIN0207_L6.3mm_D2.5mm_P10.16mm_Horizontal_2, F.Cu at (169.7, 80.7)
- added R3: 6.8K, IMRANS_LIBRARY:R_Axial_DIN0207_L6.3mm_D2.5mm_P10.16mm_Horizontal_2, F.Cu at (169.7, 147.3)
- added R3: 6.8K, IMRANS_LIBRARY:R_Axial_DIN0207_L6.3mm_D2.5mm_P10.16mm_Horizontal_2, F.Cu at (169.7, 47.4)
- added R3: 6.8K, IMRANS_LIBRARY:R_Axial_DIN0207_L6.3mm_D2.5mm_P10.16mm_Horizontal_2, F.Cu at (41.7, 147.3)
- added R3: 6.8K, IMRANS_LIBRARY:R_Axial_DIN0207_L6.3mm_D2.5mm_P10.16mm_Horizontal_2, F.Cu at (41.7, 80.7)
- added R3: 6.8K, IMRANS_LIBRARY:R_Axial_DIN0207_L6.3mm_D2.5mm_P10.16mm_Horizontal_2, F.Cu at (233.7, 114.0)
- added R3: 6.8K, IMRANS_LIBRARY:R_Axial_DIN0207_L6.3mm_D2.5mm_P10.16mm_Horizontal_2, F.Cu at (233.7, 47.4)
- added R3: 6.8K, IMRANS_LIBRARY:R_Axial_DIN0207_L6.3mm_D2.5mm_P10.16mm_Horizontal_2, F.Cu at (41.7, 114.0)
- added R3: 6.8K, IMRANS_LIBRARY:R_Axial_DIN0207_L6.3mm_D2.5mm_P10.16mm_Horizontal_2, F.Cu at (105.7, 47.4)
- added R3: 6.8K, IMRANS_LIBRARY:R_Axial_DIN0207_L6.3mm_D2.5mm_P10.16mm_Horizontal_2, F.Cu at (169.7, 114.0)
- added R3: 6.8K, IMRANS_LIBRARY:R_Axial_DIN0207_L6.3mm_D2.5mm_P10.16mm_Horizontal_2, F.Cu at (233.7, 147.3)
- added R3: 6.8K, IMRANS_LIBRARY:R_Axial_DIN0207_L6.3mm_D2.5mm_P10.16mm_Horizontal_2, F.Cu at (41.7, 47.4)
- added R3: 6.8K, IMRANS_LIBRARY:R_Axial_DIN0207_L6.3mm_D2.5mm_P10.16mm_Horizontal_2, F.Cu at (105.7, 80.7)
- added R3: 6.8K, IMRANS_LIBRARY:R_Axial_DIN0207_L6.3mm_D2.5mm_P10.16mm_Horizontal_2, F.Cu at (233.7, 80.7)
- added R3: 6.8K, IMRANS_LIBRARY:R_Axial_DIN0207_L6.3mm_D2.5mm_P10.16mm_Horizontal_2, F.Cu at (105.7, 147.3)
- added R4: 47R, IMRANS_LIBRARY:R_Axial_DIN0207_L6.3mm_D2.5mm_P10.16mm_Horizontal_2, F.Cu at (166.2, 116.5)
- added R4: 47R, IMRANS_LIBRARY:R_Axial_DIN0207_L6.3mm_D2.5mm_P10.16mm_Horizontal_2, F.Cu at (102.2, 49.9)
- added R4: 47R, IMRANS_LIBRARY:R_Axial_DIN0207_L6.3mm_D2.5mm_P10.16mm_Horizontal_2, F.Cu at (230.2, 49.9)
- added R4: 47R, IMRANS_LIBRARY:R_Axial_DIN0207_L6.3mm_D2.5mm_P10.16mm_Horizontal_2, F.Cu at (166.2, 149.8)
- added R4: 47R, IMRANS_LIBRARY:R_Axial_DIN0207_L6.3mm_D2.5mm_P10.16mm_Horizontal_2, F.Cu at (38.2, 49.9)
- added R4: 47R, IMRANS_LIBRARY:R_Axial_DIN0207_L6.3mm_D2.5mm_P10.16mm_Horizontal_2, F.Cu at (230.2, 116.5)
- added R4: 47R, IMRANS_LIBRARY:R_Axial_DIN0207_L6.3mm_D2.5mm_P10.16mm_Horizontal_2, F.Cu at (38.2, 116.5)
- added R4: 47R, IMRANS_LIBRARY:R_Axial_DIN0207_L6.3mm_D2.5mm_P10.16mm_Horizontal_2, F.Cu at (38.2, 83.2)
- added R4: 47R, IMRANS_LIBRARY:R_Axial_DIN0207_L6.3mm_D2.5mm_P10.16mm_Horizontal_2, F.Cu at (166.2, 83.2)
- added R4: 47R, IMRANS_LIBRARY:R_Axial_DIN0207_L6.3mm_D2.5mm_P10.16mm_Horizontal_2, F.Cu at (38.2, 149.8)
- added R4: 47R, IMRANS_LIBRARY:R_Axial_DIN0207_L6.3mm_D2.5mm_P10.16mm_Horizontal_2, F.Cu at (166.2, 49.9)
- added R4: 47R, IMRANS_LIBRARY:R_Axial_DIN0207_L6.3mm_D2.5mm_P10.16mm_Horizontal_2, F.Cu at (102.2, 149.8)
- added R4: 47R, IMRANS_LIBRARY:R_Axial_DIN0207_L6.3mm_D2.5mm_P10.16mm_Horizontal_2, F.Cu at (102.2, 116.5)
- added R4: 47R, IMRANS_LIBRARY:R_Axial_DIN0207_L6.3mm_D2.5mm_P10.16mm_Horizontal_2, F.Cu at (230.2, 83.2)
- added R4: 47R, IMRANS_LIBRARY:R_Axial_DIN0207_L6.3mm_D2.5mm_P10.16mm_Horizontal_2, F.Cu at (230.2, 149.8)
- added R4: 47R, IMRANS_LIBRARY:R_Axial_DIN0207_L6.3mm_D2.5mm_P10.16mm_Horizontal_2, F.Cu at (102.2, 83.2)
- added R5: 1K, IMRANS_LIBRARY:R_Axial_DIN0207_L6.3mm_D2.5mm_P10.16mm_Horizontal_2, F.Cu at (246.8, 101.9)
- added R5: 1K, IMRANS_LIBRARY:R_Axial_DIN0207_L6.3mm_D2.5mm_P10.16mm_Horizontal_2, F.Cu at (246.8, 135.2)
- added R5: 1K, IMRANS_LIBRARY:R_Axial_DIN0207_L6.3mm_D2.5mm_P10.16mm_Horizontal_2, F.Cu at (182.8, 135.2)
- added R5: 1K, IMRANS_LIBRARY:R_Axial_DIN0207_L6.3mm_D2.5mm_P10.16mm_Horizontal_2, F.Cu at (182.8, 35.3)
- added R5: 1K, IMRANS_LIBRARY:R_Axial_DIN0207_L6.3mm_D2.5mm_P10.16mm_Horizontal_2, F.Cu at (118.8, 68.6)
- added R5: 1K, IMRANS_LIBRARY:R_Axial_DIN0207_L6.3mm_D2.5mm_P10.16mm_Horizontal_2, F.Cu at (54.8, 68.6)
- added R5: 1K, IMRANS_LIBRARY:R_Axial_DIN0207_L6.3mm_D2.5mm_P10.16mm_Horizontal_2, F.Cu at (118.8, 35.3)
- added R5: 1K, IMRANS_LIBRARY:R_Axial_DIN0207_L6.3mm_D2.5mm_P10.16mm_Horizontal_2, F.Cu at (118.8, 101.9)
- added R5: 1K, IMRANS_LIBRARY:R_Axial_DIN0207_L6.3mm_D2.5mm_P10.16mm_Horizontal_2, F.Cu at (182.8, 68.6)
- added R5: 1K, IMRANS_LIBRARY:R_Axial_DIN0207_L6.3mm_D2.5mm_P10.16mm_Horizontal_2, F.Cu at (182.8, 101.9)
- added R5: 1K, IMRANS_LIBRARY:R_Axial_DIN0207_L6.3mm_D2.5mm_P10.16mm_Horizontal_2, F.Cu at (246.8, 68.6)
- added R5: 1K, IMRANS_LIBRARY:R_Axial_DIN0207_L6.3mm_D2.5mm_P10.16mm_Horizontal_2, F.Cu at (246.8, 35.3)
- added R5: 1K, IMRANS_LIBRARY:R_Axial_DIN0207_L6.3mm_D2.5mm_P10.16mm_Horizontal_2, F.Cu at (54.8, 135.2)
- added R5: 1K, IMRANS_LIBRARY:R_Axial_DIN0207_L6.3mm_D2.5mm_P10.16mm_Horizontal_2, F.Cu at (118.8, 135.2)
- added R5: 1K, IMRANS_LIBRARY:R_Axial_DIN0207_L6.3mm_D2.5mm_P10.16mm_Horizontal_2, F.Cu at (54.8, 35.3)
- added R5: 1K, IMRANS_LIBRARY:R_Axial_DIN0207_L6.3mm_D2.5mm_P10.16mm_Horizontal_2, F.Cu at (54.8, 101.9)
- added U1: LM358, Package_DIP:DIP-8_W7.62mm_Socket_LongPads, F.Cu at (190.6, 69.8)
- added U1: LM358, Package_DIP:DIP-8_W7.62mm_Socket_LongPads, F.Cu at (190.6, 136.4)
- added U1: LM358, Package_DIP:DIP-8_W7.62mm_Socket_LongPads, F.Cu at (254.6, 103.1)
- added U1: LM358, Package_DIP:DIP-8_W7.62mm_Socket_LongPads, F.Cu at (254.6, 136.4)
- added U1: LM358, Package_DIP:DIP-8_W7.62mm_Socket_LongPads, F.Cu at (126.6, 69.8)
- added U1: LM358, Package_DIP:DIP-8_W7.62mm_Socket_LongPads, F.Cu at (254.6, 36.5)
- added U1: LM358, Package_DIP:DIP-8_W7.62mm_Socket_LongPads, F.Cu at (190.6, 103.1)
- added U1: LM358, Package_DIP:DIP-8_W7.62mm_Socket_LongPads, F.Cu at (126.6, 103.1)
- added U1: LM358, Package_DIP:DIP-8_W7.62mm_Socket_LongPads, F.Cu at (62.6, 103.1)
- added U1: LM358, Package_DIP:DIP-8_W7.62mm_Socket_LongPads, F.Cu at (62.6, 136.4)
- added U1: LM358, Package_DIP:DIP-8_W7.62mm_Socket_LongPads, F.Cu at (126.6, 36.5)
- added U1: LM358, Package_DIP:DIP-8_W7.62mm_Socket_LongPads, F.Cu at (190.6, 36.5)
- added U1: LM358, Package_DIP:DIP-8_W7.62mm_Socket_LongPads, F.Cu at (62.6, 69.8)
- added U1: LM358, Package_DIP:DIP-8_W7.62mm_Socket_LongPads, F.Cu at (254.6, 69.8)
- added U1: LM358, Package_DIP:DIP-8_W7.62mm_Socket_LongPads, F.Cu at (126.6, 136.4)
- added U1: LM358, Package_DIP:DIP-8_W7.62mm_Socket_LongPads, F.Cu at (62.6, 36.5)
- added U4: LM555xN, Package_DIP:DIP-8_W7.62mm_Socket_LongPads, F.Cu at (237.1, 39.1)
- added U4: LM555xN, Package_DIP:DIP-8_W7.62mm_Socket_LongPads, F.Cu at (173.1, 72.4)
- added U4: LM555xN, Package_DIP:DIP-8_W7.62mm_Socket_LongPads, F.Cu at (109.1, 72.4)
- added U4: LM555xN, Package_DIP:DIP-8_W7.62mm_Socket_LongPads, F.Cu at (45.1, 39.1)
- added U4: LM555xN, Package_DIP:DIP-8_W7.62mm_Socket_LongPads, F.Cu at (173.1, 105.7)
- added U4: LM555xN, Package_DIP:DIP-8_W7.62mm_Socket_LongPads, F.Cu at (237.1, 139.0)
- added U4: LM555xN, Package_DIP:DIP-8_W7.62mm_Socket_LongPads, F.Cu at (237.1, 105.7)
- added U4: LM555xN, Package_DIP:DIP-8_W7.62mm_Socket_LongPads, F.Cu at (173.1, 139.0)
- added U4: LM555xN, Package_DIP:DIP-8_W7.62mm_Socket_LongPads, F.Cu at (45.1, 105.7)
- added U4: LM555xN, Package_DIP:DIP-8_W7.62mm_Socket_LongPads, F.Cu at (173.1, 39.1)
- added U4: LM555xN, Package_DIP:DIP-8_W7.62mm_Socket_LongPads, F.Cu at (109.1, 39.1)
- added U4: LM555xN, Package_DIP:DIP-8_W7.62mm_Socket_LongPads, F.Cu at (109.1, 139.0)
- added U4: LM555xN, Package_DIP:DIP-8_W7.62mm_Socket_LongPads, F.Cu at (237.1, 72.4)
- added U4: LM555xN, Package_DIP:DIP-8_W7.62mm_Socket_LongPads, F.Cu at (109.1, 105.7)
- added U4: LM555xN, Package_DIP:DIP-8_W7.62mm_Socket_LongPads, F.Cu at (45.1, 139.0)
- added U4: LM555xN, Package_DIP:DIP-8_W7.62mm_Socket_LongPads, F.Cu at (45.1, 72.4)
Routing:
- net Board_16-VCC: track 79.1 -> 0.00 mm
- net Board_22-VCC: track 79.1 -> 0.00 mm
- net Board_20-VCC: track 79.1 -> 0.00 mm
- net Board_19-VCC: track 79.1 -> 0.00 mm
- net Board_17-VCC: track 79.1 -> 0.00 mm
- net Board_21-VCC: track 79.1 -> 0.00 mm
- net Board_18-VCC: track 79.1 -> 0.00 mm
- net Board_23-VCC: track 79.1 -> 0.00 mm
- net Board_23-Net-(U4-R): track 43.6 -> 0.00 mm
- net Board_17-Net-(U4-R): track 43.6 -> 0.00 mm
- net Board_20-Net-(U4-R): track 43.6 -> 0.00 mm
- net Board_18-Net-(U4-R): track 43.6 -> 0.00 mm
- net Board_16-Net-(U4-R): track 43.6 -> 0.00 mm
- net Board_22-Net-(U4-R): track 43.6 -> 0.00 mm
- net Board_21-Net-(U4-R): track 43.6 -> 0.00 mm
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- removed copper zone on B.Cu, net Board_16-GND
- removed copper zone on B.Cu, net Board_17-GND
- removed copper zone on B.Cu, net Board_18-GND
- removed copper zone on B.Cu, net Board_19-GND
- removed copper zone on B.Cu, net Board_20-GND
- removed copper zone on B.Cu, net Board_21-GND
- removed copper zone on B.Cu, net Board_22-GND
- removed copper zone on B.Cu, net Board_23-GND
Other:
- board size 335 x 169.4 mm -> 255 x 132.7 mm
- board text added: "B.K DOCK"
- board text added: "V1.1"
- board text removed: "BOT"
- board text removed: "SERVE"
