File: mower/PCB/TRANSMITTER_DIP/TRANSMITTER_PANEL.kicad_pcb (KiCad board)
At the start: 2 copper layers, 255 x 132.7 mm, 256 parts, among them J1 BOT POWER, J2 POWER IN, J3 SHUNT, J4 COIL OUT, J5 COIL POWER IN, Q1 IRF3205, U1 LM358, U4 LM555xN

Commit message: .
Parts:
- removed the C2 at (30.2, 149.3)
- removed the C2 at (158.2, 82.7)
- removed the C2 at (158.2, 149.3)
- removed the C2 at (158.2, 116.0)
- removed the C2 at (30.2, 116.0)
- removed the C2 at (30.2, 49.4)
- removed the C2 at (222.2, 116.0)
- removed the C2 at (222.2, 149.3)
- removed the C2 at (94.2, 82.7)
- removed the C2 at (94.2, 116.0)
- removed the C2 at (30.2, 82.7)
- removed the C2 at (222.2, 49.4)
- removed the C2 at (94.2, 49.4)
- removed the C2 at (158.2, 49.4)
- removed the C2 at (94.2, 149.3)
- removed the C2 at (222.2, 82.7)
- added C2: 100nF, IMRANS_LIBRARY:C_Disc_D3.0mm_W1.6mm_P2.50mm, F.Cu at (157.8, 49.2)
- added C2: 100nF, IMRANS_LIBRARY:C_Disc_D3.0mm_W1.6mm_P2.50mm, F.Cu at (157.8, 82.5)
- added C2: 100nF, IMRANS_LIBRARY:C_Disc_D3.0mm_W1.6mm_P2.50mm, F.Cu at (157.8, 149.1)
- added C2: 100nF, IMRANS_LIBRARY:C_Disc_D3.0mm_W1.6mm_P2.50mm, F.Cu at (157.8, 115.8)
- added C2: 100nF, IMRANS_LIBRARY:C_Disc_D3.0mm_W1.6mm_P2.50mm, F.Cu at (93.8, 82.5)
- added C2: 100nF, IMRANS_LIBRARY:C_Disc_D3.0mm_W1.6mm_P2.50mm, F.Cu at (93.8, 115.8)
- added C2: 100nF, IMRANS_LIBRARY:C_Disc_D3.0mm_W1.6mm_P2.50mm, F.Cu at (93.8, 49.2)
- added C2: 100nF, IMRANS_LIBRARY:C_Disc_D3.0mm_W1.6mm_P2.50mm, F.Cu at (29.8, 115.8)
- added C2: 100nF, IMRANS_LIBRARY:C_Disc_D3.0mm_W1.6mm_P2.50mm, F.Cu at (29.8, 82.5)
- added C2: 100nF, IMRANS_LIBRARY:C_Disc_D3.0mm_W1.6mm_P2.50mm, F.Cu at (29.8, 49.2)
- added C2: 100nF, IMRANS_LIBRARY:C_Disc_D3.0mm_W1.6mm_P2.50mm, F.Cu at (221.8, 115.8)
- added C2: 100nF, IMRANS_LIBRARY:C_Disc_D3.0mm_W1.6mm_P2.50mm, F.Cu at (221.8, 149.1)
- added C2: 100nF, IMRANS_LIBRARY:C_Disc_D3.0mm_W1.6mm_P2.50mm, F.Cu at (221.8, 49.2)
- added C2: 100nF, IMRANS_LIBRARY:C_Disc_D3.0mm_W1.6mm_P2.50mm, F.Cu at (93.8, 149.1)
- added C2: 100nF, IMRANS_LIBRARY:C_Disc_D3.0mm_W1.6mm_P2.50mm, F.Cu at (29.8, 149.1)
- added C2: 100nF, IMRANS_LIBRARY:C_Disc_D3.0mm_W1.6mm_P2.50mm, F.Cu at (221.8, 82.5)
Connections:
- U1 pad 4: Board_1-unconnected-(U1C-V--Pad4) -> Board_1-GND
- U1 pad 8: Board_1-unconnected-(U1C-V+-Pad8) -> Board_1-VCC
- U1 pad 4: Board_8-unconnected-(U1C-V--Pad4) -> Board_8-GND
- U1 pad 8: Board_8-unconnected-(U1C-V+-Pad8) -> Board_8-VCC
- U1 pad 4: Board_7-unconnected-(U1C-V--Pad4) -> Board_7-GND
- U1 pad 8: Board_7-unconnected-(U1C-V+-Pad8) -> Board_7-VCC
- U1 pad 4: Board_15-unconnected-(U1C-V--Pad4) -> Board_15-GND
- U1 pad 8: Board_15-unconnected-(U1C-V+-Pad8) -> Board_15-VCC
- U1 pad 4: Board_4-unconnected-(U1C-V--Pad4) -> Board_4-GND
- U1 pad 8: Board_4-unconnected-(U1C-V+-Pad8) -> Board_4-VCC
- U1 pad 4: Board_6-unconnected-(U1C-V--Pad4) -> Board_6-GND
- U1 pad 8: Board_6-unconnected-(U1C-V+-Pad8) -> Board_6-VCC
- U1 pad 4: Board_12-unconnected-(U1C-V--Pad4) -> Board_12-GND
- U1 pad 8: Board_12-unconnected-(U1C-V+-Pad8) -> Board_12-VCC
- U1 pad 4: Board_11-unconnected-(U1C-V--Pad4) -> Board_11-GND
- U1 pad 8: Board_11-unconnected-(U1C-V+-Pad8) -> Board_11-VCC
- U1 pad 4: Board_0-unconnected-(U1C-V--Pad4) -> Board_0-GND
- U1 pad 8: Board_0-unconnected-(U1C-V+-Pad8) -> Board_0-VCC
- U1 pad 4: Board_9-unconnected-(U1C-V--Pad4) -> Board_9-GND
- U1 pad 8: Board_9-unconnected-(U1C-V+-Pad8) -> Board_9-VCC
- U1 pad 4: Board_2-unconnected-(U1C-V--Pad4) -> Board_2-GND
- U1 pad 8: Board_2-unconnected-(U1C-V+-Pad8) -> Board_2-VCC
- U1 pad 4: Board_14-unconnected-(U1C-V--Pad4) -> Board_14-GND
- U1 pad 8: Board_14-unconnected-(U1C-V+-Pad8) -> Board_14-VCC
- U1 pad 4: Board_3-unconnected-(U1C-V--Pad4) -> Board_3-GND
- U1 pad 8: Board_3-unconnected-(U1C-V+-Pad8) -> Board_3-VCC
- U1 pad 4: Board_5-unconnected-(U1C-V--Pad4) -> Board_5-GND
- U1 pad 8: Board_5-unconnected-(U1C-V+-Pad8) -> Board_5-VCC
- U1 pad 4: Board_13-unconnected-(U1C-V--Pad4) -> Board_13-GND
- U1 pad 8: Board_13-unconnected-(U1C-V+-Pad8) -> Board_13-VCC
- U1 pad 4: Board_10-unconnected-(U1C-V--Pad4) -> Board_10-GND
- U1 pad 8: Board_10-unconnected-(U1C-V+-Pad8) -> Board_10-VCC
Routing:
- net Board_15-Net-(U4-Q): track 5.56 -> 10.1 mm
- net Board_14-Net-(U4-Q): track 5.56 -> 10.1 mm
- net Board_12-Net-(U4-Q): track 5.56 -> 10.1 mm
- net Board_13-Net-(U4-Q): track 5.56 -> 10.1 mm
- net Board_7-Net-(U4-Q): track 5.56 -> 10.1 mm
- net Board_6-Net-(U4-Q): track 5.56 -> 10.1 mm
- net Board_3-Net-(U4-Q): track 5.56 -> 10.1 mm
- net Board_2-Net-(U4-Q): track 5.56 -> 10.1 mm
- net Board_11-Net-(U4-Q): track 5.56 -> 10.1 mm
- net Board_10-Net-(U4-Q): track 5.56 -> 10.1 mm
- net Board_4-Net-(U4-Q): track 5.56 -> 10.1 mm
- net Board_0-Net-(U4-Q): track 5.56 -> 10.1 mm
- net Board_8-Net-(U4-Q): track 5.56 -> 10.1 mm
- net Board_9-Net-(U4-Q): track 5.56 -> 10.1 mm
- net Board_5-Net-(U4-Q): track 5.56 -> 10.1 mm
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