File: mower/PCB/TRANSMITTER_DIP/TRANSMITTER_PANEL.kicad_pcb (KiCad board)
At the start: 2 copper layers, 255 x 132.7 mm, 256 parts, among them J1 BOT POWER, J2 POWER IN, J3 SHUNT, J4 COIL OUT, J5 COIL POWER IN, Q1 IRF3205, U1 LM358, U4 LM555xN

Commit message: Consolidate complete mower design (all branches) + zana repo structure
Mower fragments from every botkorp branch (mowbot3/4, TRANSMITTER_SMD,
IMRANS_LIBRARY) unioned into mower/. Adds legacy/opengro, README, .gitignore.
Sits on top of the preserved 13-commit mower history.

Co-Authored-By: Claude Opus 4.8 <noreply@anthropic.com>
Claude-Session: https://claude.ai/code/session_017QXBEryTihUadNUZqQzfmo
Parts:
- removed the C1 at (120.6, 111.0)
- removed the C1 at (56.6, 111.0)
- removed the C1 at (184.6, 111.0)
- removed the C1 at (120.6, 44.4)
- removed the C1 at (248.6, 111.0)
- removed the C1 at (248.6, 44.4)
- removed the C1 at (56.6, 44.4)
- removed the C1 at (248.6, 77.7)
- removed the C1 at (56.6, 144.3)
- removed the C1 at (120.6, 144.3)
- removed the C1 at (248.6, 144.3)
- removed the C1 at (184.6, 44.4)
- removed the C1 at (56.6, 77.7)
- removed the C1 at (184.6, 144.3)
- removed the C1 at (184.6, 77.7)
- removed the C1 at (120.6, 77.7)
- removed C2 (x16): 100nF, IMRANS_LIBRARY:C_Disc_D3.0mm_W1.6mm_P2.50mm
- removed the D1 at (24.7, 101.2)
- removed the D1 at (24.7, 67.9)
- removed the D1 at (152.7, 34.6)
- removed the D1 at (216.7, 34.6)
- removed the D1 at (24.7, 134.5)
- removed the D1 at (88.7, 101.2)
- removed the D1 at (216.7, 67.9)
- removed the D1 at (152.7, 134.5)
- removed the D1 at (24.7, 34.6)
- removed the D1 at (88.7, 34.6)
- removed the D1 at (88.7, 134.5)
- removed the D1 at (152.7, 101.2)
- removed the D1 at (216.7, 101.2)
- removed the D1 at (152.7, 67.9)
- removed the D1 at (216.7, 134.5)
- removed the D1 at (88.7, 67.9)
- removed the J1 at (55.1, 60.4)
- removed the J1 at (183.1, 93.7)
- removed the J1 at (119.1, 27.1)
- removed the J1 at (183.1, 127.0)
- removed the J1 at (247.1, 127.0)
- removed the J1 at (247.1, 93.7)
- removed the J1 at (183.1, 60.4)
- removed the J1 at (183.1, 27.1)
- removed the J1 at (247.1, 60.4)
- removed the J1 at (119.1, 60.4)
- removed the J1 at (55.1, 27.1)
- removed the J1 at (119.1, 127.0)
- removed the J1 at (55.1, 127.0)
- removed the J1 at (119.1, 93.7)
- removed the J1 at (247.1, 27.1)
- removed the J1 at (55.1, 93.7)
- removed the J2 at (78.1, 93.8)
- removed the J2 at (206.1, 60.5)
- removed the J2 at (78.1, 127.1)
- removed the J2 at (206.1, 127.1)
- removed the J2 at (270.1, 93.8)
- removed the J2 at (78.1, 60.5)
- removed the J2 at (270.1, 60.5)
- removed the J2 at (78.1, 27.2)
- removed the J2 at (142.1, 127.1)
- removed the J2 at (206.1, 93.8)
- removed the J2 at (270.1, 127.1)
- removed the J2 at (142.1, 93.8)
- removed the J2 at (270.1, 27.2)
- removed the J2 at (142.1, 60.5)
- removed the J2 at (142.1, 27.2)
- removed the J2 at (206.1, 27.2)
- removed the J3 at (130.5, 27.1)
- removed the J3 at (194.5, 93.7)
- removed the J3 at (130.5, 60.4)
- removed the J3 at (258.5, 127.0)
- removed the J3 at (130.5, 127.0)
- removed the J3 at (66.5, 60.4)
- removed the J3 at (258.5, 27.1)
- removed the J3 at (194.5, 60.4)
- removed the J3 at (66.5, 27.1)
- removed the J3 at (194.5, 127.0)
- removed the J3 at (130.5, 93.7)
- removed the J3 at (194.5, 27.1)
- removed the J3 at (258.5, 60.4)
- removed the J3 at (66.5, 127.0)
- removed the J3 at (258.5, 93.7)
- removed the J3 at (66.5, 93.7)
- removed the J4 at (96.4, 27.1)
- removed the J4 at (160.4, 27.1)
- removed the J4 at (96.4, 60.4)
- removed the J4 at (32.4, 27.1)
- removed the J4 at (224.4, 27.1)
- removed the J4 at (32.4, 93.7)
- removed the J4 at (224.4, 127.0)
- removed the J4 at (160.4, 93.7)
- removed the J4 at (32.4, 127.0)
- removed the J4 at (224.4, 60.4)
- removed the J4 at (32.4, 60.4)
- removed the J4 at (96.4, 93.7)
- removed the J4 at (160.4, 60.4)
- removed the J4 at (96.4, 127.0)
- removed the J4 at (224.4, 93.7)
- removed the J4 at (160.4, 127.0)
- removed the J5 at (107.7, 27.1)
- removed the J5 at (171.7, 27.1)
- removed the J5 at (171.7, 60.4)
- removed the J5 at (43.7, 93.7)
- removed the J5 at (107.7, 127.0)
- removed the J5 at (171.7, 93.7)
- removed the J5 at (107.7, 93.7)
- removed the J5 at (43.7, 60.4)
- removed the J5 at (235.7, 27.1)
- removed the J5 at (171.7, 127.0)
- removed the J5 at (235.7, 93.7)
- removed the J5 at (235.7, 60.4)
- removed the J5 at (43.7, 27.1)
- removed the J5 at (235.7, 127.0)
- removed the J5 at (43.7, 127.0)
- removed the J5 at (107.7, 60.4)
- removed the Q1 at (98.6, 44.6)
- removed the Q1 at (98.6, 111.2)
- removed the Q1 at (162.6, 77.9)
- removed the Q1 at (34.6, 144.5)
- removed the Q1 at (34.6, 77.9)
- removed the Q1 at (162.6, 111.2)
- removed the Q1 at (98.6, 77.9)
- removed the Q1 at (162.6, 144.5)
- removed the Q1 at (162.6, 44.6)
- removed the Q1 at (34.6, 44.6)
- removed the Q1 at (226.6, 44.6)
- removed the Q1 at (98.6, 144.5)
- removed the Q1 at (226.6, 144.5)
- removed the Q1 at (226.6, 77.9)
- removed the Q1 at (34.6, 111.2)
- removed the Q1 at (226.6, 111.2)
- removed the R1 at (139.1, 69.1)
- removed the R1 at (267.1, 135.7)
- removed the R1 at (75.1, 135.7)
- removed the R1 at (203.1, 69.1)
- removed the R1 at (75.1, 35.8)
- removed the R1 at (203.1, 135.7)
- removed the R1 at (139.1, 135.7)
- removed the R1 at (267.1, 102.4)
- removed the R1 at (203.1, 35.8)
- removed the R1 at (139.1, 35.8)
- removed the R1 at (139.1, 102.4)
- removed the R1 at (203.1, 102.4)
- removed the R1 at (75.1, 69.1)
- removed the R1 at (267.1, 69.1)
- removed the R1 at (267.1, 35.8)
- removed the R1 at (75.1, 102.4)
- removed the R2 at (135.8, 147.8)
- removed the R2 at (135.8, 114.5)
- removed the R2 at (263.8, 81.2)
- removed the R2 at (263.8, 114.5)
- removed the R2 at (135.8, 47.9)
- removed the R2 at (199.8, 47.9)
- removed the R2 at (263.8, 47.9)
- removed the R2 at (71.8, 81.2)
- removed the R2 at (199.8, 147.8)
- removed the R2 at (71.8, 147.8)
- removed the R2 at (199.8, 114.5)
- removed the R2 at (199.8, 81.2)
- removed the R2 at (135.8, 81.2)
- removed the R2 at (263.8, 147.8)
- removed the R2 at (71.8, 47.9)
- removed the R2 at (71.8, 114.5)
- removed the R3 at (41.7, 114.0)
- removed the R3 at (41.7, 80.7)
- removed the R3 at (169.7, 47.4)
- removed the R3 at (105.7, 80.7)
- removed the R3 at (233.7, 80.7)
- removed the R3 at (105.7, 147.3)
- removed the R3 at (169.7, 80.7)
- removed the R3 at (169.7, 147.3)
- removed the R3 at (233.7, 147.3)
- removed the R3 at (41.7, 47.4)
- removed the R3 at (41.7, 147.3)
- removed the R3 at (105.7, 114.0)
- removed the R3 at (233.7, 47.4)
- removed the R3 at (169.7, 114.0)
- removed the R3 at (105.7, 47.4)
- removed the R3 at (233.7, 114.0)
- removed the R4 at (166.2, 83.2)
- removed the R4 at (38.2, 149.8)
- removed the R4 at (38.2, 116.5)
- removed the R4 at (38.2, 83.2)
- removed the R4 at (102.2, 149.8)
- removed the R4 at (166.2, 116.5)
- removed the R4 at (102.2, 116.5)
- removed the R4 at (102.2, 83.2)
- removed the R4 at (230.2, 83.2)
- removed the R4 at (166.2, 149.8)
- removed the R4 at (230.2, 49.9)
- removed the R4 at (102.2, 49.9)
- removed the R4 at (230.2, 149.8)
- removed the R4 at (38.2, 49.9)
- removed the R4 at (230.2, 116.5)
- removed the R4 at (166.2, 49.9)
- removed R5 (x16): 1K, IMRANS_LIBRARY:R_Axial_DIN0207_L6.3mm_D2.5mm_P10.16mm_Horizontal_2
- removed the U1 at (126.6, 36.5)
- removed the U1 at (62.6, 103.1)
- removed the U1 at (254.6, 69.8)
- removed the U1 at (254.6, 136.4)
- removed the U1 at (62.6, 69.8)
- removed the U1 at (190.6, 69.8)
- removed the U1 at (62.6, 136.4)
- removed the U1 at (254.6, 103.1)
- removed the U1 at (62.6, 36.5)
- removed the U1 at (126.6, 103.1)
- removed the U1 at (190.6, 36.5)
- removed the U1 at (190.6, 136.4)
- removed the U1 at (254.6, 36.5)
- removed the U1 at (126.6, 69.8)
- removed the U1 at (126.6, 136.4)
- removed the U1 at (190.6, 103.1)
- removed the U4 at (237.1, 105.7)
- removed the U4 at (173.1, 139.0)
- removed the U4 at (109.1, 105.7)
- removed the U4 at (173.1, 72.4)
- removed the U4 at (109.1, 72.4)
- removed the U4 at (173.1, 105.7)
- removed the U4 at (237.1, 39.1)
- removed the U4 at (45.1, 39.1)
- removed the U4 at (109.1, 139.0)
- removed the U4 at (45.1, 72.4)
- removed the U4 at (45.1, 139.0)
- removed the U4 at (45.1, 105.7)
- removed the U4 at (173.1, 39.1)
- removed the U4 at (237.1, 139.0)
- removed the U4 at (237.1, 72.4)
- removed the U4 at (109.1, 39.1)
- added C1: 10nF, IMRANS_LIBRARY:C_Disc_D3.0mm_W1.6mm_P2.50mm, F.Cu at (121.3, 179.5)
- added C1: 10nF, IMRANS_LIBRARY:C_Disc_D3.0mm_W1.6mm_P2.50mm, F.Cu at (9.28, 94.3)
- added C1: 10nF, IMRANS_LIBRARY:C_Disc_D3.0mm_W1.6mm_P2.50mm, F.Cu at (177.3, 94.3)
- added C1: 10nF, IMRANS_LIBRARY:C_Disc_D3.0mm_W1.6mm_P2.50mm, F.Cu at (177.3, 179.5)
- added C1: 10nF, IMRANS_LIBRARY:C_Disc_D3.0mm_W1.6mm_P2.50mm, F.Cu at (289.3, 179.5)
- added C1: 10nF, IMRANS_LIBRARY:C_Disc_D3.0mm_W1.6mm_P2.50mm, F.Cu at (177.3, 51.7)
- added C1: 10nF, IMRANS_LIBRARY:C_Disc_D3.0mm_W1.6mm_P2.50mm, F.Cu at (289.3, 94.3)
- added C1: 10nF, IMRANS_LIBRARY:C_Disc_D3.0mm_W1.6mm_P2.50mm, F.Cu at (121.3, 94.3)
- added C1: 10nF, IMRANS_LIBRARY:C_Disc_D3.0mm_W1.6mm_P2.50mm, F.Cu at (121.3, 136.9)
- added C1: 10nF, IMRANS_LIBRARY:C_Disc_D3.0mm_W1.6mm_P2.50mm, F.Cu at (65.3, 179.5)
- added C1: 10nF, IMRANS_LIBRARY:C_Disc_D3.0mm_W1.6mm_P2.50mm, F.Cu at (289.3, 51.7)
- added C1: 10nF, IMRANS_LIBRARY:C_Disc_D3.0mm_W1.6mm_P2.50mm, F.Cu at (233.3, 136.9)
- added C1: 10nF, IMRANS_LIBRARY:C_Disc_D3.0mm_W1.6mm_P2.50mm, F.Cu at (9.28, 51.7)
- added C1: 10nF, IMRANS_LIBRARY:C_Disc_D3.0mm_W1.6mm_P2.50mm, F.Cu at (233.3, 94.3)
- added C1: 10nF, IMRANS_LIBRARY:C_Disc_D3.0mm_W1.6mm_P2.50mm, F.Cu at (289.3, 136.9)
- added C1: 10nF, IMRANS_LIBRARY:C_Disc_D3.0mm_W1.6mm_P2.50mm, F.Cu at (9.28, 179.5)
- added C1: 10nF, IMRANS_LIBRARY:C_Disc_D3.0mm_W1.6mm_P2.50mm, F.Cu at (65.3, 51.7)
- added C1: 10nF, IMRANS_LIBRARY:C_Disc_D3.0mm_W1.6mm_P2.50mm, F.Cu at (9.28, 136.9)
- added C1: 10nF, IMRANS_LIBRARY:C_Disc_D3.0mm_W1.6mm_P2.50mm, F.Cu at (121.3, 51.7)
- added C1: 10nF, IMRANS_LIBRARY:C_Disc_D3.0mm_W1.6mm_P2.50mm, F.Cu at (65.3, 94.3)
- added C1: 10nF, IMRANS_LIBRARY:C_Disc_D3.0mm_W1.6mm_P2.50mm, F.Cu at (233.3, 51.7)
- added C1: 10nF, IMRANS_LIBRARY:C_Disc_D3.0mm_W1.6mm_P2.50mm, F.Cu at (65.3, 136.9)
- added C1: 10nF, IMRANS_LIBRARY:C_Disc_D3.0mm_W1.6mm_P2.50mm, F.Cu at (233.3, 179.5)
- added C1: 10nF, IMRANS_LIBRARY:C_Disc_D3.0mm_W1.6mm_P2.50mm, F.Cu at (177.3, 136.9)
- added D1: 1N5819, IMRANS_LIBRARY:R_Axial_DIN0207_L6.3mm_D2.5mm_P10.16mm_Horizontal_2, F.Cu at (100.6, 123.0)
- added D1: 1N5819, IMRANS_LIBRARY:R_Axial_DIN0207_L6.3mm_D2.5mm_P10.16mm_Horizontal_2, F.Cu at (212.6, 80.4)
- added D1: 1N5819, IMRANS_LIBRARY:R_Axial_DIN0207_L6.3mm_D2.5mm_P10.16mm_Horizontal_2, F.Cu at (268.6, 123.0)
- added D1: 1N5819, IMRANS_LIBRARY:R_Axial_DIN0207_L6.3mm_D2.5mm_P10.16mm_Horizontal_2, F.Cu at (100.6, 80.4)
- added D1: 1N5819, IMRANS_LIBRARY:R_Axial_DIN0207_L6.3mm_D2.5mm_P10.16mm_Horizontal_2, F.Cu at (-11.4, 80.4)
- added D1: 1N5819, IMRANS_LIBRARY:R_Axial_DIN0207_L6.3mm_D2.5mm_P10.16mm_Horizontal_2, F.Cu at (268.6, 165.6)
- added D1: 1N5819, IMRANS_LIBRARY:R_Axial_DIN0207_L6.3mm_D2.5mm_P10.16mm_Horizontal_2, F.Cu at (100.6, 37.8)
- added D1: 1N5819, IMRANS_LIBRARY:R_Axial_DIN0207_L6.3mm_D2.5mm_P10.16mm_Horizontal_2, F.Cu at (156.6, 37.8)
- added D1: 1N5819, IMRANS_LIBRARY:R_Axial_DIN0207_L6.3mm_D2.5mm_P10.16mm_Horizontal_2, F.Cu at (44.6, 123.0)
- added D1: 1N5819, IMRANS_LIBRARY:R_Axial_DIN0207_L6.3mm_D2.5mm_P10.16mm_Horizontal_2, F.Cu at (44.6, 165.6)
- added D1: 1N5819, IMRANS_LIBRARY:R_Axial_DIN0207_L6.3mm_D2.5mm_P10.16mm_Horizontal_2, F.Cu at (-11.4, 123.0)
- added D1: 1N5819, IMRANS_LIBRARY:R_Axial_DIN0207_L6.3mm_D2.5mm_P10.16mm_Horizontal_2, F.Cu at (44.6, 37.8)
- added D1: 1N5819, IMRANS_LIBRARY:R_Axial_DIN0207_L6.3mm_D2.5mm_P10.16mm_Horizontal_2, F.Cu at (156.6, 123.0)
- added D1: 1N5819, IMRANS_LIBRARY:R_Axial_DIN0207_L6.3mm_D2.5mm_P10.16mm_Horizontal_2, F.Cu at (268.6, 37.8)
- added D1: 1N5819, IMRANS_LIBRARY:R_Axial_DIN0207_L6.3mm_D2.5mm_P10.16mm_Horizontal_2, F.Cu at (212.6, 165.6)
- added D1: 1N5819, IMRANS_LIBRARY:R_Axial_DIN0207_L6.3mm_D2.5mm_P10.16mm_Horizontal_2, F.Cu at (156.6, 80.4)
- added D1: 1N5819, IMRANS_LIBRARY:R_Axial_DIN0207_L6.3mm_D2.5mm_P10.16mm_Horizontal_2, F.Cu at (-11.4, 37.8)
- added D1: 1N5819, IMRANS_LIBRARY:R_Axial_DIN0207_L6.3mm_D2.5mm_P10.16mm_Horizontal_2, F.Cu at (156.6, 165.6)
- added D1: 1N5819, IMRANS_LIBRARY:R_Axial_DIN0207_L6.3mm_D2.5mm_P10.16mm_Horizontal_2, F.Cu at (212.6, 37.8)
- added D1: 1N5819, IMRANS_LIBRARY:R_Axial_DIN0207_L6.3mm_D2.5mm_P10.16mm_Horizontal_2, F.Cu at (212.6, 123.0)
- added D1: 1N5819, IMRANS_LIBRARY:R_Axial_DIN0207_L6.3mm_D2.5mm_P10.16mm_Horizontal_2, F.Cu at (-11.4, 165.6)
- added D1: 1N5819, IMRANS_LIBRARY:R_Axial_DIN0207_L6.3mm_D2.5mm_P10.16mm_Horizontal_2, F.Cu at (44.6, 80.4)
- added D1: 1N5819, IMRANS_LIBRARY:R_Axial_DIN0207_L6.3mm_D2.5mm_P10.16mm_Horizontal_2, F.Cu at (100.6, 165.6)
- added D1: 1N5819, IMRANS_LIBRARY:R_Axial_DIN0207_L6.3mm_D2.5mm_P10.16mm_Horizontal_2, F.Cu at (268.6, 80.4)
- added J1: BOT POWER, TerminalBlock_Phoenix:TerminalBlock_Phoenix_MKDS-1,5-2-5.08_1x02_P5.08mm_Horizontal, F.Cu at (175.5, 30.2)
- added J1: BOT POWER, TerminalBlock_Phoenix:TerminalBlock_Phoenix_MKDS-1,5-2-5.08_1x02_P5.08mm_Horizontal, F.Cu at (287.5, 115.4)
- added J1: BOT POWER, TerminalBlock_Phoenix:TerminalBlock_Phoenix_MKDS-1,5-2-5.08_1x02_P5.08mm_Horizontal, F.Cu at (175.5, 115.4)
- added J1: BOT POWER, TerminalBlock_Phoenix:TerminalBlock_Phoenix_MKDS-1,5-2-5.08_1x02_P5.08mm_Horizontal, F.Cu at (119.5, 158.0)
- added J1: BOT POWER, TerminalBlock_Phoenix:TerminalBlock_Phoenix_MKDS-1,5-2-5.08_1x02_P5.08mm_Horizontal, F.Cu at (63.5, 158.0)
- added J1: BOT POWER, TerminalBlock_Phoenix:TerminalBlock_Phoenix_MKDS-1,5-2-5.08_1x02_P5.08mm_Horizontal, F.Cu at (63.5, 115.4)
- added J1: BOT POWER, TerminalBlock_Phoenix:TerminalBlock_Phoenix_MKDS-1,5-2-5.08_1x02_P5.08mm_Horizontal, F.Cu at (231.5, 115.4)
- added J1: BOT POWER, TerminalBlock_Phoenix:TerminalBlock_Phoenix_MKDS-1,5-2-5.08_1x02_P5.08mm_Horizontal, F.Cu at (63.5, 72.8)
- added J1: BOT POWER, TerminalBlock_Phoenix:TerminalBlock_Phoenix_MKDS-1,5-2-5.08_1x02_P5.08mm_Horizontal, F.Cu at (231.5, 72.8)
- added J1: BOT POWER, TerminalBlock_Phoenix:TerminalBlock_Phoenix_MKDS-1,5-2-5.08_1x02_P5.08mm_Horizontal, F.Cu at (175.5, 72.8)
- added J1: BOT POWER, TerminalBlock_Phoenix:TerminalBlock_Phoenix_MKDS-1,5-2-5.08_1x02_P5.08mm_Horizontal, F.Cu at (7.50, 115.4)
- added J1: BOT POWER, TerminalBlock_Phoenix:TerminalBlock_Phoenix_MKDS-1,5-2-5.08_1x02_P5.08mm_Horizontal, F.Cu at (231.5, 30.2)
- added J1: BOT POWER, TerminalBlock_Phoenix:TerminalBlock_Phoenix_MKDS-1,5-2-5.08_1x02_P5.08mm_Horizontal, F.Cu at (287.5, 158.0)
- added J1: BOT POWER, TerminalBlock_Phoenix:TerminalBlock_Phoenix_MKDS-1,5-2-5.08_1x02_P5.08mm_Horizontal, F.Cu at (119.5, 72.8)
- added J1: BOT POWER, TerminalBlock_Phoenix:TerminalBlock_Phoenix_MKDS-1,5-2-5.08_1x02_P5.08mm_Horizontal, F.Cu at (7.50, 72.8)
- added J1: BOT POWER, TerminalBlock_Phoenix:TerminalBlock_Phoenix_MKDS-1,5-2-5.08_1x02_P5.08mm_Horizontal, F.Cu at (7.50, 30.2)
- added J1: BOT POWER, TerminalBlock_Phoenix:TerminalBlock_Phoenix_MKDS-1,5-2-5.08_1x02_P5.08mm_Horizontal, F.Cu at (287.5, 30.2)
- added J1: BOT POWER, TerminalBlock_Phoenix:TerminalBlock_Phoenix_MKDS-1,5-2-5.08_1x02_P5.08mm_Horizontal, F.Cu at (7.50, 158.0)
- added J1: BOT POWER, TerminalBlock_Phoenix:TerminalBlock_Phoenix_MKDS-1,5-2-5.08_1x02_P5.08mm_Horizontal, F.Cu at (63.5, 30.2)
- added J1: BOT POWER, TerminalBlock_Phoenix:TerminalBlock_Phoenix_MKDS-1,5-2-5.08_1x02_P5.08mm_Horizontal, F.Cu at (287.5, 72.8)
- added J1: BOT POWER, TerminalBlock_Phoenix:TerminalBlock_Phoenix_MKDS-1,5-2-5.08_1x02_P5.08mm_Horizontal, F.Cu at (119.5, 30.2)
- added J1: BOT POWER, TerminalBlock_Phoenix:TerminalBlock_Phoenix_MKDS-1,5-2-5.08_1x02_P5.08mm_Horizontal, F.Cu at (175.5, 158.0)
- added J1: BOT POWER, TerminalBlock_Phoenix:TerminalBlock_Phoenix_MKDS-1,5-2-5.08_1x02_P5.08mm_Horizontal, F.Cu at (231.5, 158.0)
- added J1: BOT POWER, TerminalBlock_Phoenix:TerminalBlock_Phoenix_MKDS-1,5-2-5.08_1x02_P5.08mm_Horizontal, F.Cu at (119.5, 115.4)
- added J2: POWER IN, TerminalBlock_Phoenix:TerminalBlock_Phoenix_MKDS-1,5-2-5.08_1x02_P5.08mm_Horizontal, F.Cu at (86.5, 72.8)
- added J2: POWER IN, TerminalBlock_Phoenix:TerminalBlock_Phoenix_MKDS-1,5-2-5.08_1x02_P5.08mm_Horizontal, F.Cu at (30.5, 158.0)
- added J2: POWER IN, TerminalBlock_Phoenix:TerminalBlock_Phoenix_MKDS-1,5-2-5.08_1x02_P5.08mm_Horizontal, F.Cu at (142.5, 30.2)
- added J2: POWER IN, TerminalBlock_Phoenix:TerminalBlock_Phoenix_MKDS-1,5-2-5.08_1x02_P5.08mm_Horizontal, F.Cu at (86.5, 158.0)
- added J2: POWER IN, TerminalBlock_Phoenix:TerminalBlock_Phoenix_MKDS-1,5-2-5.08_1x02_P5.08mm_Horizontal, F.Cu at (30.5, 72.8)
- added J2: POWER IN, TerminalBlock_Phoenix:TerminalBlock_Phoenix_MKDS-1,5-2-5.08_1x02_P5.08mm_Horizontal, F.Cu at (254.5, 158.0)
- added J2: POWER IN, TerminalBlock_Phoenix:TerminalBlock_Phoenix_MKDS-1,5-2-5.08_1x02_P5.08mm_Horizontal, F.Cu at (198.5, 158.0)
- added J2: POWER IN, TerminalBlock_Phoenix:TerminalBlock_Phoenix_MKDS-1,5-2-5.08_1x02_P5.08mm_Horizontal, F.Cu at (198.5, 30.2)
- added J2: POWER IN, TerminalBlock_Phoenix:TerminalBlock_Phoenix_MKDS-1,5-2-5.08_1x02_P5.08mm_Horizontal, F.Cu at (310.5, 30.2)
- added J2: POWER IN, TerminalBlock_Phoenix:TerminalBlock_Phoenix_MKDS-1,5-2-5.08_1x02_P5.08mm_Horizontal, F.Cu at (86.5, 30.2)
- added J2: POWER IN, TerminalBlock_Phoenix:TerminalBlock_Phoenix_MKDS-1,5-2-5.08_1x02_P5.08mm_Horizontal, F.Cu at (254.5, 30.2)
- added J2: POWER IN, TerminalBlock_Phoenix:TerminalBlock_Phoenix_MKDS-1,5-2-5.08_1x02_P5.08mm_Horizontal, F.Cu at (86.5, 115.4)
- added J2: POWER IN, TerminalBlock_Phoenix:TerminalBlock_Phoenix_MKDS-1,5-2-5.08_1x02_P5.08mm_Horizontal, F.Cu at (142.5, 115.4)
- added J2: POWER IN, TerminalBlock_Phoenix:TerminalBlock_Phoenix_MKDS-1,5-2-5.08_1x02_P5.08mm_Horizontal, F.Cu at (254.5, 115.4)
- added J2: POWER IN, TerminalBlock_Phoenix:TerminalBlock_Phoenix_MKDS-1,5-2-5.08_1x02_P5.08mm_Horizontal, F.Cu at (310.5, 158.0)
- added J2: POWER IN, TerminalBlock_Phoenix:TerminalBlock_Phoenix_MKDS-1,5-2-5.08_1x02_P5.08mm_Horizontal, F.Cu at (142.5, 158.0)
- added J2: POWER IN, TerminalBlock_Phoenix:TerminalBlock_Phoenix_MKDS-1,5-2-5.08_1x02_P5.08mm_Horizontal, F.Cu at (254.5, 72.8)
- added J2: POWER IN, TerminalBlock_Phoenix:TerminalBlock_Phoenix_MKDS-1,5-2-5.08_1x02_P5.08mm_Horizontal, F.Cu at (30.5, 30.2)
- added J2: POWER IN, TerminalBlock_Phoenix:TerminalBlock_Phoenix_MKDS-1,5-2-5.08_1x02_P5.08mm_Horizontal, F.Cu at (310.5, 115.4)
- added J2: POWER IN, TerminalBlock_Phoenix:TerminalBlock_Phoenix_MKDS-1,5-2-5.08_1x02_P5.08mm_Horizontal, F.Cu at (198.5, 115.4)
- added J2: POWER IN, TerminalBlock_Phoenix:TerminalBlock_Phoenix_MKDS-1,5-2-5.08_1x02_P5.08mm_Horizontal, F.Cu at (310.5, 72.8)
- added J2: POWER IN, TerminalBlock_Phoenix:TerminalBlock_Phoenix_MKDS-1,5-2-5.08_1x02_P5.08mm_Horizontal, F.Cu at (30.5, 115.4)
- added J2: POWER IN, TerminalBlock_Phoenix:TerminalBlock_Phoenix_MKDS-1,5-2-5.08_1x02_P5.08mm_Horizontal, F.Cu at (198.5, 72.8)
- added J2: POWER IN, TerminalBlock_Phoenix:TerminalBlock_Phoenix_MKDS-1,5-2-5.08_1x02_P5.08mm_Horizontal, F.Cu at (142.5, 72.8)
- added J3: SHUNT, TerminalBlock_Phoenix:TerminalBlock_Phoenix_MKDS-1,5-2-5.08_1x02_P5.08mm_Horizontal, F.Cu at (186.9, 115.4)
- added J3: SHUNT, TerminalBlock_Phoenix:TerminalBlock_Phoenix_MKDS-1,5-2-5.08_1x02_P5.08mm_Horizontal, F.Cu at (74.9, 72.8)
- added J3: SHUNT, TerminalBlock_Phoenix:TerminalBlock_Phoenix_MKDS-1,5-2-5.08_1x02_P5.08mm_Horizontal, F.Cu at (298.9, 72.8)
- added J3: SHUNT, TerminalBlock_Phoenix:TerminalBlock_Phoenix_MKDS-1,5-2-5.08_1x02_P5.08mm_Horizontal, F.Cu at (18.9, 115.4)
- added J3: SHUNT, TerminalBlock_Phoenix:TerminalBlock_Phoenix_MKDS-1,5-2-5.08_1x02_P5.08mm_Horizontal, F.Cu at (298.9, 158.0)
- added J3: SHUNT, TerminalBlock_Phoenix:TerminalBlock_Phoenix_MKDS-1,5-2-5.08_1x02_P5.08mm_Horizontal, F.Cu at (74.9, 115.4)
- added J3: SHUNT, TerminalBlock_Phoenix:TerminalBlock_Phoenix_MKDS-1,5-2-5.08_1x02_P5.08mm_Horizontal, F.Cu at (74.9, 30.2)
- added J3: SHUNT, TerminalBlock_Phoenix:TerminalBlock_Phoenix_MKDS-1,5-2-5.08_1x02_P5.08mm_Horizontal, F.Cu at (298.9, 115.4)
- added J3: SHUNT, TerminalBlock_Phoenix:TerminalBlock_Phoenix_MKDS-1,5-2-5.08_1x02_P5.08mm_Horizontal, F.Cu at (130.9, 158.0)
- added J3: SHUNT, TerminalBlock_Phoenix:TerminalBlock_Phoenix_MKDS-1,5-2-5.08_1x02_P5.08mm_Horizontal, F.Cu at (242.9, 115.4)
- added J3: SHUNT, TerminalBlock_Phoenix:TerminalBlock_Phoenix_MKDS-1,5-2-5.08_1x02_P5.08mm_Horizontal, F.Cu at (130.9, 115.4)
- added J3: SHUNT, TerminalBlock_Phoenix:TerminalBlock_Phoenix_MKDS-1,5-2-5.08_1x02_P5.08mm_Horizontal, F.Cu at (242.9, 158.0)
- added J3: SHUNT, TerminalBlock_Phoenix:TerminalBlock_Phoenix_MKDS-1,5-2-5.08_1x02_P5.08mm_Horizontal, F.Cu at (18.9, 158.0)
- added J3: SHUNT, TerminalBlock_Phoenix:TerminalBlock_Phoenix_MKDS-1,5-2-5.08_1x02_P5.08mm_Horizontal, F.Cu at (18.9, 30.2)
- added J3: SHUNT, TerminalBlock_Phoenix:TerminalBlock_Phoenix_MKDS-1,5-2-5.08_1x02_P5.08mm_Horizontal, F.Cu at (130.9, 72.8)
- added J3: SHUNT, TerminalBlock_Phoenix:TerminalBlock_Phoenix_MKDS-1,5-2-5.08_1x02_P5.08mm_Horizontal, F.Cu at (242.9, 72.8)
- added J3: SHUNT, TerminalBlock_Phoenix:TerminalBlock_Phoenix_MKDS-1,5-2-5.08_1x02_P5.08mm_Horizontal, F.Cu at (130.9, 30.2)
- added J3: SHUNT, TerminalBlock_Phoenix:TerminalBlock_Phoenix_MKDS-1,5-2-5.08_1x02_P5.08mm_Horizontal, F.Cu at (298.9, 30.2)
- added J3: SHUNT, TerminalBlock_Phoenix:TerminalBlock_Phoenix_MKDS-1,5-2-5.08_1x02_P5.08mm_Horizontal, F.Cu at (186.9, 30.2)
- added J3: SHUNT, TerminalBlock_Phoenix:TerminalBlock_Phoenix_MKDS-1,5-2-5.08_1x02_P5.08mm_Horizontal, F.Cu at (186.9, 72.8)
- added J3: SHUNT, TerminalBlock_Phoenix:TerminalBlock_Phoenix_MKDS-1,5-2-5.08_1x02_P5.08mm_Horizontal, F.Cu at (74.9, 158.0)
- added J3: SHUNT, TerminalBlock_Phoenix:TerminalBlock_Phoenix_MKDS-1,5-2-5.08_1x02_P5.08mm_Horizontal, F.Cu at (18.9, 72.8)
- added J3: SHUNT, TerminalBlock_Phoenix:TerminalBlock_Phoenix_MKDS-1,5-2-5.08_1x02_P5.08mm_Horizontal, F.Cu at (186.9, 158.0)
- added J3: SHUNT, TerminalBlock_Phoenix:TerminalBlock_Phoenix_MKDS-1,5-2-5.08_1x02_P5.08mm_Horizontal, F.Cu at (242.9, 30.2)
- added J4: COIL OUT, TerminalBlock_Phoenix:TerminalBlock_Phoenix_MKDS-1,5-2-5.08_1x02_P5.08mm_Horizontal, F.Cu at (107.9, 72.8)
- added J4: COIL OUT, TerminalBlock_Phoenix:TerminalBlock_Phoenix_MKDS-1,5-2-5.08_1x02_P5.08mm_Horizontal, F.Cu at (-4.06, 115.4)
- added J4: COIL OUT, TerminalBlock_Phoenix:TerminalBlock_Phoenix_MKDS-1,5-2-5.08_1x02_P5.08mm_Horizontal, F.Cu at (163.9, 30.2)
- added J4: COIL OUT, TerminalBlock_Phoenix:TerminalBlock_Phoenix_MKDS-1,5-2-5.08_1x02_P5.08mm_Horizontal, F.Cu at (-4.06, 72.8)
- added J4: COIL OUT, TerminalBlock_Phoenix:TerminalBlock_Phoenix_MKDS-1,5-2-5.08_1x02_P5.08mm_Horizontal, F.Cu at (107.9, 30.2)
- added J4: COIL OUT, TerminalBlock_Phoenix:TerminalBlock_Phoenix_MKDS-1,5-2-5.08_1x02_P5.08mm_Horizontal, F.Cu at (219.9, 158.0)
- added J4: COIL OUT, TerminalBlock_Phoenix:TerminalBlock_Phoenix_MKDS-1,5-2-5.08_1x02_P5.08mm_Horizontal, F.Cu at (275.9, 158.0)
- added J4: COIL OUT, TerminalBlock_Phoenix:TerminalBlock_Phoenix_MKDS-1,5-2-5.08_1x02_P5.08mm_Horizontal, F.Cu at (51.9, 72.8)
- added J4: COIL OUT, TerminalBlock_Phoenix:TerminalBlock_Phoenix_MKDS-1,5-2-5.08_1x02_P5.08mm_Horizontal, F.Cu at (-4.06, 30.2)
- added J4: COIL OUT, TerminalBlock_Phoenix:TerminalBlock_Phoenix_MKDS-1,5-2-5.08_1x02_P5.08mm_Horizontal, F.Cu at (219.9, 72.8)
- added J4: COIL OUT, TerminalBlock_Phoenix:TerminalBlock_Phoenix_MKDS-1,5-2-5.08_1x02_P5.08mm_Horizontal, F.Cu at (219.9, 115.4)
- added J4: COIL OUT, TerminalBlock_Phoenix:TerminalBlock_Phoenix_MKDS-1,5-2-5.08_1x02_P5.08mm_Horizontal, F.Cu at (275.9, 115.4)
- added J4: COIL OUT, TerminalBlock_Phoenix:TerminalBlock_Phoenix_MKDS-1,5-2-5.08_1x02_P5.08mm_Horizontal, F.Cu at (107.9, 158.0)
- added J4: COIL OUT, TerminalBlock_Phoenix:TerminalBlock_Phoenix_MKDS-1,5-2-5.08_1x02_P5.08mm_Horizontal, F.Cu at (163.9, 115.4)
- added J4: COIL OUT, TerminalBlock_Phoenix:TerminalBlock_Phoenix_MKDS-1,5-2-5.08_1x02_P5.08mm_Horizontal, F.Cu at (51.9, 158.0)
- added J4: COIL OUT, TerminalBlock_Phoenix:TerminalBlock_Phoenix_MKDS-1,5-2-5.08_1x02_P5.08mm_Horizontal, F.Cu at (163.9, 158.0)
- added J4: COIL OUT, TerminalBlock_Phoenix:TerminalBlock_Phoenix_MKDS-1,5-2-5.08_1x02_P5.08mm_Horizontal, F.Cu at (51.9, 30.2)
- added J4: COIL OUT, TerminalBlock_Phoenix:TerminalBlock_Phoenix_MKDS-1,5-2-5.08_1x02_P5.08mm_Horizontal, F.Cu at (275.9, 30.2)
- added J4: COIL OUT, TerminalBlock_Phoenix:TerminalBlock_Phoenix_MKDS-1,5-2-5.08_1x02_P5.08mm_Horizontal, F.Cu at (275.9, 72.8)
- added J4: COIL OUT, TerminalBlock_Phoenix:TerminalBlock_Phoenix_MKDS-1,5-2-5.08_1x02_P5.08mm_Horizontal, F.Cu at (107.9, 115.4)
- added J4: COIL OUT, TerminalBlock_Phoenix:TerminalBlock_Phoenix_MKDS-1,5-2-5.08_1x02_P5.08mm_Horizontal, F.Cu at (51.9, 115.4)
- added J4: COIL OUT, TerminalBlock_Phoenix:TerminalBlock_Phoenix_MKDS-1,5-2-5.08_1x02_P5.08mm_Horizontal, F.Cu at (219.9, 30.2)
- added J4: COIL OUT, TerminalBlock_Phoenix:TerminalBlock_Phoenix_MKDS-1,5-2-5.08_1x02_P5.08mm_Horizontal, F.Cu at (-4.06, 158.0)
- added J4: COIL OUT, TerminalBlock_Phoenix:TerminalBlock_Phoenix_MKDS-1,5-2-5.08_1x02_P5.08mm_Horizontal, F.Cu at (163.9, 72.8)
- added J5: COIL POWER IN, TerminalBlock_Phoenix:TerminalBlock_Phoenix_MKDS-1,5-2-5.08_1x02_P5.08mm_Horizontal, F.Cu at (210.3, 42.5)
- added J5: COIL POWER IN, TerminalBlock_Phoenix:TerminalBlock_Phoenix_MKDS-1,5-2-5.08_1x02_P5.08mm_Horizontal, F.Cu at (154.3, 170.3)
- added J5: COIL POWER IN, TerminalBlock_Phoenix:TerminalBlock_Phoenix_MKDS-1,5-2-5.08_1x02_P5.08mm_Horizontal, F.Cu at (210.3, 85.1)
- added J5: COIL POWER IN, TerminalBlock_Phoenix:TerminalBlock_Phoenix_MKDS-1,5-2-5.08_1x02_P5.08mm_Horizontal, F.Cu at (154.3, 127.7)
- added J5: COIL POWER IN, TerminalBlock_Phoenix:TerminalBlock_Phoenix_MKDS-1,5-2-5.08_1x02_P5.08mm_Horizontal, F.Cu at (98.3, 42.5)
- added J5: COIL POWER IN, TerminalBlock_Phoenix:TerminalBlock_Phoenix_MKDS-1,5-2-5.08_1x02_P5.08mm_Horizontal, F.Cu at (266.3, 170.3)
- added J5: COIL POWER IN, TerminalBlock_Phoenix:TerminalBlock_Phoenix_MKDS-1,5-2-5.08_1x02_P5.08mm_Horizontal, F.Cu at (154.3, 42.5)
- added J5: COIL POWER IN, TerminalBlock_Phoenix:TerminalBlock_Phoenix_MKDS-1,5-2-5.08_1x02_P5.08mm_Horizontal, F.Cu at (266.3, 85.1)
- added J5: COIL POWER IN, TerminalBlock_Phoenix:TerminalBlock_Phoenix_MKDS-1,5-2-5.08_1x02_P5.08mm_Horizontal, F.Cu at (42.3, 127.7)
- added J5: COIL POWER IN, TerminalBlock_Phoenix:TerminalBlock_Phoenix_MKDS-1,5-2-5.08_1x02_P5.08mm_Horizontal, F.Cu at (266.3, 42.5)
- added J5: COIL POWER IN, TerminalBlock_Phoenix:TerminalBlock_Phoenix_MKDS-1,5-2-5.08_1x02_P5.08mm_Horizontal, F.Cu at (98.3, 170.3)
- added J5: COIL POWER IN, TerminalBlock_Phoenix:TerminalBlock_Phoenix_MKDS-1,5-2-5.08_1x02_P5.08mm_Horizontal, F.Cu at (154.3, 85.1)
- added J5: COIL POWER IN, TerminalBlock_Phoenix:TerminalBlock_Phoenix_MKDS-1,5-2-5.08_1x02_P5.08mm_Horizontal, F.Cu at (266.3, 127.7)
- added J5: COIL POWER IN, TerminalBlock_Phoenix:TerminalBlock_Phoenix_MKDS-1,5-2-5.08_1x02_P5.08mm_Horizontal, F.Cu at (210.3, 127.7)
- added J5: COIL POWER IN, TerminalBlock_Phoenix:TerminalBlock_Phoenix_MKDS-1,5-2-5.08_1x02_P5.08mm_Horizontal, F.Cu at (-13.7, 170.3)
- added J5: COIL POWER IN, TerminalBlock_Phoenix:TerminalBlock_Phoenix_MKDS-1,5-2-5.08_1x02_P5.08mm_Horizontal, F.Cu at (42.3, 170.3)
- added J5: COIL POWER IN, TerminalBlock_Phoenix:TerminalBlock_Phoenix_MKDS-1,5-2-5.08_1x02_P5.08mm_Horizontal, F.Cu at (42.3, 42.5)
- added J5: COIL POWER IN, TerminalBlock_Phoenix:TerminalBlock_Phoenix_MKDS-1,5-2-5.08_1x02_P5.08mm_Horizontal, F.Cu at (-13.7, 42.5)
- added J5: COIL POWER IN, TerminalBlock_Phoenix:TerminalBlock_Phoenix_MKDS-1,5-2-5.08_1x02_P5.08mm_Horizontal, F.Cu at (210.3, 170.3)
- added J5: COIL POWER IN, TerminalBlock_Phoenix:TerminalBlock_Phoenix_MKDS-1,5-2-5.08_1x02_P5.08mm_Horizontal, F.Cu at (-13.7, 127.7)
- added J5: COIL POWER IN, TerminalBlock_Phoenix:TerminalBlock_Phoenix_MKDS-1,5-2-5.08_1x02_P5.08mm_Horizontal, F.Cu at (-13.7, 85.1)
- added J5: COIL POWER IN, TerminalBlock_Phoenix:TerminalBlock_Phoenix_MKDS-1,5-2-5.08_1x02_P5.08mm_Horizontal, F.Cu at (42.3, 85.1)
- added J5: COIL POWER IN, TerminalBlock_Phoenix:TerminalBlock_Phoenix_MKDS-1,5-2-5.08_1x02_P5.08mm_Horizontal, F.Cu at (98.3, 85.1)
- added J5: COIL POWER IN, TerminalBlock_Phoenix:TerminalBlock_Phoenix_MKDS-1,5-2-5.08_1x02_P5.08mm_Horizontal, F.Cu at (98.3, 127.7)
- added Q1: IRF3205, IMRANS_LIBRARY:TO-220-3_Vertical, F.Cu at (2.90, 40.8)
- added Q1: IRF3205, IMRANS_LIBRARY:TO-220-3_Vertical, F.Cu at (114.9, 40.8)
- added Q1: IRF3205, IMRANS_LIBRARY:TO-220-3_Vertical, F.Cu at (170.9, 168.6)
- added Q1: IRF3205, IMRANS_LIBRARY:TO-220-3_Vertical, F.Cu at (2.90, 168.6)
- added Q1: IRF3205, IMRANS_LIBRARY:TO-220-3_Vertical, F.Cu at (58.9, 40.8)
- added Q1: IRF3205, IMRANS_LIBRARY:TO-220-3_Vertical, F.Cu at (226.9, 168.6)
- added Q1: IRF3205, IMRANS_LIBRARY:TO-220-3_Vertical, F.Cu at (226.9, 40.8)
- added Q1: IRF3205, IMRANS_LIBRARY:TO-220-3_Vertical, F.Cu at (226.9, 126.0)
- added Q1: IRF3205, IMRANS_LIBRARY:TO-220-3_Vertical, F.Cu at (114.9, 83.4)
- added Q1: IRF3205, IMRANS_LIBRARY:TO-220-3_Vertical, F.Cu at (170.9, 40.8)
- added Q1: IRF3205, IMRANS_LIBRARY:TO-220-3_Vertical, F.Cu at (170.9, 126.0)
- added Q1: IRF3205, IMRANS_LIBRARY:TO-220-3_Vertical, F.Cu at (282.9, 168.6)
- added Q1: IRF3205, IMRANS_LIBRARY:TO-220-3_Vertical, F.Cu at (282.9, 40.8)
- added Q1: IRF3205, IMRANS_LIBRARY:TO-220-3_Vertical, F.Cu at (58.9, 126.0)
- added Q1: IRF3205, IMRANS_LIBRARY:TO-220-3_Vertical, F.Cu at (58.9, 83.4)
- added Q1: IRF3205, IMRANS_LIBRARY:TO-220-3_Vertical, F.Cu at (226.9, 83.4)
- added Q1: IRF3205, IMRANS_LIBRARY:TO-220-3_Vertical, F.Cu at (58.9, 168.6)
- added Q1: IRF3205, IMRANS_LIBRARY:TO-220-3_Vertical, F.Cu at (282.9, 126.0)
- added Q1: IRF3205, IMRANS_LIBRARY:TO-220-3_Vertical, F.Cu at (2.90, 83.4)
- added Q1: IRF3205, IMRANS_LIBRARY:TO-220-3_Vertical, F.Cu at (114.9, 168.6)
- added Q1: IRF3205, IMRANS_LIBRARY:TO-220-3_Vertical, F.Cu at (282.9, 83.4)
- added Q1: IRF3205, IMRANS_LIBRARY:TO-220-3_Vertical, F.Cu at (2.90, 126.0)
- added Q1: IRF3205, IMRANS_LIBRARY:TO-220-3_Vertical, F.Cu at (114.9, 126.0)
- added Q1: IRF3205, IMRANS_LIBRARY:TO-220-3_Vertical, F.Cu at (170.9, 83.4)
- added R1: 10k, IMRANS_LIBRARY:R_Axial_DIN0207_L6.3mm_D2.5mm_P10.16mm_Horizontal_2, F.Cu at (127.4, 168.2)
- added R1: 10k, IMRANS_LIBRARY:R_Axial_DIN0207_L6.3mm_D2.5mm_P10.16mm_Horizontal_2, F.Cu at (183.4, 40.4)
- added R1: 10k, IMRANS_LIBRARY:R_Axial_DIN0207_L6.3mm_D2.5mm_P10.16mm_Horizontal_2, F.Cu at (71.4, 125.6)
- added R1: 10k, IMRANS_LIBRARY:R_Axial_DIN0207_L6.3mm_D2.5mm_P10.16mm_Horizontal_2, F.Cu at (295.4, 125.6)
- added R1: 10k, IMRANS_LIBRARY:R_Axial_DIN0207_L6.3mm_D2.5mm_P10.16mm_Horizontal_2, F.Cu at (15.4, 168.2)
- added R1: 10k, IMRANS_LIBRARY:R_Axial_DIN0207_L6.3mm_D2.5mm_P10.16mm_Horizontal_2, F.Cu at (71.4, 40.4)
- added R1: 10k, IMRANS_LIBRARY:R_Axial_DIN0207_L6.3mm_D2.5mm_P10.16mm_Horizontal_2, F.Cu at (295.4, 83.0)
- added R1: 10k, IMRANS_LIBRARY:R_Axial_DIN0207_L6.3mm_D2.5mm_P10.16mm_Horizontal_2, F.Cu at (71.4, 83.0)
- added R1: 10k, IMRANS_LIBRARY:R_Axial_DIN0207_L6.3mm_D2.5mm_P10.16mm_Horizontal_2, F.Cu at (295.4, 40.4)
- added R1: 10k, IMRANS_LIBRARY:R_Axial_DIN0207_L6.3mm_D2.5mm_P10.16mm_Horizontal_2, F.Cu at (127.4, 125.6)
- added R1: 10k, IMRANS_LIBRARY:R_Axial_DIN0207_L6.3mm_D2.5mm_P10.16mm_Horizontal_2, F.Cu at (183.4, 83.0)
- added R1: 10k, IMRANS_LIBRARY:R_Axial_DIN0207_L6.3mm_D2.5mm_P10.16mm_Horizontal_2, F.Cu at (239.4, 168.2)
- added R1: 10k, IMRANS_LIBRARY:R_Axial_DIN0207_L6.3mm_D2.5mm_P10.16mm_Horizontal_2, F.Cu at (127.4, 83.0)
- added R1: 10k, IMRANS_LIBRARY:R_Axial_DIN0207_L6.3mm_D2.5mm_P10.16mm_Horizontal_2, F.Cu at (239.4, 83.0)
- added R1: 10k, IMRANS_LIBRARY:R_Axial_DIN0207_L6.3mm_D2.5mm_P10.16mm_Horizontal_2, F.Cu at (71.4, 168.2)
- added R1: 10k, IMRANS_LIBRARY:R_Axial_DIN0207_L6.3mm_D2.5mm_P10.16mm_Horizontal_2, F.Cu at (183.4, 168.2)
- added R1: 10k, IMRANS_LIBRARY:R_Axial_DIN0207_L6.3mm_D2.5mm_P10.16mm_Horizontal_2, F.Cu at (15.4, 40.4)
- added R1: 10k, IMRANS_LIBRARY:R_Axial_DIN0207_L6.3mm_D2.5mm_P10.16mm_Horizontal_2, F.Cu at (15.4, 125.6)
- added R1: 10k, IMRANS_LIBRARY:R_Axial_DIN0207_L6.3mm_D2.5mm_P10.16mm_Horizontal_2, F.Cu at (239.4, 125.6)
- added R1: 10k, IMRANS_LIBRARY:R_Axial_DIN0207_L6.3mm_D2.5mm_P10.16mm_Horizontal_2, F.Cu at (127.4, 40.4)
- added R1: 10k, IMRANS_LIBRARY:R_Axial_DIN0207_L6.3mm_D2.5mm_P10.16mm_Horizontal_2, F.Cu at (239.4, 40.4)
- added R1: 10k, IMRANS_LIBRARY:R_Axial_DIN0207_L6.3mm_D2.5mm_P10.16mm_Horizontal_2, F.Cu at (295.4, 168.2)
- added R1: 10k, IMRANS_LIBRARY:R_Axial_DIN0207_L6.3mm_D2.5mm_P10.16mm_Horizontal_2, F.Cu at (15.4, 83.0)
- added R1: 10k, IMRANS_LIBRARY:R_Axial_DIN0207_L6.3mm_D2.5mm_P10.16mm_Horizontal_2, F.Cu at (183.4, 125.6)
- added R2: 10k, IMRANS_LIBRARY:Potentiometer_Bourns_3386P_Vertical, F.Cu at (16.1, 174.4)
- added R2: 10k, IMRANS_LIBRARY:Potentiometer_Bourns_3386P_Vertical, F.Cu at (72.1, 131.8)
- added R2: 10k, IMRANS_LIBRARY:Potentiometer_Bourns_3386P_Vertical, F.Cu at (16.1, 131.8)
- added R2: 10k, IMRANS_LIBRARY:Potentiometer_Bourns_3386P_Vertical, F.Cu at (16.1, 89.2)
- added R2: 10k, IMRANS_LIBRARY:Potentiometer_Bourns_3386P_Vertical, F.Cu at (72.1, 174.4)
- added R2: 10k, IMRANS_LIBRARY:Potentiometer_Bourns_3386P_Vertical, F.Cu at (240.1, 174.4)
- added R2: 10k, IMRANS_LIBRARY:Potentiometer_Bourns_3386P_Vertical, F.Cu at (296.1, 174.4)
- added R2: 10k, IMRANS_LIBRARY:Potentiometer_Bourns_3386P_Vertical, F.Cu at (240.1, 131.8)
- added R2: 10k, IMRANS_LIBRARY:Potentiometer_Bourns_3386P_Vertical, F.Cu at (240.1, 89.2)
- added R2: 10k, IMRANS_LIBRARY:Potentiometer_Bourns_3386P_Vertical, F.Cu at (296.1, 46.6)
- added R2: 10k, IMRANS_LIBRARY:Potentiometer_Bourns_3386P_Vertical, F.Cu at (296.1, 89.2)
- added R2: 10k, IMRANS_LIBRARY:Potentiometer_Bourns_3386P_Vertical, F.Cu at (128.1, 131.8)
- added R2: 10k, IMRANS_LIBRARY:Potentiometer_Bourns_3386P_Vertical, F.Cu at (184.1, 131.8)
- added R2: 10k, IMRANS_LIBRARY:Potentiometer_Bourns_3386P_Vertical, F.Cu at (72.1, 46.6)
- added R2: 10k, IMRANS_LIBRARY:Potentiometer_Bourns_3386P_Vertical, F.Cu at (128.1, 89.2)
- added R2: 10k, IMRANS_LIBRARY:Potentiometer_Bourns_3386P_Vertical, F.Cu at (296.1, 131.8)
- added R2: 10k, IMRANS_LIBRARY:Potentiometer_Bourns_3386P_Vertical, F.Cu at (240.1, 46.6)
- added R2: 10k, IMRANS_LIBRARY:Potentiometer_Bourns_3386P_Vertical, F.Cu at (184.1, 89.2)
- added R2: 10k, IMRANS_LIBRARY:Potentiometer_Bourns_3386P_Vertical, F.Cu at (184.1, 46.6)
- added R2: 10k, IMRANS_LIBRARY:Potentiometer_Bourns_3386P_Vertical, F.Cu at (128.1, 174.4)
- added R2: 10k, IMRANS_LIBRARY:Potentiometer_Bourns_3386P_Vertical, F.Cu at (128.1, 46.6)
- added R2: 10k, IMRANS_LIBRARY:Potentiometer_Bourns_3386P_Vertical, F.Cu at (16.1, 46.6)
- added R2: 10k, IMRANS_LIBRARY:Potentiometer_Bourns_3386P_Vertical, F.Cu at (72.1, 89.2)
- added R2: 10k, IMRANS_LIBRARY:Potentiometer_Bourns_3386P_Vertical, F.Cu at (184.1, 174.4)
- added R3: 6.8K, IMRANS_LIBRARY:R_Axial_DIN0207_L6.3mm_D2.5mm_P10.16mm_Horizontal_2, F.Cu at (-5.92, 140.3)
- added R3: 6.8K, IMRANS_LIBRARY:R_Axial_DIN0207_L6.3mm_D2.5mm_P10.16mm_Horizontal_2, F.Cu at (-5.92, 55.1)
- added R3: 6.8K, IMRANS_LIBRARY:R_Axial_DIN0207_L6.3mm_D2.5mm_P10.16mm_Horizontal_2, F.Cu at (50.1, 97.7)
- added R3: 6.8K, IMRANS_LIBRARY:R_Axial_DIN0207_L6.3mm_D2.5mm_P10.16mm_Horizontal_2, F.Cu at (274.1, 140.3)
- added R3: 6.8K, IMRANS_LIBRARY:R_Axial_DIN0207_L6.3mm_D2.5mm_P10.16mm_Horizontal_2, F.Cu at (162.1, 97.7)
- added R3: 6.8K, IMRANS_LIBRARY:R_Axial_DIN0207_L6.3mm_D2.5mm_P10.16mm_Horizontal_2, F.Cu at (218.1, 182.9)
- added R3: 6.8K, IMRANS_LIBRARY:R_Axial_DIN0207_L6.3mm_D2.5mm_P10.16mm_Horizontal_2, F.Cu at (-5.92, 182.9)
- added R3: 6.8K, IMRANS_LIBRARY:R_Axial_DIN0207_L6.3mm_D2.5mm_P10.16mm_Horizontal_2, F.Cu at (274.1, 97.7)
- added R3: 6.8K, IMRANS_LIBRARY:R_Axial_DIN0207_L6.3mm_D2.5mm_P10.16mm_Horizontal_2, F.Cu at (218.1, 140.3)
- added R3: 6.8K, IMRANS_LIBRARY:R_Axial_DIN0207_L6.3mm_D2.5mm_P10.16mm_Horizontal_2, F.Cu at (50.1, 182.9)
- added R3: 6.8K, IMRANS_LIBRARY:R_Axial_DIN0207_L6.3mm_D2.5mm_P10.16mm_Horizontal_2, F.Cu at (-5.92, 97.7)
- added R3: 6.8K, IMRANS_LIBRARY:R_Axial_DIN0207_L6.3mm_D2.5mm_P10.16mm_Horizontal_2, F.Cu at (106.1, 55.1)
- added R3: 6.8K, IMRANS_LIBRARY:R_Axial_DIN0207_L6.3mm_D2.5mm_P10.16mm_Horizontal_2, F.Cu at (162.1, 55.1)
- added R3: 6.8K, IMRANS_LIBRARY:R_Axial_DIN0207_L6.3mm_D2.5mm_P10.16mm_Horizontal_2, F.Cu at (106.1, 97.7)
- added R3: 6.8K, IMRANS_LIBRARY:R_Axial_DIN0207_L6.3mm_D2.5mm_P10.16mm_Horizontal_2, F.Cu at (162.1, 140.3)
- added R3: 6.8K, IMRANS_LIBRARY:R_Axial_DIN0207_L6.3mm_D2.5mm_P10.16mm_Horizontal_2, F.Cu at (50.1, 140.3)
- added R3: 6.8K, IMRANS_LIBRARY:R_Axial_DIN0207_L6.3mm_D2.5mm_P10.16mm_Horizontal_2, F.Cu at (106.1, 140.3)
- added R3: 6.8K, IMRANS_LIBRARY:R_Axial_DIN0207_L6.3mm_D2.5mm_P10.16mm_Horizontal_2, F.Cu at (274.1, 182.9)
- added R3: 6.8K, IMRANS_LIBRARY:R_Axial_DIN0207_L6.3mm_D2.5mm_P10.16mm_Horizontal_2, F.Cu at (50.1, 55.1)
- added R3: 6.8K, IMRANS_LIBRARY:R_Axial_DIN0207_L6.3mm_D2.5mm_P10.16mm_Horizontal_2, F.Cu at (162.1, 182.9)
- added R3: 6.8K, IMRANS_LIBRARY:R_Axial_DIN0207_L6.3mm_D2.5mm_P10.16mm_Horizontal_2, F.Cu at (106.1, 182.9)
- added R3: 6.8K, IMRANS_LIBRARY:R_Axial_DIN0207_L6.3mm_D2.5mm_P10.16mm_Horizontal_2, F.Cu at (218.1, 55.1)
- added R3: 6.8K, IMRANS_LIBRARY:R_Axial_DIN0207_L6.3mm_D2.5mm_P10.16mm_Horizontal_2, F.Cu at (274.1, 55.1)
- added R3: 6.8K, IMRANS_LIBRARY:R_Axial_DIN0207_L6.3mm_D2.5mm_P10.16mm_Horizontal_2, F.Cu at (218.1, 97.7)
- added R4: 47R, IMRANS_LIBRARY:R_Axial_DIN0207_L6.3mm_D2.5mm_P10.16mm_Horizontal_2, F.Cu at (162.0, 185.4)
- added R4: 47R, IMRANS_LIBRARY:R_Axial_DIN0207_L6.3mm_D2.5mm_P10.16mm_Horizontal_2, F.Cu at (274.0, 57.6)
- added R4: 47R, IMRANS_LIBRARY:R_Axial_DIN0207_L6.3mm_D2.5mm_P10.16mm_Horizontal_2, F.Cu at (218.0, 185.4)
- added R4: 47R, IMRANS_LIBRARY:R_Axial_DIN0207_L6.3mm_D2.5mm_P10.16mm_Horizontal_2, F.Cu at (162.0, 100.2)
- added R4: 47R, IMRANS_LIBRARY:R_Axial_DIN0207_L6.3mm_D2.5mm_P10.16mm_Horizontal_2, F.Cu at (162.0, 57.6)
- added R4: 47R, IMRANS_LIBRARY:R_Axial_DIN0207_L6.3mm_D2.5mm_P10.16mm_Horizontal_2, F.Cu at (106.0, 57.6)
- added R4: 47R, IMRANS_LIBRARY:R_Axial_DIN0207_L6.3mm_D2.5mm_P10.16mm_Horizontal_2, F.Cu at (106.0, 185.4)
- added R4: 47R, IMRANS_LIBRARY:R_Axial_DIN0207_L6.3mm_D2.5mm_P10.16mm_Horizontal_2, F.Cu at (50.0, 100.2)
- added R4: 47R, IMRANS_LIBRARY:R_Axial_DIN0207_L6.3mm_D2.5mm_P10.16mm_Horizontal_2, F.Cu at (106.0, 100.2)
- added R4: 47R, IMRANS_LIBRARY:R_Axial_DIN0207_L6.3mm_D2.5mm_P10.16mm_Horizontal_2, F.Cu at (106.0, 142.8)
- added R4: 47R, IMRANS_LIBRARY:R_Axial_DIN0207_L6.3mm_D2.5mm_P10.16mm_Horizontal_2, F.Cu at (-6.00, 185.4)
- added R4: 47R, IMRANS_LIBRARY:R_Axial_DIN0207_L6.3mm_D2.5mm_P10.16mm_Horizontal_2, F.Cu at (-6.00, 100.2)
- added R4: 47R, IMRANS_LIBRARY:R_Axial_DIN0207_L6.3mm_D2.5mm_P10.16mm_Horizontal_2, F.Cu at (218.0, 57.6)
- added R4: 47R, IMRANS_LIBRARY:R_Axial_DIN0207_L6.3mm_D2.5mm_P10.16mm_Horizontal_2, F.Cu at (-6.00, 57.6)
- added R4: 47R, IMRANS_LIBRARY:R_Axial_DIN0207_L6.3mm_D2.5mm_P10.16mm_Horizontal_2, F.Cu at (274.0, 185.4)
- added R4: 47R, IMRANS_LIBRARY:R_Axial_DIN0207_L6.3mm_D2.5mm_P10.16mm_Horizontal_2, F.Cu at (218.0, 142.8)
- added R4: 47R, IMRANS_LIBRARY:R_Axial_DIN0207_L6.3mm_D2.5mm_P10.16mm_Horizontal_2, F.Cu at (218.0, 100.2)
- added R4: 47R, IMRANS_LIBRARY:R_Axial_DIN0207_L6.3mm_D2.5mm_P10.16mm_Horizontal_2, F.Cu at (162.0, 142.8)
- added R4: 47R, IMRANS_LIBRARY:R_Axial_DIN0207_L6.3mm_D2.5mm_P10.16mm_Horizontal_2, F.Cu at (50.0, 57.6)
- added R4: 47R, IMRANS_LIBRARY:R_Axial_DIN0207_L6.3mm_D2.5mm_P10.16mm_Horizontal_2, F.Cu at (274.0, 142.8)
- added R4: 47R, IMRANS_LIBRARY:R_Axial_DIN0207_L6.3mm_D2.5mm_P10.16mm_Horizontal_2, F.Cu at (-6.00, 142.8)
- added R4: 47R, IMRANS_LIBRARY:R_Axial_DIN0207_L6.3mm_D2.5mm_P10.16mm_Horizontal_2, F.Cu at (50.0, 185.4)
- added R4: 47R, IMRANS_LIBRARY:R_Axial_DIN0207_L6.3mm_D2.5mm_P10.16mm_Horizontal_2, F.Cu at (274.0, 100.2)
- added R4: 47R, IMRANS_LIBRARY:R_Axial_DIN0207_L6.3mm_D2.5mm_P10.16mm_Horizontal_2, F.Cu at (50.0, 142.8)
- added U1: LM358, Package_DIP:DIP-8_W7.62mm_Socket_LongPads, F.Cu at (248.2, 45.7)
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Routing:
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- added copper zone on B.Cu, net Board_16-GND
- added copper zone on B.Cu, net Board_17-GND
- added copper zone on B.Cu, net Board_18-GND
- added copper zone on B.Cu, net Board_19-GND
- added copper zone on B.Cu, net Board_20-GND
- added copper zone on B.Cu, net Board_21-GND
- added copper zone on B.Cu, net Board_22-GND
- added copper zone on B.Cu, net Board_23-GND
Other:
- board size 255 x 132.7 mm -> 335 x 169.4 mm
- board text added: "BOT"
- board text added: "SERVE"
- board text removed: "B.K DOCK"
- board text removed: "V1.1"
