File: mower/PCB/TRANSMITTER_DIP/TRANSMITTER.kicad_pcb (KiCad board)
At the start: 2 copper layers, 55 x 41.6 mm, 14 parts, among them J1 BOT POWER, J2 POWER IN, J3 SHUNT, J4 COIL OUT, J5 COIL POWER IN, Q1 IRF3205, U1 LM358, U4 LM555xN

Commit message: .
Parts:
- added C2: 100nF, IMRANS_LIBRARY:C_Disc_D3.0mm_W1.6mm_P2.50mm, F.Cu at (104.0, 63.6)
- added R5: 1K, IMRANS_LIBRARY:R_Axial_DIN0207_L6.3mm_D2.5mm_P10.16mm_Horizontal_2, F.Cu at (128.6, 49.5)
- D1: value 1N5819 -> 1N4007
- R1: value 10k -> 10K
- R2: value 10k -> 10K; footprint IMRANS_LIBRARY:Potentiometer_Bourns_3386P_Vertical -> IMRANS_LIBRARY:R_Axial_DIN0207_L6.3mm_D2.5mm_P10.16mm_Horizontal_2
- moved J5 18.9 mm to (117.5, 41.3), turned to 180 degrees
- moved Q1 16.3 mm to (108.4, 58.8), turned to 90 degrees
- moved U1 13.6 mm to (136.4, 50.7)
- moved R1 13.1 mm to (148.9, 50.0), turned to -90 degrees
- moved D1 12.3 mm to (98.5, 48.8)
- moved J4 11.9 mm to (106.2, 41.3)
- moved R4 9.19 mm to (112.0, 64.1), turned to 90 degrees
- moved R3 8.46 mm to (115.5, 61.6)
- moved U4 8.46 mm to (118.9, 53.3)
- moved C1 8.13 mm to (130.4, 58.6), turned to -90 degrees
- moved R2 8.04 mm to (145.6, 62.1)
- moved J1 3.86 mm to (128.9, 41.3)
- moved J2 3.86 mm to (151.9, 41.4)
- moved J3 3.86 mm to (140.3, 41.3)
Connections:
- J2 pad 1: VCC -> GND
- J2 pad 2: GND -> VCC
- R1 pad 2: Net-(U1A--) -> Net-(U1B-+)
- R2 pad 1: Net-(U1A--) -> Net-(U1B-+)
- U1 pad 1: Net-(U4-R) -> Net-(U1B--)
- U1 pad 2: Net-(U1A--) -> Net-(J1-Pin_1)
- U1 pad 3: Net-(J1-Pin_1) -> GND
- U1 pad 4: GND -> unconnected-(U1C-V--Pad4)
- U1 pad 5: (no net) -> Net-(U1B-+)
- U1 pad 6: (no net) -> Net-(U1B--)
- U1 pad 7: (no net) -> Net-(U4-R)
- U1 pad 8: VCC -> unconnected-(U1C-V+-Pad8)
Routing:
- net VCC: track 79.1 -> 57.0 mm, vias 0 -> 2
- net Net-(U1A--): track 18.9 -> 0.00 mm
- net VCOIL: track 14.2 -> 29.3 mm
- net Net-(D1-A): track 20.3 -> 34.2 mm
- net Net-(Q1-G): track 34.0 -> 21.2 mm
- net Net-(J1-Pin_1): track 38.0 -> 27.0 mm, vias 2 -> 0
- net Net-(U1B--): track 0.00 -> 10.8 mm
- net Net-(U1B-+): track 0.00 -> 8.86 mm
- net Net-(U4-R): track 43.6 -> 51.8 mm
- net GND: track 0.00 -> 7.19 mm
- net Net-(U4-Q): track 8.82 -> 5.56 mm
- net Net-(U4-THR): track 20.6 -> 19.8 mm
Other:
- board size 55 x 41.6 mm -> 63 x 32.8 mm
- board text added: "B.K DOCK"
- board text added: "V1.1"
- board text removed: "BOT"
- board text removed: "SERVE"

Commit message: .
Parts:
- moved C2 0.45 mm to (103.6, 63.4), turned to 180 degrees
Connections:
- U1 pad 4: unconnected-(U1C-V--Pad4) -> GND
- U1 pad 8: unconnected-(U1C-V+-Pad8) -> VCC
Routing:
- net Net-(U4-Q): track 5.56 -> 10.1 mm
- net VCC: track 57.0 -> 60.5 mm
- net Net-(D1-A): track 34.2 -> 33.6 mm
Changed lines of the file:
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@@
 	(net 12 "Net-(U1B-+)")
 	(net 13 "Net-(U1B--)")
-	(net 14 "unconnected-(U1C-V--Pad4)")
-	(net 15 "unconnected-(U1C-V+-Pad8)")
 	(footprint "IMRANS_LIBRARY:TO-220-3_Vertical"
 		(layer "F.Cu")
@@
 			(layers "*.Cu" "*.Mask")
 			(remove_unused_layers no)
-			(net 14 "unconnected-(U1C-V--Pad4)")
+			(net 2 "GND")
 			(pinfunction "V-")
 			(pintype "power_in")
@@
 			(layers "*.Cu" "*.Mask")
 			(remove_unused_layers no)
-			(net 15 "unconnected-(U1C-V+-Pad8)")
+			(net 4 "VCC")
 			(pinfunction "V+")
 			(pintype "power_in")
@@
 	(footprint "IMRANS_LIBRARY:C_Disc_D3.0mm_W1.6mm_P2.50mm"
 		(layer "F.Cu")
-		(at 104 63.6)
+		(at 103.6 63.4 180)
 		(descr "C, Disc series, Radial, pin pitch=2.50mm, diameter*width=3.0*1.6mm^2, Capacitor, http://www.vishay.com/docs/45233/krseries.pdf")
 		(tags "C Disc series Radial pin pitch 2.50mm diameter 3.0mm width 1.6mm Capacitor")
@@
 		(attr through_hole)
 		(fp_line
-			(start 0.485 -0.92)
-			(end 2.015 -0.92)
+			(start 0.485 0.92)
+			(end 2.015 0.92)
 			(stroke
 				(width 0.12)
@@
 		)
 		(fp_line
-			(start 0.485 0.92)
-			(end 2.015 0.92)
+			(start 0.485 -0.92)
+			(end 2.015 -0.92)
 			(stroke
 				(width 0.12)
@@
 		)
 		(pad "1" thru_hole oval
-			(at 0.025 -0.025 90)
+			(at 0.025 -0.025 270)
 			(size 3 1.5)
 			(drill 0.8)
@@
 		)
 		(pad "2" thru_hole oval
-			(at 2.525 0.025 90)
+			(at 2.525 0.025 270)
 			(size 3 1.5)
 			(drill 0.8)
@@
 	)
 	(gr_text "B.K DOCK"
-		(at 99 66 90)
+		(at 98.2 51.2 90)
 		(layer "B.Cu" knockout)
 		(effects
 			(font
 				(size 2 2)
-				(thickness 0.4)
+				(thickness 0.5)
 				(bold yes)
 			)
-			(justify left bottom)
+			(justify left bottom mirror)
 		)
 	)
 	(gr_text "V1.1"
-		(at 155.2 52.2 90)
+		(at 155.2 45.2 90)
 		(layer "B.Cu" knockout)
 		(effects
 			(font
 				(size 2 2)
-				(thickness 0.4)
+				(thickness 0.5)
 				(bold yes)
 			)
-			(justify left bottom)
+			(justify left bottom mirror)
 		)
 	)
@@
 	)
 	(segment
+		(start 143.6 47.4)
+		(end 143.6 50.3)
+		(width 0.8)
+		(layer "B.Cu")
+		(net 4)
+	)
+	(segment
+		(start 143.6 50.3)
+		(end 144.02 50.72)
+		(width 0.8)
+		(layer "B.Cu")
+		(net 4)
+	)
+	(segment
 		(start 146.835 46.34)
 		(end 146.835 41.3675)
@@
 	)
 	(segment
-		(start 104.525 56.275)
-		(end 103.2 57.6)
-		(width 0.8)
+		(start 106.155 41.34)
+		(end 106.155 46.355)
+		(width 1.2)
 		(layer "B.Cu")
 		(net 5)
 	)
 	(segment
-		(start 106.155 41.34)
-		(end 106.155 46.355)
-		(width 1.2)
+		(start 103.575 63.425)
+		(end 103.575 57.225)
+		(width 0.8)
 		(layer "B.Cu")
 		(net 5)
@@
 	)
 	(segment
-		(start 103.2 57.6)
-		(end 103.2 61.6)
-		(width 0.8)
-		(layer "B.Cu")
-		(net 5)
-	)
-	(segment
-		(start 104.025 62.425)
-		(end 104.025 63.575)
+		(start 103.575 57.225)
+		(end 104.525 56.275)
 		(width 0.8)
 		(layer "B.Cu")
@@
 	)
 	(segment
-		(start 103.2 61.6)
-		(end 104.025 62.425)
-		(width 0.8)
-		(layer "B.Cu")
-		(net 5)
-	)
-	(segment
 		(start 112.025 54.025)
 		(end 112.825 54.025)
@@
 	)
 	(segment
+		(start 112 63.6)
+		(end 114.2 61.4)
+		(width 0.8)
+		(layer "B.Cu")
+		(net 7)
+	)
+	(segment
 		(start 115.49 59.365)
 		(end 115.49 61.115)
@@
 		(width 0.8)
 		(layer "B.Cu")
+		(net 7)
+	)
+	(segment
+		(start 115.205 61.4)
+		(end 115.49 61.115)
+		(width 0.8)
+		(layer "B.Cu")
+		(net 7)
+	)
+	(segment
+		(start 114.2 61.4)
+		(end 115.205 61.4)
+		(width 0.8)
+		(layer "B.Cu")
