File: mower/PCB/EMF_SENSOR_DIP/EMF_SENSOR_PANEL.kicad_pcb (KiCad board)
At the start: 2 copper layers, 225.2 x 135 mm, 288 parts, among them J1 Conn_01x03_Pin, U1 LM358, U2 LM393

Commit message: Consolidate complete mower design (all branches) + zana repo structure
Mower fragments from every botkorp branch (mowbot3/4, TRANSMITTER_SMD,
IMRANS_LIBRARY) unioned into mower/. Adds legacy/opengro, README, .gitignore.
Sits on top of the preserved 13-commit mower history.

Co-Authored-By: Claude Opus 4.8 <noreply@anthropic.com>
Claude-Session: https://claude.ai/code/session_017QXBEryTihUadNUZqQzfmo
Parts:
- removed the C1 at (117.9, 37.8)
- removed the C1 at (42.5, 139.8)
- removed the C1 at (42.5, 105.8)
- removed the C1 at (117.9, 105.8)
- removed the C1 at (193.3, 139.8)
- removed the C1 at (42.5, 37.8)
- removed the C1 at (117.9, 139.8)
- removed the C1 at (193.3, 71.8)
- removed the C1 at (42.5, 71.8)
- removed the C1 at (117.9, 71.8)
- removed the C1 at (193.3, 37.8)
- removed the C1 at (193.3, 105.8)
- removed C2 (x12), C4 (x12): 10uF, IMRANS_LIBRARY:C_Disc_D3.0mm_W1.6mm_P2.50mm
- removed the C3 at (83.1, 111.8)
- removed the C3 at (233.9, 145.8)
- removed the C3 at (158.5, 77.8)
- removed the C3 at (233.9, 43.8)
- removed the C3 at (158.5, 111.8)
- removed the C3 at (158.5, 43.8)
- removed the C3 at (233.9, 77.8)
- removed the C3 at (158.5, 145.8)
- removed the C3 at (83.1, 77.8)
- removed the C3 at (233.9, 111.8)
- removed the C3 at (83.1, 43.8)
- removed the C3 at (83.1, 145.8)
- removed C5 (x12): 1nF, IMRANS_LIBRARY:C_Disc_D3.0mm_W1.6mm_P2.50mm
- removed C6 (x12): 0.01uF, IMRANS_LIBRARY:C_Disc_D3.0mm_W1.6mm_P2.50mm
- removed the D1 at (83.8, 40.8)
- removed the D1 at (159.2, 142.8)
- removed the D1 at (83.8, 142.8)
- removed the D1 at (83.8, 108.8)
- removed the D1 at (159.2, 40.8)
- removed the D1 at (159.2, 74.8)
- removed the D1 at (234.6, 74.8)
- removed the D1 at (234.6, 142.8)
- removed the D1 at (234.6, 108.8)
- removed the D1 at (83.8, 74.8)
- removed the D1 at (159.2, 108.8)
- removed the D1 at (234.6, 40.8)
- removed the D2 at (223.8, 101.4)
- removed the D2 at (73.0, 67.4)
- removed the D2 at (148.4, 135.4)
- removed the D2 at (73.0, 33.4)
- removed the D2 at (148.4, 33.4)
- removed the D2 at (223.8, 67.4)
- removed the D2 at (73.0, 101.4)
- removed the D2 at (148.4, 67.4)
- removed the D2 at (223.8, 135.4)
- removed the D2 at (73.0, 135.4)
- removed the D2 at (223.8, 33.4)
- removed the D2 at (148.4, 101.4)
- removed the J1 at (166.9, 27.4)
- removed the J1 at (242.3, 129.4)
- removed the J1 at (91.5, 27.4)
- removed the J1 at (166.9, 95.4)
- removed the J1 at (166.9, 61.4)
- removed the J1 at (242.3, 95.4)
- removed the J1 at (242.3, 27.4)
- removed the J1 at (91.5, 95.4)
- removed the J1 at (242.3, 61.4)
- removed the J1 at (91.5, 61.4)
- removed the J1 at (166.9, 129.4)
- removed the J1 at (91.5, 129.4)
- removed the L1 at (115.7, 146.4)
- removed the L1 at (191.1, 78.4)
- removed the L1 at (191.1, 146.4)
- removed the L1 at (115.7, 78.4)
- removed the L1 at (191.1, 44.4)
- removed the L1 at (191.1, 112.4)
- removed the L1 at (40.3, 78.4)
- removed the L1 at (115.7, 112.4)
- removed the L1 at (40.3, 146.4)
- removed the L1 at (40.3, 44.4)
- removed the L1 at (115.7, 44.4)
- removed the L1 at (40.3, 112.4)
- removed the R1 at (47.1, 48.4)
- removed the R1 at (122.5, 82.4)
- removed the R1 at (122.5, 48.4)
- removed the R1 at (122.5, 116.4)
- removed the R1 at (47.1, 116.4)
- removed the R1 at (197.9, 82.4)
- removed the R1 at (47.1, 150.4)
- removed the R1 at (47.1, 82.4)
- removed the R1 at (197.9, 116.4)
- removed the R1 at (197.9, 48.4)
- removed the R1 at (197.9, 150.4)
- removed the R1 at (122.5, 150.4)
- removed R10 (x12), R11 (x12): 10K, IMRANS_LIBRARY:R_Axial_DIN0207_L6.3mm_D2.5mm_P10.16mm_Horizontal_2
- removed R12 (x12): 100K, IMRANS_LIBRARY:R_Axial_DIN0207_L6.3mm_D2.5mm_P10.16mm_Horizontal_2
- removed the R2 at (73.0, 60.8)
- removed the R2 at (73.0, 94.8)
- removed the R2 at (223.8, 128.8)
- removed the R2 at (223.8, 94.8)
- removed the R2 at (148.4, 128.8)
- removed the R2 at (223.8, 60.8)
- removed the R2 at (73.0, 26.8)
- removed the R2 at (223.8, 26.8)
- removed the R2 at (73.0, 128.8)
- removed the R2 at (148.4, 60.8)
- removed the R2 at (148.4, 26.8)
- removed the R2 at (148.4, 94.8)
- removed the R3 at (115.1, 37.1)
- removed the R3 at (190.5, 37.1)
- removed the R3 at (115.1, 71.1)
- removed the R3 at (115.1, 139.1)
- removed the R3 at (190.5, 71.1)
- removed the R3 at (190.5, 105.1)
- removed the R3 at (190.5, 139.1)
- removed the R3 at (39.7, 139.1)
- removed the R3 at (39.7, 37.1)
- removed the R3 at (115.1, 105.1)
- removed the R3 at (39.7, 71.1)
- removed the R3 at (39.7, 105.1)
- removed the R4 at (127.3, 104.1)
- removed the R4 at (202.7, 138.1)
- removed the R4 at (51.9, 36.1)
- removed the R4 at (51.9, 104.1)
- removed the R4 at (127.3, 36.1)
- removed the R4 at (127.3, 138.1)
- removed the R4 at (51.9, 138.1)
- removed the R4 at (202.7, 36.1)
- removed the R4 at (127.3, 70.1)
- removed the R4 at (202.7, 104.1)
- removed the R4 at (202.7, 70.1)
- removed the R4 at (51.9, 70.1)
- removed the R5 at (123.9, 110.3)
- removed the R5 at (123.9, 76.3)
- removed the R5 at (199.3, 76.3)
- removed the R5 at (199.3, 42.3)
- removed the R5 at (48.5, 76.3)
- removed the R5 at (123.9, 144.3)
- removed the R5 at (199.3, 110.3)
- removed the R5 at (123.9, 42.3)
- removed the R5 at (199.3, 144.3)
- removed the R5 at (48.5, 110.3)
- removed the R5 at (48.5, 144.3)
- removed the R5 at (48.5, 42.3)
- removed the R6 at (234.4, 132.2)
- removed the R6 at (159.0, 30.2)
- removed the R6 at (159.0, 64.2)
- removed the R6 at (83.6, 132.2)
- removed the R6 at (234.4, 30.2)
- removed the R6 at (159.0, 98.2)
- removed the R6 at (83.6, 30.2)
- removed the R6 at (234.4, 98.2)
- removed the R6 at (83.6, 98.2)
- removed the R6 at (234.4, 64.2)
- removed the R6 at (83.6, 64.2)
- removed the R6 at (159.0, 132.2)
- removed the R7 at (197.9, 79.2)
- removed the R7 at (47.1, 113.2)
- removed the R7 at (197.9, 113.2)
- removed the R7 at (47.1, 79.2)
- removed the R7 at (122.5, 147.2)
- removed the R7 at (47.1, 147.2)
- removed the R7 at (47.1, 45.2)
- removed the R7 at (122.5, 113.2)
- removed the R7 at (197.9, 45.2)
- removed the R7 at (122.5, 79.2)
- removed the R7 at (197.9, 147.2)
- removed the R7 at (122.5, 45.2)
- removed R8 (x12): 1M, IMRANS_LIBRARY:R_Axial_DIN0207_L6.3mm_D2.5mm_P10.16mm_Horizontal_2
- removed the R9 at (73.0, 138.8)
- removed the R9 at (223.8, 138.8)
- removed the R9 at (73.0, 104.8)
- removed the R9 at (148.4, 36.8)
- removed the R9 at (148.4, 70.8)
- removed the R9 at (148.4, 104.8)
- removed the R9 at (223.8, 104.8)
- removed the R9 at (73.0, 70.8)
- removed the R9 at (223.8, 36.8)
- removed the R9 at (73.0, 36.8)
- removed the R9 at (148.4, 138.8)
- removed the R9 at (223.8, 70.8)
- removed the U1 at (55.9, 133.4)
- removed the U1 at (131.3, 99.4)
- removed the U1 at (55.9, 99.4)
- removed the U1 at (206.7, 133.4)
- removed the U1 at (206.7, 99.4)
- removed the U1 at (131.3, 65.4)
- removed the U1 at (55.9, 65.4)
- removed the U1 at (206.7, 31.4)
- removed the U1 at (131.3, 133.4)
- removed the U1 at (131.3, 31.4)
- removed the U1 at (55.9, 31.4)
- removed the U1 at (206.7, 65.4)
- removed U2 (x12): LM393, Package_DIP:DIP-8_W7.62mm_Socket_LongPads
- added C1: 100nF, IMRANS_LIBRARY:C_Disc_D3.0mm_W1.6mm_P2.50mm, F.Cu at (81.6, 151.0)
- added C1: 100nF, IMRANS_LIBRARY:C_Disc_D3.0mm_W1.6mm_P2.50mm, F.Cu at (40.6, 28.0)
- added C1: 100nF, IMRANS_LIBRARY:C_Disc_D3.0mm_W1.6mm_P2.50mm, F.Cu at (245.6, 28.0)
- added C1: 100nF, IMRANS_LIBRARY:C_Disc_D3.0mm_W1.6mm_P2.50mm, F.Cu at (122.6, 110.0)
- added C1: 100nF, IMRANS_LIBRARY:C_Disc_D3.0mm_W1.6mm_P2.50mm, F.Cu at (163.6, 110.0)
- added C1: 100nF, IMRANS_LIBRARY:C_Disc_D3.0mm_W1.6mm_P2.50mm, F.Cu at (40.6, 69.0)
- added C1: 100nF, IMRANS_LIBRARY:C_Disc_D3.0mm_W1.6mm_P2.50mm, F.Cu at (163.6, 69.0)
- added C1: 100nF, IMRANS_LIBRARY:C_Disc_D3.0mm_W1.6mm_P2.50mm, F.Cu at (40.6, 151.0)
- added C1: 100nF, IMRANS_LIBRARY:C_Disc_D3.0mm_W1.6mm_P2.50mm, F.Cu at (81.6, 69.0)
- added C1: 100nF, IMRANS_LIBRARY:C_Disc_D3.0mm_W1.6mm_P2.50mm, F.Cu at (163.6, 28.0)
- added C1: 100nF, IMRANS_LIBRARY:C_Disc_D3.0mm_W1.6mm_P2.50mm, F.Cu at (204.6, 110.0)
- added C1: 100nF, IMRANS_LIBRARY:C_Disc_D3.0mm_W1.6mm_P2.50mm, F.Cu at (122.6, 151.0)
- added C1: 100nF, IMRANS_LIBRARY:C_Disc_D3.0mm_W1.6mm_P2.50mm, F.Cu at (81.6, 28.0)
- added C1: 100nF, IMRANS_LIBRARY:C_Disc_D3.0mm_W1.6mm_P2.50mm, F.Cu at (245.6, 69.0)
- added C1: 100nF, IMRANS_LIBRARY:C_Disc_D3.0mm_W1.6mm_P2.50mm, F.Cu at (122.6, 69.0)
- added C1: 100nF, IMRANS_LIBRARY:C_Disc_D3.0mm_W1.6mm_P2.50mm, F.Cu at (81.6, 110.0)
- added C1: 100nF, IMRANS_LIBRARY:C_Disc_D3.0mm_W1.6mm_P2.50mm, F.Cu at (122.6, 28.0)
- added C1: 100nF, IMRANS_LIBRARY:C_Disc_D3.0mm_W1.6mm_P2.50mm, F.Cu at (204.6, 28.0)
- added C1: 100nF, IMRANS_LIBRARY:C_Disc_D3.0mm_W1.6mm_P2.50mm, F.Cu at (204.6, 151.0)
- added C1: 100nF, IMRANS_LIBRARY:C_Disc_D3.0mm_W1.6mm_P2.50mm, F.Cu at (245.6, 151.0)
- added C1: 100nF, IMRANS_LIBRARY:C_Disc_D3.0mm_W1.6mm_P2.50mm, F.Cu at (40.6, 110.0)
- added C1: 100nF, IMRANS_LIBRARY:C_Disc_D3.0mm_W1.6mm_P2.50mm, F.Cu at (204.6, 69.0)
- added C1: 100nF, IMRANS_LIBRARY:C_Disc_D3.0mm_W1.6mm_P2.50mm, F.Cu at (163.6, 151.0)
- added C1: 100nF, IMRANS_LIBRARY:C_Disc_D3.0mm_W1.6mm_P2.50mm, F.Cu at (245.6, 110.0)
- added C3: 100nF (104), IMRANS_LIBRARY:C_Disc_D3.0mm_W1.6mm_P2.50mm, F.Cu at (143.8, 106.8)
- added C3: 100nF (104), IMRANS_LIBRARY:C_Disc_D3.0mm_W1.6mm_P2.50mm, F.Cu at (225.8, 24.8)
- added C3: 100nF (104), IMRANS_LIBRARY:C_Disc_D3.0mm_W1.6mm_P2.50mm, F.Cu at (266.8, 106.8)
- added C3: 100nF (104), IMRANS_LIBRARY:C_Disc_D3.0mm_W1.6mm_P2.50mm, F.Cu at (61.8, 24.8)
- added C3: 100nF (104), IMRANS_LIBRARY:C_Disc_D3.0mm_W1.6mm_P2.50mm, F.Cu at (102.8, 106.8)
- added C3: 100nF (104), IMRANS_LIBRARY:C_Disc_D3.0mm_W1.6mm_P2.50mm, F.Cu at (225.8, 147.8)
- added C3: 100nF (104), IMRANS_LIBRARY:C_Disc_D3.0mm_W1.6mm_P2.50mm, F.Cu at (143.8, 65.8)
- added C3: 100nF (104), IMRANS_LIBRARY:C_Disc_D3.0mm_W1.6mm_P2.50mm, F.Cu at (61.8, 147.8)
- added C3: 100nF (104), IMRANS_LIBRARY:C_Disc_D3.0mm_W1.6mm_P2.50mm, F.Cu at (225.8, 65.8)
- added C3: 100nF (104), IMRANS_LIBRARY:C_Disc_D3.0mm_W1.6mm_P2.50mm, F.Cu at (102.8, 147.8)
- added C3: 100nF (104), IMRANS_LIBRARY:C_Disc_D3.0mm_W1.6mm_P2.50mm, F.Cu at (184.8, 65.8)
- added C3: 100nF (104), IMRANS_LIBRARY:C_Disc_D3.0mm_W1.6mm_P2.50mm, F.Cu at (266.8, 65.8)
- added C3: 100nF (104), IMRANS_LIBRARY:C_Disc_D3.0mm_W1.6mm_P2.50mm, F.Cu at (143.8, 24.8)
- added C3: 100nF (104), IMRANS_LIBRARY:C_Disc_D3.0mm_W1.6mm_P2.50mm, F.Cu at (266.8, 24.8)
- added C3: 100nF (104), IMRANS_LIBRARY:C_Disc_D3.0mm_W1.6mm_P2.50mm, F.Cu at (225.8, 106.8)
- added C3: 100nF (104), IMRANS_LIBRARY:C_Disc_D3.0mm_W1.6mm_P2.50mm, F.Cu at (143.8, 147.8)
- added C3: 100nF (104), IMRANS_LIBRARY:C_Disc_D3.0mm_W1.6mm_P2.50mm, F.Cu at (102.8, 65.8)
- added C3: 100nF (104), IMRANS_LIBRARY:C_Disc_D3.0mm_W1.6mm_P2.50mm, F.Cu at (184.8, 106.8)
- added C3: 100nF (104), IMRANS_LIBRARY:C_Disc_D3.0mm_W1.6mm_P2.50mm, F.Cu at (266.8, 147.8)
- added C3: 100nF (104), IMRANS_LIBRARY:C_Disc_D3.0mm_W1.6mm_P2.50mm, F.Cu at (102.8, 24.8)
- added C3: 100nF (104), IMRANS_LIBRARY:C_Disc_D3.0mm_W1.6mm_P2.50mm, F.Cu at (61.8, 106.8)
- added C3: 100nF (104), IMRANS_LIBRARY:C_Disc_D3.0mm_W1.6mm_P2.50mm, F.Cu at (61.8, 65.8)
- added C3: 100nF (104), IMRANS_LIBRARY:C_Disc_D3.0mm_W1.6mm_P2.50mm, F.Cu at (184.8, 147.8)
- added C3: 100nF (104), IMRANS_LIBRARY:C_Disc_D3.0mm_W1.6mm_P2.50mm, F.Cu at (184.8, 24.8)
- added D1: 1N4007, IMRANS_LIBRARY:R_Axial_DIN0207_L6.3mm_D2.5mm_P10.16mm_Horizontal_2, F.Cu at (215.1, 82.0)
- added D1: 1N4007, IMRANS_LIBRARY:R_Axial_DIN0207_L6.3mm_D2.5mm_P10.16mm_Horizontal_2, F.Cu at (51.1, 82.0)
- added D1: 1N4007, IMRANS_LIBRARY:R_Axial_DIN0207_L6.3mm_D2.5mm_P10.16mm_Horizontal_2, F.Cu at (256.1, 123.0)
- added D1: 1N4007, IMRANS_LIBRARY:R_Axial_DIN0207_L6.3mm_D2.5mm_P10.16mm_Horizontal_2, F.Cu at (215.1, 41.0)
- added D1: 1N4007, IMRANS_LIBRARY:R_Axial_DIN0207_L6.3mm_D2.5mm_P10.16mm_Horizontal_2, F.Cu at (256.1, 82.0)
- added D1: 1N4007, IMRANS_LIBRARY:R_Axial_DIN0207_L6.3mm_D2.5mm_P10.16mm_Horizontal_2, F.Cu at (133.1, 41.0)
- added D1: 1N4007, IMRANS_LIBRARY:R_Axial_DIN0207_L6.3mm_D2.5mm_P10.16mm_Horizontal_2, F.Cu at (133.1, 123.0)
- added D1: 1N4007, IMRANS_LIBRARY:R_Axial_DIN0207_L6.3mm_D2.5mm_P10.16mm_Horizontal_2, F.Cu at (174.1, 82.0)
- added D1: 1N4007, IMRANS_LIBRARY:R_Axial_DIN0207_L6.3mm_D2.5mm_P10.16mm_Horizontal_2, F.Cu at (215.1, 164.0)
- added D1: 1N4007, IMRANS_LIBRARY:R_Axial_DIN0207_L6.3mm_D2.5mm_P10.16mm_Horizontal_2, F.Cu at (51.1, 164.0)
- added D1: 1N4007, IMRANS_LIBRARY:R_Axial_DIN0207_L6.3mm_D2.5mm_P10.16mm_Horizontal_2, F.Cu at (215.1, 123.0)
- added D1: 1N4007, IMRANS_LIBRARY:R_Axial_DIN0207_L6.3mm_D2.5mm_P10.16mm_Horizontal_2, F.Cu at (92.1, 164.0)
- added D1: 1N4007, IMRANS_LIBRARY:R_Axial_DIN0207_L6.3mm_D2.5mm_P10.16mm_Horizontal_2, F.Cu at (256.1, 41.0)
- added D1: 1N4007, IMRANS_LIBRARY:R_Axial_DIN0207_L6.3mm_D2.5mm_P10.16mm_Horizontal_2, F.Cu at (174.1, 41.0)
- added D1: 1N4007, IMRANS_LIBRARY:R_Axial_DIN0207_L6.3mm_D2.5mm_P10.16mm_Horizontal_2, F.Cu at (133.1, 164.0)
- added D1: 1N4007, IMRANS_LIBRARY:R_Axial_DIN0207_L6.3mm_D2.5mm_P10.16mm_Horizontal_2, F.Cu at (51.1, 41.0)
- added D1: 1N4007, IMRANS_LIBRARY:R_Axial_DIN0207_L6.3mm_D2.5mm_P10.16mm_Horizontal_2, F.Cu at (51.1, 123.0)
- added D1: 1N4007, IMRANS_LIBRARY:R_Axial_DIN0207_L6.3mm_D2.5mm_P10.16mm_Horizontal_2, F.Cu at (92.1, 41.0)
- added D1: 1N4007, IMRANS_LIBRARY:R_Axial_DIN0207_L6.3mm_D2.5mm_P10.16mm_Horizontal_2, F.Cu at (133.1, 82.0)
- added D1: 1N4007, IMRANS_LIBRARY:R_Axial_DIN0207_L6.3mm_D2.5mm_P10.16mm_Horizontal_2, F.Cu at (92.1, 123.0)
- added D1: 1N4007, IMRANS_LIBRARY:R_Axial_DIN0207_L6.3mm_D2.5mm_P10.16mm_Horizontal_2, F.Cu at (174.1, 164.0)
- added D1: 1N4007, IMRANS_LIBRARY:R_Axial_DIN0207_L6.3mm_D2.5mm_P10.16mm_Horizontal_2, F.Cu at (174.1, 123.0)
- added D1: 1N4007, IMRANS_LIBRARY:R_Axial_DIN0207_L6.3mm_D2.5mm_P10.16mm_Horizontal_2, F.Cu at (256.1, 164.0)
- added D1: 1N4007, IMRANS_LIBRARY:R_Axial_DIN0207_L6.3mm_D2.5mm_P10.16mm_Horizontal_2, F.Cu at (92.1, 82.0)
- added D2: D, IMRANS_LIBRARY:R_Axial_DIN0207_L6.3mm_D2.5mm_P10.16mm_Horizontal_2, F.Cu at (225.7, 167.2)
- added D2: D, IMRANS_LIBRARY:R_Axial_DIN0207_L6.3mm_D2.5mm_P10.16mm_Horizontal_2, F.Cu at (61.7, 167.2)
- added D2: D, IMRANS_LIBRARY:R_Axial_DIN0207_L6.3mm_D2.5mm_P10.16mm_Horizontal_2, F.Cu at (266.7, 44.2)
- added D2: D, IMRANS_LIBRARY:R_Axial_DIN0207_L6.3mm_D2.5mm_P10.16mm_Horizontal_2, F.Cu at (102.7, 44.2)
- added D2: D, IMRANS_LIBRARY:R_Axial_DIN0207_L6.3mm_D2.5mm_P10.16mm_Horizontal_2, F.Cu at (143.7, 44.2)
- added D2: D, IMRANS_LIBRARY:R_Axial_DIN0207_L6.3mm_D2.5mm_P10.16mm_Horizontal_2, F.Cu at (225.7, 126.2)
- added D2: D, IMRANS_LIBRARY:R_Axial_DIN0207_L6.3mm_D2.5mm_P10.16mm_Horizontal_2, F.Cu at (184.7, 44.2)
- added D2: D, IMRANS_LIBRARY:R_Axial_DIN0207_L6.3mm_D2.5mm_P10.16mm_Horizontal_2, F.Cu at (266.7, 85.2)
- added D2: D, IMRANS_LIBRARY:R_Axial_DIN0207_L6.3mm_D2.5mm_P10.16mm_Horizontal_2, F.Cu at (61.7, 44.2)
- added D2: D, IMRANS_LIBRARY:R_Axial_DIN0207_L6.3mm_D2.5mm_P10.16mm_Horizontal_2, F.Cu at (102.7, 85.2)
- added D2: D, IMRANS_LIBRARY:R_Axial_DIN0207_L6.3mm_D2.5mm_P10.16mm_Horizontal_2, F.Cu at (61.7, 126.2)
- added D2: D, IMRANS_LIBRARY:R_Axial_DIN0207_L6.3mm_D2.5mm_P10.16mm_Horizontal_2, F.Cu at (266.7, 126.2)
- added D2: D, IMRANS_LIBRARY:R_Axial_DIN0207_L6.3mm_D2.5mm_P10.16mm_Horizontal_2, F.Cu at (225.7, 44.2)
- added D2: D, IMRANS_LIBRARY:R_Axial_DIN0207_L6.3mm_D2.5mm_P10.16mm_Horizontal_2, F.Cu at (102.7, 167.2)
- added D2: D, IMRANS_LIBRARY:R_Axial_DIN0207_L6.3mm_D2.5mm_P10.16mm_Horizontal_2, F.Cu at (61.7, 85.2)
- added D2: D, IMRANS_LIBRARY:R_Axial_DIN0207_L6.3mm_D2.5mm_P10.16mm_Horizontal_2, F.Cu at (184.7, 126.2)
- added D2: D, IMRANS_LIBRARY:R_Axial_DIN0207_L6.3mm_D2.5mm_P10.16mm_Horizontal_2, F.Cu at (184.7, 167.2)
- added D2: D, IMRANS_LIBRARY:R_Axial_DIN0207_L6.3mm_D2.5mm_P10.16mm_Horizontal_2, F.Cu at (266.7, 167.2)
- added D2: D, IMRANS_LIBRARY:R_Axial_DIN0207_L6.3mm_D2.5mm_P10.16mm_Horizontal_2, F.Cu at (143.7, 85.2)
- added D2: D, IMRANS_LIBRARY:R_Axial_DIN0207_L6.3mm_D2.5mm_P10.16mm_Horizontal_2, F.Cu at (143.7, 167.2)
- added D2: D, IMRANS_LIBRARY:R_Axial_DIN0207_L6.3mm_D2.5mm_P10.16mm_Horizontal_2, F.Cu at (184.7, 85.2)
- added D2: D, IMRANS_LIBRARY:R_Axial_DIN0207_L6.3mm_D2.5mm_P10.16mm_Horizontal_2, F.Cu at (225.7, 85.2)
- added D2: D, IMRANS_LIBRARY:R_Axial_DIN0207_L6.3mm_D2.5mm_P10.16mm_Horizontal_2, F.Cu at (143.7, 126.2)
- added D2: D, IMRANS_LIBRARY:R_Axial_DIN0207_L6.3mm_D2.5mm_P10.16mm_Horizontal_2, F.Cu at (102.7, 126.2)
- added J1: Conn_01x03_Pin, IMRANS_LIBRARY:PinHeader_1x03_P2.54mm_Vertical, F.Cu at (93.4, 148.4)
- added J1: Conn_01x03_Pin, IMRANS_LIBRARY:PinHeader_1x03_P2.54mm_Vertical, F.Cu at (257.4, 148.4)
- added J1: Conn_01x03_Pin, IMRANS_LIBRARY:PinHeader_1x03_P2.54mm_Vertical, F.Cu at (175.4, 66.4)
- added J1: Conn_01x03_Pin, IMRANS_LIBRARY:PinHeader_1x03_P2.54mm_Vertical, F.Cu at (216.4, 66.4)
- added J1: Conn_01x03_Pin, IMRANS_LIBRARY:PinHeader_1x03_P2.54mm_Vertical, F.Cu at (257.4, 25.4)
- added J1: Conn_01x03_Pin, IMRANS_LIBRARY:PinHeader_1x03_P2.54mm_Vertical, F.Cu at (134.4, 66.4)
- added J1: Conn_01x03_Pin, IMRANS_LIBRARY:PinHeader_1x03_P2.54mm_Vertical, F.Cu at (257.4, 66.4)
- added J1: Conn_01x03_Pin, IMRANS_LIBRARY:PinHeader_1x03_P2.54mm_Vertical, F.Cu at (93.4, 107.4)
- added J1: Conn_01x03_Pin, IMRANS_LIBRARY:PinHeader_1x03_P2.54mm_Vertical, F.Cu at (93.4, 66.4)
- added J1: Conn_01x03_Pin, IMRANS_LIBRARY:PinHeader_1x03_P2.54mm_Vertical, F.Cu at (134.4, 148.4)
- added J1: Conn_01x03_Pin, IMRANS_LIBRARY:PinHeader_1x03_P2.54mm_Vertical, F.Cu at (216.4, 107.4)
- added J1: Conn_01x03_Pin, IMRANS_LIBRARY:PinHeader_1x03_P2.54mm_Vertical, F.Cu at (257.4, 107.4)
- added J1: Conn_01x03_Pin, IMRANS_LIBRARY:PinHeader_1x03_P2.54mm_Vertical, F.Cu at (175.4, 25.4)
- added J1: Conn_01x03_Pin, IMRANS_LIBRARY:PinHeader_1x03_P2.54mm_Vertical, F.Cu at (52.4, 107.4)
- added J1: Conn_01x03_Pin, IMRANS_LIBRARY:PinHeader_1x03_P2.54mm_Vertical, F.Cu at (175.4, 107.4)
- added J1: Conn_01x03_Pin, IMRANS_LIBRARY:PinHeader_1x03_P2.54mm_Vertical, F.Cu at (216.4, 25.4)
- added J1: Conn_01x03_Pin, IMRANS_LIBRARY:PinHeader_1x03_P2.54mm_Vertical, F.Cu at (52.4, 66.4)
- added J1: Conn_01x03_Pin, IMRANS_LIBRARY:PinHeader_1x03_P2.54mm_Vertical, F.Cu at (93.4, 25.4)
- added J1: Conn_01x03_Pin, IMRANS_LIBRARY:PinHeader_1x03_P2.54mm_Vertical, F.Cu at (52.4, 25.4)
- added J1: Conn_01x03_Pin, IMRANS_LIBRARY:PinHeader_1x03_P2.54mm_Vertical, F.Cu at (134.4, 107.4)
- added J1: Conn_01x03_Pin, IMRANS_LIBRARY:PinHeader_1x03_P2.54mm_Vertical, F.Cu at (52.4, 148.4)
- added J1: Conn_01x03_Pin, IMRANS_LIBRARY:PinHeader_1x03_P2.54mm_Vertical, F.Cu at (134.4, 25.4)
- added J1: Conn_01x03_Pin, IMRANS_LIBRARY:PinHeader_1x03_P2.54mm_Vertical, F.Cu at (175.4, 148.4)
- added J1: Conn_01x03_Pin, IMRANS_LIBRARY:PinHeader_1x03_P2.54mm_Vertical, F.Cu at (216.4, 148.4)
- added L1: L, Inductor_THT:L_Radial_D10.0mm_P5.00mm_Fastron_07M, F.Cu at (235.4, 54.8)
- added L1: L, Inductor_THT:L_Radial_D10.0mm_P5.00mm_Fastron_07M, F.Cu at (30.4, 54.8)
- added L1: L, Inductor_THT:L_Radial_D10.0mm_P5.00mm_Fastron_07M, F.Cu at (71.4, 136.8)
- added L1: L, Inductor_THT:L_Radial_D10.0mm_P5.00mm_Fastron_07M, F.Cu at (112.4, 136.8)
- added L1: L, Inductor_THT:L_Radial_D10.0mm_P5.00mm_Fastron_07M, F.Cu at (153.4, 177.8)
- added L1: L, Inductor_THT:L_Radial_D10.0mm_P5.00mm_Fastron_07M, F.Cu at (194.4, 177.8)
- added L1: L, Inductor_THT:L_Radial_D10.0mm_P5.00mm_Fastron_07M, F.Cu at (30.4, 95.8)
- added L1: L, Inductor_THT:L_Radial_D10.0mm_P5.00mm_Fastron_07M, F.Cu at (71.4, 95.8)
- added L1: L, Inductor_THT:L_Radial_D10.0mm_P5.00mm_Fastron_07M, F.Cu at (235.4, 177.8)
- added L1: L, Inductor_THT:L_Radial_D10.0mm_P5.00mm_Fastron_07M, F.Cu at (194.4, 95.8)
- added L1: L, Inductor_THT:L_Radial_D10.0mm_P5.00mm_Fastron_07M, F.Cu at (30.4, 177.8)
- added L1: L, Inductor_THT:L_Radial_D10.0mm_P5.00mm_Fastron_07M, F.Cu at (30.4, 136.8)
- added L1: L, Inductor_THT:L_Radial_D10.0mm_P5.00mm_Fastron_07M, F.Cu at (153.4, 136.8)
- added L1: L, Inductor_THT:L_Radial_D10.0mm_P5.00mm_Fastron_07M, F.Cu at (235.4, 136.8)
- added L1: L, Inductor_THT:L_Radial_D10.0mm_P5.00mm_Fastron_07M, F.Cu at (153.4, 95.8)
- added L1: L, Inductor_THT:L_Radial_D10.0mm_P5.00mm_Fastron_07M, F.Cu at (71.4, 54.8)
- added L1: L, Inductor_THT:L_Radial_D10.0mm_P5.00mm_Fastron_07M, F.Cu at (153.4, 54.8)
- added L1: L, Inductor_THT:L_Radial_D10.0mm_P5.00mm_Fastron_07M, F.Cu at (112.4, 54.8)
- added L1: L, Inductor_THT:L_Radial_D10.0mm_P5.00mm_Fastron_07M, F.Cu at (112.4, 95.8)
- added L1: L, Inductor_THT:L_Radial_D10.0mm_P5.00mm_Fastron_07M, F.Cu at (112.4, 177.8)
- added L1: L, Inductor_THT:L_Radial_D10.0mm_P5.00mm_Fastron_07M, F.Cu at (194.4, 136.8)
- added L1: L, Inductor_THT:L_Radial_D10.0mm_P5.00mm_Fastron_07M, F.Cu at (71.4, 177.8)
- added L1: L, Inductor_THT:L_Radial_D10.0mm_P5.00mm_Fastron_07M, F.Cu at (235.4, 95.8)
- added L1: L, Inductor_THT:L_Radial_D10.0mm_P5.00mm_Fastron_07M, F.Cu at (194.4, 54.8)
- added R1: 10k, IMRANS_LIBRARY:R_Axial_DIN0207_L6.3mm_D2.5mm_P10.16mm_Horizontal_2, F.Cu at (49.9, 174.4)
- added R1: 10k, IMRANS_LIBRARY:R_Axial_DIN0207_L6.3mm_D2.5mm_P10.16mm_Horizontal_2, F.Cu at (254.9, 51.4)
- added R1: 10k, IMRANS_LIBRARY:R_Axial_DIN0207_L6.3mm_D2.5mm_P10.16mm_Horizontal_2, F.Cu at (172.9, 92.4)
- added R1: 10k, IMRANS_LIBRARY:R_Axial_DIN0207_L6.3mm_D2.5mm_P10.16mm_Horizontal_2, F.Cu at (213.9, 174.4)
- added R1: 10k, IMRANS_LIBRARY:R_Axial_DIN0207_L6.3mm_D2.5mm_P10.16mm_Horizontal_2, F.Cu at (172.9, 51.4)
- added R1: 10k, IMRANS_LIBRARY:R_Axial_DIN0207_L6.3mm_D2.5mm_P10.16mm_Horizontal_2, F.Cu at (131.9, 133.4)
- added R1: 10k, IMRANS_LIBRARY:R_Axial_DIN0207_L6.3mm_D2.5mm_P10.16mm_Horizontal_2, F.Cu at (90.9, 51.4)
- added R1: 10k, IMRANS_LIBRARY:R_Axial_DIN0207_L6.3mm_D2.5mm_P10.16mm_Horizontal_2, F.Cu at (254.9, 133.4)
- added R1: 10k, IMRANS_LIBRARY:R_Axial_DIN0207_L6.3mm_D2.5mm_P10.16mm_Horizontal_2, F.Cu at (90.9, 174.4)
- added R1: 10k, IMRANS_LIBRARY:R_Axial_DIN0207_L6.3mm_D2.5mm_P10.16mm_Horizontal_2, F.Cu at (254.9, 92.4)
- added R1: 10k, IMRANS_LIBRARY:R_Axial_DIN0207_L6.3mm_D2.5mm_P10.16mm_Horizontal_2, F.Cu at (172.9, 133.4)
- added R1: 10k, IMRANS_LIBRARY:R_Axial_DIN0207_L6.3mm_D2.5mm_P10.16mm_Horizontal_2, F.Cu at (254.9, 174.4)
- added R1: 10k, IMRANS_LIBRARY:R_Axial_DIN0207_L6.3mm_D2.5mm_P10.16mm_Horizontal_2, F.Cu at (49.9, 133.4)
- added R1: 10k, IMRANS_LIBRARY:R_Axial_DIN0207_L6.3mm_D2.5mm_P10.16mm_Horizontal_2, F.Cu at (49.9, 92.4)
- added R1: 10k, IMRANS_LIBRARY:R_Axial_DIN0207_L6.3mm_D2.5mm_P10.16mm_Horizontal_2, F.Cu at (90.9, 92.4)
- added R1: 10k, IMRANS_LIBRARY:R_Axial_DIN0207_L6.3mm_D2.5mm_P10.16mm_Horizontal_2, F.Cu at (213.9, 51.4)
- added R1: 10k, IMRANS_LIBRARY:R_Axial_DIN0207_L6.3mm_D2.5mm_P10.16mm_Horizontal_2, F.Cu at (131.9, 92.4)
- added R1: 10k, IMRANS_LIBRARY:R_Axial_DIN0207_L6.3mm_D2.5mm_P10.16mm_Horizontal_2, F.Cu at (90.9, 133.4)
- added R1: 10k, IMRANS_LIBRARY:R_Axial_DIN0207_L6.3mm_D2.5mm_P10.16mm_Horizontal_2, F.Cu at (49.9, 51.4)
- added R1: 10k, IMRANS_LIBRARY:R_Axial_DIN0207_L6.3mm_D2.5mm_P10.16mm_Horizontal_2, F.Cu at (213.9, 133.4)
- added R1: 10k, IMRANS_LIBRARY:R_Axial_DIN0207_L6.3mm_D2.5mm_P10.16mm_Horizontal_2, F.Cu at (172.9, 174.4)
- added R1: 10k, IMRANS_LIBRARY:R_Axial_DIN0207_L6.3mm_D2.5mm_P10.16mm_Horizontal_2, F.Cu at (213.9, 92.4)
- added R1: 10k, IMRANS_LIBRARY:R_Axial_DIN0207_L6.3mm_D2.5mm_P10.16mm_Horizontal_2, F.Cu at (131.9, 51.4)
- added R1: 10k, IMRANS_LIBRARY:R_Axial_DIN0207_L6.3mm_D2.5mm_P10.16mm_Horizontal_2, F.Cu at (131.9, 174.4)
- added R2: 10k, IMRANS_LIBRARY:R_Axial_DIN0207_L6.3mm_D2.5mm_P10.16mm_Horizontal_2, F.Cu at (215.3, 154.2)
- added R2: 10k, IMRANS_LIBRARY:R_Axial_DIN0207_L6.3mm_D2.5mm_P10.16mm_Horizontal_2, F.Cu at (133.3, 31.2)
- added R2: 10k, IMRANS_LIBRARY:R_Axial_DIN0207_L6.3mm_D2.5mm_P10.16mm_Horizontal_2, F.Cu at (51.3, 113.2)
- added R2: 10k, IMRANS_LIBRARY:R_Axial_DIN0207_L6.3mm_D2.5mm_P10.16mm_Horizontal_2, F.Cu at (256.3, 72.2)
- added R2: 10k, IMRANS_LIBRARY:R_Axial_DIN0207_L6.3mm_D2.5mm_P10.16mm_Horizontal_2, F.Cu at (174.3, 154.2)
- added R2: 10k, IMRANS_LIBRARY:R_Axial_DIN0207_L6.3mm_D2.5mm_P10.16mm_Horizontal_2, F.Cu at (215.3, 113.2)
- added R2: 10k, IMRANS_LIBRARY:R_Axial_DIN0207_L6.3mm_D2.5mm_P10.16mm_Horizontal_2, F.Cu at (215.3, 31.2)
- added R2: 10k, IMRANS_LIBRARY:R_Axial_DIN0207_L6.3mm_D2.5mm_P10.16mm_Horizontal_2, F.Cu at (256.3, 31.2)
- added R2: 10k, IMRANS_LIBRARY:R_Axial_DIN0207_L6.3mm_D2.5mm_P10.16mm_Horizontal_2, F.Cu at (133.3, 154.2)
- added R2: 10k, IMRANS_LIBRARY:R_Axial_DIN0207_L6.3mm_D2.5mm_P10.16mm_Horizontal_2, F.Cu at (256.3, 113.2)
- added R2: 10k, IMRANS_LIBRARY:R_Axial_DIN0207_L6.3mm_D2.5mm_P10.16mm_Horizontal_2, F.Cu at (92.3, 154.2)
- added R2: 10k, IMRANS_LIBRARY:R_Axial_DIN0207_L6.3mm_D2.5mm_P10.16mm_Horizontal_2, F.Cu at (133.3, 113.2)
- added R2: 10k, IMRANS_LIBRARY:R_Axial_DIN0207_L6.3mm_D2.5mm_P10.16mm_Horizontal_2, F.Cu at (92.3, 113.2)
- added R2: 10k, IMRANS_LIBRARY:R_Axial_DIN0207_L6.3mm_D2.5mm_P10.16mm_Horizontal_2, F.Cu at (51.3, 72.2)
- added R2: 10k, IMRANS_LIBRARY:R_Axial_DIN0207_L6.3mm_D2.5mm_P10.16mm_Horizontal_2, F.Cu at (256.3, 154.2)
- added R2: 10k, IMRANS_LIBRARY:R_Axial_DIN0207_L6.3mm_D2.5mm_P10.16mm_Horizontal_2, F.Cu at (92.3, 72.2)
- added R2: 10k, IMRANS_LIBRARY:R_Axial_DIN0207_L6.3mm_D2.5mm_P10.16mm_Horizontal_2, F.Cu at (51.3, 154.2)
- added R2: 10k, IMRANS_LIBRARY:R_Axial_DIN0207_L6.3mm_D2.5mm_P10.16mm_Horizontal_2, F.Cu at (174.3, 113.2)
- added R2: 10k, IMRANS_LIBRARY:R_Axial_DIN0207_L6.3mm_D2.5mm_P10.16mm_Horizontal_2, F.Cu at (215.3, 72.2)
- added R2: 10k, IMRANS_LIBRARY:R_Axial_DIN0207_L6.3mm_D2.5mm_P10.16mm_Horizontal_2, F.Cu at (92.3, 31.2)
- added R2: 10k, IMRANS_LIBRARY:R_Axial_DIN0207_L6.3mm_D2.5mm_P10.16mm_Horizontal_2, F.Cu at (133.3, 72.2)
- added R2: 10k, IMRANS_LIBRARY:R_Axial_DIN0207_L6.3mm_D2.5mm_P10.16mm_Horizontal_2, F.Cu at (174.3, 72.2)
- added R2: 10k, IMRANS_LIBRARY:R_Axial_DIN0207_L6.3mm_D2.5mm_P10.16mm_Horizontal_2, F.Cu at (51.3, 31.2)
- added R2: 10k, IMRANS_LIBRARY:R_Axial_DIN0207_L6.3mm_D2.5mm_P10.16mm_Horizontal_2, F.Cu at (174.3, 31.2)
- added R3: 220, IMRANS_LIBRARY:R_Axial_DIN0207_L6.3mm_D2.5mm_P10.16mm_Horizontal_2, F.Cu at (197.2, 130.9)
- added R3: 220, IMRANS_LIBRARY:R_Axial_DIN0207_L6.3mm_D2.5mm_P10.16mm_Horizontal_2, F.Cu at (238.2, 171.9)
- added R3: 220, IMRANS_LIBRARY:R_Axial_DIN0207_L6.3mm_D2.5mm_P10.16mm_Horizontal_2, F.Cu at (197.2, 48.9)
- added R3: 220, IMRANS_LIBRARY:R_Axial_DIN0207_L6.3mm_D2.5mm_P10.16mm_Horizontal_2, F.Cu at (33.2, 130.9)
- added R3: 220, IMRANS_LIBRARY:R_Axial_DIN0207_L6.3mm_D2.5mm_P10.16mm_Horizontal_2, F.Cu at (115.2, 48.9)
- added R3: 220, IMRANS_LIBRARY:R_Axial_DIN0207_L6.3mm_D2.5mm_P10.16mm_Horizontal_2, F.Cu at (74.2, 89.9)
- added R3: 220, IMRANS_LIBRARY:R_Axial_DIN0207_L6.3mm_D2.5mm_P10.16mm_Horizontal_2, F.Cu at (115.2, 171.9)
- added R3: 220, IMRANS_LIBRARY:R_Axial_DIN0207_L6.3mm_D2.5mm_P10.16mm_Horizontal_2, F.Cu at (238.2, 89.9)
- added R3: 220, IMRANS_LIBRARY:R_Axial_DIN0207_L6.3mm_D2.5mm_P10.16mm_Horizontal_2, F.Cu at (156.2, 130.9)
- added R3: 220, IMRANS_LIBRARY:R_Axial_DIN0207_L6.3mm_D2.5mm_P10.16mm_Horizontal_2, F.Cu at (197.2, 89.9)
- added R3: 220, IMRANS_LIBRARY:R_Axial_DIN0207_L6.3mm_D2.5mm_P10.16mm_Horizontal_2, F.Cu at (33.2, 48.9)
- added R3: 220, IMRANS_LIBRARY:R_Axial_DIN0207_L6.3mm_D2.5mm_P10.16mm_Horizontal_2, F.Cu at (238.2, 130.9)
- added R3: 220, IMRANS_LIBRARY:R_Axial_DIN0207_L6.3mm_D2.5mm_P10.16mm_Horizontal_2, F.Cu at (33.2, 89.9)
- added R3: 220, IMRANS_LIBRARY:R_Axial_DIN0207_L6.3mm_D2.5mm_P10.16mm_Horizontal_2, F.Cu at (156.2, 89.9)
- added R3: 220, IMRANS_LIBRARY:R_Axial_DIN0207_L6.3mm_D2.5mm_P10.16mm_Horizontal_2, F.Cu at (115.2, 89.9)
- added R3: 220, IMRANS_LIBRARY:R_Axial_DIN0207_L6.3mm_D2.5mm_P10.16mm_Horizontal_2, F.Cu at (74.2, 171.9)
- added R3: 220, IMRANS_LIBRARY:R_Axial_DIN0207_L6.3mm_D2.5mm_P10.16mm_Horizontal_2, F.Cu at (197.2, 171.9)
- added R3: 220, IMRANS_LIBRARY:R_Axial_DIN0207_L6.3mm_D2.5mm_P10.16mm_Horizontal_2, F.Cu at (238.2, 48.9)
- added R3: 220, IMRANS_LIBRARY:R_Axial_DIN0207_L6.3mm_D2.5mm_P10.16mm_Horizontal_2, F.Cu at (74.2, 130.9)
- added R3: 220, IMRANS_LIBRARY:R_Axial_DIN0207_L6.3mm_D2.5mm_P10.16mm_Horizontal_2, F.Cu at (156.2, 171.9)
- added R3: 220, IMRANS_LIBRARY:R_Axial_DIN0207_L6.3mm_D2.5mm_P10.16mm_Horizontal_2, F.Cu at (156.2, 48.9)
- added R3: 220, IMRANS_LIBRARY:R_Axial_DIN0207_L6.3mm_D2.5mm_P10.16mm_Horizontal_2, F.Cu at (74.2, 48.9)
- added R3: 220, IMRANS_LIBRARY:R_Axial_DIN0207_L6.3mm_D2.5mm_P10.16mm_Horizontal_2, F.Cu at (115.2, 130.9)
- added R3: 220, IMRANS_LIBRARY:R_Axial_DIN0207_L6.3mm_D2.5mm_P10.16mm_Horizontal_2, F.Cu at (33.2, 171.9)
- added R4: 1M, IMRANS_LIBRARY:R_Axial_DIN0207_L6.3mm_D2.5mm_P10.16mm_Horizontal_2, F.Cu at (200.6, 38.9)
- added R4: 1M, IMRANS_LIBRARY:R_Axial_DIN0207_L6.3mm_D2.5mm_P10.16mm_Horizontal_2, F.Cu at (36.6, 161.9)
- added R4: 1M, IMRANS_LIBRARY:R_Axial_DIN0207_L6.3mm_D2.5mm_P10.16mm_Horizontal_2, F.Cu at (36.6, 79.9)
- added R4: 1M, IMRANS_LIBRARY:R_Axial_DIN0207_L6.3mm_D2.5mm_P10.16mm_Horizontal_2, F.Cu at (159.6, 161.9)
- added R4: 1M, IMRANS_LIBRARY:R_Axial_DIN0207_L6.3mm_D2.5mm_P10.16mm_Horizontal_2, F.Cu at (118.6, 79.9)
- added R4: 1M, IMRANS_LIBRARY:R_Axial_DIN0207_L6.3mm_D2.5mm_P10.16mm_Horizontal_2, F.Cu at (200.6, 161.9)
- added R4: 1M, IMRANS_LIBRARY:R_Axial_DIN0207_L6.3mm_D2.5mm_P10.16mm_Horizontal_2, F.Cu at (36.6, 120.9)
- added R4: 1M, IMRANS_LIBRARY:R_Axial_DIN0207_L6.3mm_D2.5mm_P10.16mm_Horizontal_2, F.Cu at (118.6, 38.9)
- added R4: 1M, IMRANS_LIBRARY:R_Axial_DIN0207_L6.3mm_D2.5mm_P10.16mm_Horizontal_2, F.Cu at (118.6, 161.9)
- added R4: 1M, IMRANS_LIBRARY:R_Axial_DIN0207_L6.3mm_D2.5mm_P10.16mm_Horizontal_2, F.Cu at (77.6, 161.9)
- added R4: 1M, IMRANS_LIBRARY:R_Axial_DIN0207_L6.3mm_D2.5mm_P10.16mm_Horizontal_2, F.Cu at (36.6, 38.9)
- added R4: 1M, IMRANS_LIBRARY:R_Axial_DIN0207_L6.3mm_D2.5mm_P10.16mm_Horizontal_2, F.Cu at (159.6, 79.9)
- added R4: 1M, IMRANS_LIBRARY:R_Axial_DIN0207_L6.3mm_D2.5mm_P10.16mm_Horizontal_2, F.Cu at (241.6, 161.9)
- added R4: 1M, IMRANS_LIBRARY:R_Axial_DIN0207_L6.3mm_D2.5mm_P10.16mm_Horizontal_2, F.Cu at (241.6, 79.9)
- added R4: 1M, IMRANS_LIBRARY:R_Axial_DIN0207_L6.3mm_D2.5mm_P10.16mm_Horizontal_2, F.Cu at (200.6, 120.9)
- added R4: 1M, IMRANS_LIBRARY:R_Axial_DIN0207_L6.3mm_D2.5mm_P10.16mm_Horizontal_2, F.Cu at (159.6, 120.9)
- added R4: 1M, IMRANS_LIBRARY:R_Axial_DIN0207_L6.3mm_D2.5mm_P10.16mm_Horizontal_2, F.Cu at (118.6, 120.9)
- added R4: 1M, IMRANS_LIBRARY:R_Axial_DIN0207_L6.3mm_D2.5mm_P10.16mm_Horizontal_2, F.Cu at (77.6, 120.9)
- added R4: 1M, IMRANS_LIBRARY:R_Axial_DIN0207_L6.3mm_D2.5mm_P10.16mm_Horizontal_2, F.Cu at (200.6, 79.9)
- added R4: 1M, IMRANS_LIBRARY:R_Axial_DIN0207_L6.3mm_D2.5mm_P10.16mm_Horizontal_2, F.Cu at (77.6, 38.9)
- added R4: 1M, IMRANS_LIBRARY:R_Axial_DIN0207_L6.3mm_D2.5mm_P10.16mm_Horizontal_2, F.Cu at (241.6, 38.9)
- added R4: 1M, IMRANS_LIBRARY:R_Axial_DIN0207_L6.3mm_D2.5mm_P10.16mm_Horizontal_2, F.Cu at (77.6, 79.9)
- added R4: 1M, IMRANS_LIBRARY:R_Axial_DIN0207_L6.3mm_D2.5mm_P10.16mm_Horizontal_2, F.Cu at (159.6, 38.9)
- added R4: 1M, IMRANS_LIBRARY:R_Axial_DIN0207_L6.3mm_D2.5mm_P10.16mm_Horizontal_2, F.Cu at (241.6, 120.9)
- added R5: 1K, IMRANS_LIBRARY:R_Axial_DIN0207_L6.3mm_D2.5mm_P10.16mm_Horizontal_2, F.Cu at (77.2, 51.7)
- added R5: 1K, IMRANS_LIBRARY:R_Axial_DIN0207_L6.3mm_D2.5mm_P10.16mm_Horizontal_2, F.Cu at (200.2, 174.7)
- added R5: 1K, IMRANS_LIBRARY:R_Axial_DIN0207_L6.3mm_D2.5mm_P10.16mm_Horizontal_2, F.Cu at (159.2, 51.7)
- added R5: 1K, IMRANS_LIBRARY:R_Axial_DIN0207_L6.3mm_D2.5mm_P10.16mm_Horizontal_2, F.Cu at (241.2, 174.7)
- added R5: 1K, IMRANS_LIBRARY:R_Axial_DIN0207_L6.3mm_D2.5mm_P10.16mm_Horizontal_2, F.Cu at (241.2, 51.7)
- added R5: 1K, IMRANS_LIBRARY:R_Axial_DIN0207_L6.3mm_D2.5mm_P10.16mm_Horizontal_2, F.Cu at (77.2, 92.7)
- added R5: 1K, IMRANS_LIBRARY:R_Axial_DIN0207_L6.3mm_D2.5mm_P10.16mm_Horizontal_2, F.Cu at (118.2, 92.7)
- added R5: 1K, IMRANS_LIBRARY:R_Axial_DIN0207_L6.3mm_D2.5mm_P10.16mm_Horizontal_2, F.Cu at (200.2, 51.7)
- added R5: 1K, IMRANS_LIBRARY:R_Axial_DIN0207_L6.3mm_D2.5mm_P10.16mm_Horizontal_2, F.Cu at (118.2, 174.7)
- added R5: 1K, IMRANS_LIBRARY:R_Axial_DIN0207_L6.3mm_D2.5mm_P10.16mm_Horizontal_2, F.Cu at (200.2, 133.7)
- added R5: 1K, IMRANS_LIBRARY:R_Axial_DIN0207_L6.3mm_D2.5mm_P10.16mm_Horizontal_2, F.Cu at (118.2, 133.7)
- added R5: 1K, IMRANS_LIBRARY:R_Axial_DIN0207_L6.3mm_D2.5mm_P10.16mm_Horizontal_2, F.Cu at (77.2, 133.7)
- added R5: 1K, IMRANS_LIBRARY:R_Axial_DIN0207_L6.3mm_D2.5mm_P10.16mm_Horizontal_2, F.Cu at (159.2, 133.7)
- added R5: 1K, IMRANS_LIBRARY:R_Axial_DIN0207_L6.3mm_D2.5mm_P10.16mm_Horizontal_2, F.Cu at (159.2, 174.7)
- added R5: 1K, IMRANS_LIBRARY:R_Axial_DIN0207_L6.3mm_D2.5mm_P10.16mm_Horizontal_2, F.Cu at (200.2, 92.7)
- added R5: 1K, IMRANS_LIBRARY:R_Axial_DIN0207_L6.3mm_D2.5mm_P10.16mm_Horizontal_2, F.Cu at (241.2, 133.7)
- added R5: 1K, IMRANS_LIBRARY:R_Axial_DIN0207_L6.3mm_D2.5mm_P10.16mm_Horizontal_2, F.Cu at (159.2, 92.7)
- added R5: 1K, IMRANS_LIBRARY:R_Axial_DIN0207_L6.3mm_D2.5mm_P10.16mm_Horizontal_2, F.Cu at (118.2, 51.7)
- added R5: 1K, IMRANS_LIBRARY:R_Axial_DIN0207_L6.3mm_D2.5mm_P10.16mm_Horizontal_2, F.Cu at (36.2, 133.7)
- added R5: 1K, IMRANS_LIBRARY:R_Axial_DIN0207_L6.3mm_D2.5mm_P10.16mm_Horizontal_2, F.Cu at (36.2, 51.7)
- added R5: 1K, IMRANS_LIBRARY:R_Axial_DIN0207_L6.3mm_D2.5mm_P10.16mm_Horizontal_2, F.Cu at (77.2, 174.7)
- added R5: 1K, IMRANS_LIBRARY:R_Axial_DIN0207_L6.3mm_D2.5mm_P10.16mm_Horizontal_2, F.Cu at (36.2, 92.7)
- added R5: 1K, IMRANS_LIBRARY:R_Axial_DIN0207_L6.3mm_D2.5mm_P10.16mm_Horizontal_2, F.Cu at (241.2, 92.7)
- added R5: 1K, IMRANS_LIBRARY:R_Axial_DIN0207_L6.3mm_D2.5mm_P10.16mm_Horizontal_2, F.Cu at (36.2, 174.7)
- added R6: 100K, IMRANS_LIBRARY:R_Axial_DIN0207_L6.3mm_D2.5mm_P10.16mm_Horizontal_2, F.Cu at (61.9, 34.4)
- added R6: 100K, IMRANS_LIBRARY:R_Axial_DIN0207_L6.3mm_D2.5mm_P10.16mm_Horizontal_2, F.Cu at (143.9, 75.4)
- added R6: 100K, IMRANS_LIBRARY:R_Axial_DIN0207_L6.3mm_D2.5mm_P10.16mm_Horizontal_2, F.Cu at (102.9, 75.4)
- added R6: 100K, IMRANS_LIBRARY:R_Axial_DIN0207_L6.3mm_D2.5mm_P10.16mm_Horizontal_2, F.Cu at (266.9, 75.4)
- added R6: 100K, IMRANS_LIBRARY:R_Axial_DIN0207_L6.3mm_D2.5mm_P10.16mm_Horizontal_2, F.Cu at (61.9, 157.4)
- added R6: 100K, IMRANS_LIBRARY:R_Axial_DIN0207_L6.3mm_D2.5mm_P10.16mm_Horizontal_2, F.Cu at (266.9, 157.4)
- added R6: 100K, IMRANS_LIBRARY:R_Axial_DIN0207_L6.3mm_D2.5mm_P10.16mm_Horizontal_2, F.Cu at (266.9, 116.4)
- added R6: 100K, IMRANS_LIBRARY:R_Axial_DIN0207_L6.3mm_D2.5mm_P10.16mm_Horizontal_2, F.Cu at (102.9, 157.4)
- added R6: 100K, IMRANS_LIBRARY:R_Axial_DIN0207_L6.3mm_D2.5mm_P10.16mm_Horizontal_2, F.Cu at (184.9, 34.4)
- added R6: 100K, IMRANS_LIBRARY:R_Axial_DIN0207_L6.3mm_D2.5mm_P10.16mm_Horizontal_2, F.Cu at (143.9, 116.4)
- added R6: 100K, IMRANS_LIBRARY:R_Axial_DIN0207_L6.3mm_D2.5mm_P10.16mm_Horizontal_2, F.Cu at (61.9, 116.4)
- added R6: 100K, IMRANS_LIBRARY:R_Axial_DIN0207_L6.3mm_D2.5mm_P10.16mm_Horizontal_2, F.Cu at (102.9, 116.4)
- added R6: 100K, IMRANS_LIBRARY:R_Axial_DIN0207_L6.3mm_D2.5mm_P10.16mm_Horizontal_2, F.Cu at (266.9, 34.4)
- added R6: 100K, IMRANS_LIBRARY:R_Axial_DIN0207_L6.3mm_D2.5mm_P10.16mm_Horizontal_2, F.Cu at (225.9, 116.4)
- added R6: 100K, IMRANS_LIBRARY:R_Axial_DIN0207_L6.3mm_D2.5mm_P10.16mm_Horizontal_2, F.Cu at (225.9, 75.4)
- added R6: 100K, IMRANS_LIBRARY:R_Axial_DIN0207_L6.3mm_D2.5mm_P10.16mm_Horizontal_2, F.Cu at (143.9, 34.4)
- added R6: 100K, IMRANS_LIBRARY:R_Axial_DIN0207_L6.3mm_D2.5mm_P10.16mm_Horizontal_2, F.Cu at (102.9, 34.4)
- added R6: 100K, IMRANS_LIBRARY:R_Axial_DIN0207_L6.3mm_D2.5mm_P10.16mm_Horizontal_2, F.Cu at (184.9, 157.4)
- added R6: 100K, IMRANS_LIBRARY:R_Axial_DIN0207_L6.3mm_D2.5mm_P10.16mm_Horizontal_2, F.Cu at (184.9, 75.4)
- added R6: 100K, IMRANS_LIBRARY:R_Axial_DIN0207_L6.3mm_D2.5mm_P10.16mm_Horizontal_2, F.Cu at (225.9, 34.4)
- added R6: 100K, IMRANS_LIBRARY:R_Axial_DIN0207_L6.3mm_D2.5mm_P10.16mm_Horizontal_2, F.Cu at (143.9, 157.4)
- added R6: 100K, IMRANS_LIBRARY:R_Axial_DIN0207_L6.3mm_D2.5mm_P10.16mm_Horizontal_2, F.Cu at (61.9, 75.4)
- added R6: 100K, IMRANS_LIBRARY:R_Axial_DIN0207_L6.3mm_D2.5mm_P10.16mm_Horizontal_2, F.Cu at (225.9, 157.4)
- added R6: 100K, IMRANS_LIBRARY:R_Axial_DIN0207_L6.3mm_D2.5mm_P10.16mm_Horizontal_2, F.Cu at (184.9, 116.4)
- added R7: 1K, IMRANS_LIBRARY:R_Axial_DIN0207_L6.3mm_D2.5mm_P10.16mm_Horizontal_2, F.Cu at (174.7, 170.6)
- added R7: 1K, IMRANS_LIBRARY:R_Axial_DIN0207_L6.3mm_D2.5mm_P10.16mm_Horizontal_2, F.Cu at (215.7, 170.6)
- added R7: 1K, IMRANS_LIBRARY:R_Axial_DIN0207_L6.3mm_D2.5mm_P10.16mm_Horizontal_2, F.Cu at (51.7, 170.6)
- added R7: 1K, IMRANS_LIBRARY:R_Axial_DIN0207_L6.3mm_D2.5mm_P10.16mm_Horizontal_2, F.Cu at (92.7, 47.6)
- added R7: 1K, IMRANS_LIBRARY:R_Axial_DIN0207_L6.3mm_D2.5mm_P10.16mm_Horizontal_2, F.Cu at (256.7, 170.6)
- added R7: 1K, IMRANS_LIBRARY:R_Axial_DIN0207_L6.3mm_D2.5mm_P10.16mm_Horizontal_2, F.Cu at (256.7, 129.6)
- added R7: 1K, IMRANS_LIBRARY:R_Axial_DIN0207_L6.3mm_D2.5mm_P10.16mm_Horizontal_2, F.Cu at (215.7, 47.6)
- added R7: 1K, IMRANS_LIBRARY:R_Axial_DIN0207_L6.3mm_D2.5mm_P10.16mm_Horizontal_2, F.Cu at (133.7, 47.6)
- added R7: 1K, IMRANS_LIBRARY:R_Axial_DIN0207_L6.3mm_D2.5mm_P10.16mm_Horizontal_2, F.Cu at (92.7, 129.6)
- added R7: 1K, IMRANS_LIBRARY:R_Axial_DIN0207_L6.3mm_D2.5mm_P10.16mm_Horizontal_2, F.Cu at (256.7, 88.6)
- added R7: 1K, IMRANS_LIBRARY:R_Axial_DIN0207_L6.3mm_D2.5mm_P10.16mm_Horizontal_2, F.Cu at (51.7, 88.6)
- added R7: 1K, IMRANS_LIBRARY:R_Axial_DIN0207_L6.3mm_D2.5mm_P10.16mm_Horizontal_2, F.Cu at (133.7, 88.6)
- added R7: 1K, IMRANS_LIBRARY:R_Axial_DIN0207_L6.3mm_D2.5mm_P10.16mm_Horizontal_2, F.Cu at (133.7, 170.6)
- added R7: 1K, IMRANS_LIBRARY:R_Axial_DIN0207_L6.3mm_D2.5mm_P10.16mm_Horizontal_2, F.Cu at (174.7, 129.6)
- added R7: 1K, IMRANS_LIBRARY:R_Axial_DIN0207_L6.3mm_D2.5mm_P10.16mm_Horizontal_2, F.Cu at (256.7, 47.6)
- added R7: 1K, IMRANS_LIBRARY:R_Axial_DIN0207_L6.3mm_D2.5mm_P10.16mm_Horizontal_2, F.Cu at (174.7, 88.6)
- added R7: 1K, IMRANS_LIBRARY:R_Axial_DIN0207_L6.3mm_D2.5mm_P10.16mm_Horizontal_2, F.Cu at (133.7, 129.6)
- added R7: 1K, IMRANS_LIBRARY:R_Axial_DIN0207_L6.3mm_D2.5mm_P10.16mm_Horizontal_2, F.Cu at (215.7, 129.6)
- added R7: 1K, IMRANS_LIBRARY:R_Axial_DIN0207_L6.3mm_D2.5mm_P10.16mm_Horizontal_2, F.Cu at (215.7, 88.6)
- added R7: 1K, IMRANS_LIBRARY:R_Axial_DIN0207_L6.3mm_D2.5mm_P10.16mm_Horizontal_2, F.Cu at (92.7, 88.6)
- added R7: 1K, IMRANS_LIBRARY:R_Axial_DIN0207_L6.3mm_D2.5mm_P10.16mm_Horizontal_2, F.Cu at (92.7, 170.6)
- added R7: 1K, IMRANS_LIBRARY:R_Axial_DIN0207_L6.3mm_D2.5mm_P10.16mm_Horizontal_2, F.Cu at (174.7, 47.6)
- added R7: 1K, IMRANS_LIBRARY:R_Axial_DIN0207_L6.3mm_D2.5mm_P10.16mm_Horizontal_2, F.Cu at (51.7, 47.6)
- added R7: 1K, IMRANS_LIBRARY:R_Axial_DIN0207_L6.3mm_D2.5mm_P10.16mm_Horizontal_2, F.Cu at (51.7, 129.6)
- added R9: 1K, IMRANS_LIBRARY:R_Axial_DIN0207_L6.3mm_D2.5mm_P10.16mm_Horizontal_2, F.Cu at (185.0, 160.8)
- added R9: 1K, IMRANS_LIBRARY:R_Axial_DIN0207_L6.3mm_D2.5mm_P10.16mm_Horizontal_2, F.Cu at (226.0, 37.8)
- added R9: 1K, IMRANS_LIBRARY:R_Axial_DIN0207_L6.3mm_D2.5mm_P10.16mm_Horizontal_2, F.Cu at (144.0, 160.8)
- added R9: 1K, IMRANS_LIBRARY:R_Axial_DIN0207_L6.3mm_D2.5mm_P10.16mm_Horizontal_2, F.Cu at (103.0, 37.8)
- added R9: 1K, IMRANS_LIBRARY:R_Axial_DIN0207_L6.3mm_D2.5mm_P10.16mm_Horizontal_2, F.Cu at (103.0, 119.8)
- added R9: 1K, IMRANS_LIBRARY:R_Axial_DIN0207_L6.3mm_D2.5mm_P10.16mm_Horizontal_2, F.Cu at (185.0, 78.8)
- added R9: 1K, IMRANS_LIBRARY:R_Axial_DIN0207_L6.3mm_D2.5mm_P10.16mm_Horizontal_2, F.Cu at (144.0, 119.8)
- added R9: 1K, IMRANS_LIBRARY:R_Axial_DIN0207_L6.3mm_D2.5mm_P10.16mm_Horizontal_2, F.Cu at (185.0, 119.8)
- added R9: 1K, IMRANS_LIBRARY:R_Axial_DIN0207_L6.3mm_D2.5mm_P10.16mm_Horizontal_2, F.Cu at (103.0, 78.8)
- added R9: 1K, IMRANS_LIBRARY:R_Axial_DIN0207_L6.3mm_D2.5mm_P10.16mm_Horizontal_2, F.Cu at (62.0, 160.8)
- added R9: 1K, IMRANS_LIBRARY:R_Axial_DIN0207_L6.3mm_D2.5mm_P10.16mm_Horizontal_2, F.Cu at (267.0, 160.8)
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Routing:
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- added copper zone on B.Cu, net Board_12-GNDREF
- added copper zone on B.Cu, net Board_13-GNDREF
- added copper zone on B.Cu, net Board_14-GNDREF
- added copper zone on B.Cu, net Board_15-GNDREF
- added copper zone on B.Cu, net Board_16-GNDREF
- added copper zone on B.Cu, net Board_17-GNDREF
- added copper zone on B.Cu, net Board_18-GNDREF
- added copper zone on B.Cu, net Board_19-GNDREF
- added copper zone on B.Cu, net Board_20-GNDREF
- added copper zone on B.Cu, net Board_21-GNDREF
- added copper zone on B.Cu, net Board_22-GNDREF
- added copper zone on B.Cu, net Board_23-GNDREF
Other:
- board size 225.2 x 135 mm -> 245 x 163 mm
- board text added: "B."
- board text added: "SERVE"
- board text added: "V1.4"
- board text removed: "B.KORP V2.1"
